File: Nucleo_F446_power_can_shield/Nucleo_F446_power_can_shield.kicad_pcb (KiCad board)
At the start: 2 copper layers, 139.7 x 104.9 mm, 53 parts, among them J1 ISOCAN1, J10 ISOCAN2, J11 CAN1, J12 CAN2, J13 ISOCAN1, J14 ISOCAN2, J15 CAN1, J16 CAN2, J17 RJ45, J18 RJ45, J19 I2C3, J2 ISOCAN2, J20 UART4, J21 xt60 male, J22 enable, J23 enable, J24 enable, J25 enable, J3 CAN1, J4 CAN2, J5 ISOCAN1, J6 ISOCAN2, J7 CAN1, J8 CAN2, J9 ISOCAN1, M1 Isolated-Can-Transceiver-Modu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, M2 Isolated-Can-Transceiver-Modu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, M3 TJA1050_Module, M4 TJA1050_Module, U1 NUCLEO-F446RE, U2 MP1584

Commit message: gerber
Parts:
- D6, D7, D8: footprint Diode_SMD:D_SMB-SMC_Universal_Handsoldering -> Diode_SMD:D_SMB_Handsoldering
Routing:
- net Net-(J25-Pad2): track 88.9 -> 89.7 mm
- net GND: vias 190 -> 198
Other:
- outline, holes or cut-outs redrawn
