File: canbus_board/canbus_board.kicad_pcb (KiCad board)
At the start: 2 copper layers, 14 parts, among them J1 mx3.0_2x2, J10 mx3.0_2x2, J11 TR, J12 TR, J2 mx3.0_2x2, J3 mx3.0_2x2, J4 mx3.0_2x2, J5 mx3.0_2x2, J6 mx3.0_2x2, J7 mx3.0_2x2, J8 mx3.0_2x2, J9 mx3.0_2x2

Commit message: added gerber
Parts:
- J11, J12: value TR -> Termination Resistor
- turned R1 to 0 degrees
Routing:
- net /CAN_P: track 141.8 -> 144.5 mm
- net /CAN_N: track 139.8 -> 140.7 mm
- net (no net): vias 0 -> 4
Other:
- board outline added: 73.8 x 34 mm
- board text added: "CAN BUS DIVIDER BOARD MONKEY VERSION Rev 1.0 Follow IGGG-can-molex standard by Samson Chau"
- board text added: "CAN_BUS_BRAKEOUT_BOARD"

Commit message: add all
Routing:
- added copper zone on B.Cu, net (none)
- added copper zone on F.Cu, net (none)
Other:
- board text added: "CAN BUS BRAKEOUT BOARD MONKEY VERSION Rev 1.0 Follow IGGG-can-molex standard by Samson Chau"
- board text removed: "CAN BUS DIVIDER BOARD MONKEY VERSION Rev 1.0 Follow IGGG-can-molex standard by Samson Chau"
Changed lines of the file:
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@@
       (outputformat 1)
       (mirror false)
-      (drillshape 1)
+      (drillshape 0)
       (scaleselection 1)
-      (outputdirectory "")
+      (outputdirectory "gerber/")
     )
   )
@@
     (pad "" np_thru_hole circle locked (at -3 3.94 270) (size 1 1) (drill 1) (layers *.Cu *.Mask))
     (pad "" np_thru_hole circle locked (at 6 3.94 270) (size 1 1) (drill 1) (layers *.Cu *.Mask))
-    (pad "1" thru_hole roundrect locked (at 0 0 270) (size 1.5 1.5) (drill 1) (layers *.Cu *.Mask) (roundrect_rratio 0.166667)
+    (pad "1" thru_hole roundrect locked (at 0 0 270) (size 1.5 1.5) (drill 1) (layers *.Cu *.Mask) (roundrect_rratio 0.1666673333)
       (net 1 "/CAN_P") (pinfunction "Pin_1") (pintype "passive"))
     (pad "2" thru_hole circle locked (at 3 0 270) (size 1.5 1.5) (drill 1) (layers *.Cu *.Mask)
@@
     (pad "" np_thru_hole circle locked (at 6 3.94) (size 1 1) (drill 1) (layers *.Cu *.Mask))
     (pad "" np_thru_hole circle locked (at -3 3.94) (size 1 1) (drill 1) (layers *.Cu *.Mask))
-    (pad "1" thru_hole roundrect locked (at 0 0) (size 1.5 1.5) (drill 1) (layers *.Cu *.Mask) (roundrect_rratio 0.166667)
+    (pad "1" thru_hole roundrect locked (at 0 0) (size 1.5 1.5) (drill 1) (layers *.Cu *.Mask) (roundrect_rratio 0.1666673333)
       (net 1 "/CAN_P") (pinfunction "Pin_1") (pintype "passive"))
     (pad "2" thru_hole circle locked (at 3 0) (size 1.5 1.5) (drill 1) (layers *.Cu *.Mask)
@@
     (pad "" np_thru_hole circle locked (at -3 3.94) (size 1 1) (drill 1) (layers *.Cu *.Mask))
     (pad "" np_thru_hole circle locked (at 6 3.94) (size 1 1) (drill 1) (layers *.Cu *.Mask))
-    (pad "1" thru_hole roundrect locked (at 0 0) (size 1.5 1.5) (drill 1) (layers *.Cu *.Mask) (roundrect_rratio 0.166667)
+    (pad "1" thru_hole roundrect locked (at 0 0) (size 1.5 1.5) (drill 1) (layers *.Cu *.Mask) (roundrect_rratio 0.1666673333)
       (net 1 "/CAN_P") (pinfunction "Pin_1") (pintype "passive"))
     (pad "2" thru_hole circle locked (at 3 0) (size 1.5 1.5) (drill 1) (layers *.Cu *.Mask)
@@
     (pad "" np_thru_hole circle locked (at 6 3.94 180) (size 1 1) (drill 1) (layers *.Cu *.Mask))
     (pad "" np_thru_hole circle locked (at -3 3.94 180) (size 1 1) (drill 1) (layers *.Cu *.Mask))
-    (pad "1" thru_hole roundrect locked (at 0 0 180) (size 1.5 1.5) (drill 1) (layers *.Cu *.Mask) (roundrect_rratio 0.166667)
+    (pad "1" thru_hole roundrect locked (at 0 0 180) (size 1.5 1.5) (drill 1) (layers *.Cu *.Mask) (roundrect_rratio 0.1666673333)
       (net 1 "/CAN_P") (pinfunction "Pin_1") (pintype "passive"))
     (pad "2" thru_hole circle locked (at 3 0 180) (size 1.5 1.5) (drill 1) (layers *.Cu *.Mask)
@@
     (pad "" np_thru_hole circle locked (at 6 3.94 180) (size 1 1) (drill 1) (layers *.Cu *.Mask))
     (pad "" np_thru_hole circle locked (at -3 3.94 180) (size 1 1) (drill 1) (layers *.Cu *.Mask))
-    (pad "1" thru_hole roundrect locked (at 0 0 180) (size 1.5 1.5) (drill 1) (layers *.Cu *.Mask) (roundrect_rratio 0.166667)
+    (pad "1" thru_hole roundrect locked (at 0 0 180) (size 1.5 1.5) (drill 1) (layers *.Cu *.Mask) (roundrect_rratio 0.1666673333)
       (net 1 "/CAN_P") (pinfunction "Pin_1") (pintype "passive"))
     (pad "2" thru_hole circle locked (at 3 0 180) (size 1.5 1.5) (drill 1) (layers *.Cu *.Mask)
@@
     (fp_line (start -1 0.625) (end -1 -0.625) (layer "F.Fab") (width 0.1))
     (fp_line (start -1 -0.625) (end 1 -0.625) (layer "F.Fab") (width 0.1))
-    (pad "1" smd roundrect locked (at -1 0) (size 1.2 1.4) (layers "F.Cu" "F.Paste" "F.Mask") (roundrect_rratio 0.208333)
+    (pad "1" smd roundrect locked (at -1 0) (size 1.2 1.4) (layers "F.Cu" "F.Paste" "F.Mask") (roundrect_rratio 0.2083333333)
       (net 4 "Net-(J11-Pad2)") (pintype "passive"))
-    (pad "2" smd roundrect locked (at 1 0) (size 1.2 1.4) (layers "F.Cu" "F.Paste" "F.Mask") (roundrect_rratio 0.208333)
+    (pad "2" smd roundrect locked (at 1 0) (size 1.2 1.4) (layers "F.Cu" "F.Paste" "F.Mask") (roundrect_rratio 0.2083333333)
       (net 1 "/CAN_P") (pintype "passive"))
     (model "${KICAD6_3DMODEL_DIR}/Resistor_SMD.3dshapes/R_0805_2012Metric.wrl"
@@
     (pad "" np_thru_hole circle locked (at -3 3.94) (size 1 1) (drill 1) (layers *.Cu *.Mask))
     (pad "" np_thru_hole circle locked (at 6 3.94) (size 1 1) (drill 1) (layers *.Cu *.Mask))
-    (pad "1" thru_hole roundrect locked (at 0 0) (size 1.5 1.5) (drill 1) (layers *.Cu *.Mask) (roundrect_rratio 0.166667)
+    (pad "1" thru_hole roundrect locked (at 0 0) (size 1.5 1.5) (drill 1) (layers *.Cu *.Mask) (roundrect_rratio 0.1666673333)
       (net 1 "/CAN_P") (pinfunction "Pin_1") (pintype "passive"))
     (pad "2" thru_hole circle locked (at 3 0) (size 1.5 1.5) (drill 1) (layers *.Cu *.Mask)
@@
     (pad "" np_thru_hole circle locked (at 6 3.94) (size 1 1) (drill 1) (layers *.Cu *.Mask))
     (pad "" np_thru_hole circle locked (at -3 3.94) (size 1 1) (drill 1) (layers *.Cu *.Mask))
-    (pad "1" thru_hole roundrect locked (at 0 0) (size 1.5 1.5) (drill 1) (layers *.Cu *.Mask) (roundrect_rratio 0.166667)
+    (pad "1" thru_hole roundrect locked (at 0 0) (size 1.5 1.5) (drill 1) (layers *.Cu *.Mask) (roundrect_rratio 0.1666673333)
       (net 1 "/CAN_P") (pinfunction "Pin_1") (pintype "passive"))
     (pad "2" thru_hole circle locked (at 3 0) (size 1.5 1.5) (drill 1) (layers *.Cu *.Mask)
@@
     (pad "" np_thru_hole circle locked (at -3 3.94 270) (size 1 1) (drill 1) (layers *.Cu *.Mask))
     (pad "" np_thru_hole circle locked (at 6 3.94 270) (size 1 1) (drill 1) (layers *.Cu *.Mask))
-    (pad "1" thru_hole roundrect locked (at 0 0 270) (size 1.5 1.5) (drill 1) (layers *.Cu *.Mask) (roundrect_rratio 0.166667)
+    (pad "1" thru_hole roundrect locked (at 0 0 270) (size 1.5 1.5) (drill 1) (layers *.Cu *.Mask) (roundrect_rratio 0.1666673333)
       (net 1 "/CAN_P") (pinfunction "Pin_1") (pintype "passive"))
     (pad "2" thru_hole circle locked (at 3 0 270) (size 1.5 1.5) (drill 1) (layers *.Cu *.Mask)
@@
     (pad "" np_thru_hole circle locked (at -3 3.94 180) (size 1 1) (drill 1) (layers *.Cu *.Mask))
     (pad "" np_thru_hole circle locked (at 6 3.94 180) (size 1 1) (drill 1) (layers *.Cu *.Mask))
-    (pad "1" thru_hole roundrect locked (at 0 0 180) (size 1.5 1.5) (drill 1) (layers *.Cu *.Mask) (roundrect_rratio 0.166667)
+    (pad "1" thru_hole roundrect locked (at 0 0 180) (size 1.5 1.5) (drill 1) (layers *.Cu *.Mask) (roundrect_rratio 0.1666673333)
       (net 1 "/CAN_P") (pinfunction "Pin_1") (pintype "passive"))
     (pad "2" thru_hole circle locked (at 3 0 180) (size 1.5 1.5) (drill 1) (layers *.Cu *.Mask)
@@
     (pad "" np_thru_hole circle locked (at -3 3.94 180) (size 1 1) (drill 1) (layers *.Cu *.Mask))
     (pad "" np_thru_hole circle locked (at 6 3.94 180) (size 1 1) (drill 1) (layers *.Cu *.Mask))
-    (pad "1" thru_hole roundrect locked (at 0 0 180) (size 1.5 1.5) (drill 1) (layers *.Cu *.Mask) (roundrect_rratio 0.166667)
+    (pad "1" thru_hole roundrect locked (at 0 0 180) (size 1.5 1.5) (drill 1) (layers *.Cu *.Mask) (roundrect_rratio 0.1666673333)
       (net 1 "/CAN_P") (pinfunction "Pin_1") (pintype "passive"))
     (pad "2" thru_hole circle locked (at 3 0 180) (size 1.5 1.5) (drill 1) (layers *.Cu *.Mask)
@@
     (fp_line (start -1 0.625) (end -1 -0.625) (layer "F.Fab") (width 0.1))
     (fp_line (start -1 -0.625) (end 1 -0.625) (layer "F.Fab") (width 0.1))
-    (pad "1" smd roundrect locked (at -1 0) (size 1.2 1.4) (layers "F.Cu" "F.Paste" "F.Mask") (roundrect_rratio 0.208333)
+    (pad "1" smd roundrect locked (at -1 0) (size 1.2 1.4) (layers "F.Cu" "F.Paste" "F.Mask") (roundrect_rratio 0.2083333333)
       (net 5 "Net-(J12-Pad2)") (pintype "passive"))
-    (pad "2" smd roundrect locked (at 1 0) (size 1.2 1.4) (layers "F.Cu" "F.Paste" "F.Mask") (roundrect_rratio 0.208333)
+    (pad "2" smd roundrect locked (at 1 0) (size 1.2 1.4) (layers "F.Cu" "F.Paste" "F.Mask") (roundrect_rratio 0.2083333333)
       (net 1 "/CAN_P") (pintype "passive"))
     (model "${KICAD6_3DMODEL_DIR}/Resistor_SMD.3dshapes/R_0805_2012Metric.wrl"
@@
   )
   (gr_rect (start 127.635 34.544) (end 53.848 68.58) (layer "Edge.Cuts") (width 0.1) (fill none))
-  (gr_text "CAN BUS DIVIDER BOARD MONKEY VERSION\nRev 1.0 \n\nFollow IGGG-can-molex standard\nby Samson Chau " (at 88.9 52.07) (layer "B.SilkS")
+  (gr_text "CAN BUS BRAKEOUT BOARD MONKEY VERSION\nRev 1.0 \nFollow IGGG-can-molex standard\nby Samson Chau " (at 88.9 52.07) (layer "B.SilkS")
     (effects (font (size 1 1) (thickness 0.15)) (justify mirror))
   )
@@
   (segment (start 57.531 50.165) (end 57.531 46.096) (width 0.25) (layer "F.Cu") (net 5))
   (segment (start 57.531 46.096) (end 58.42 45.207) (width 0.25) (layer "F.Cu") (net 5))
+  (zone (net 0) (net_name "") (layer "F.Cu") (hatch edge 0.508)
+    (connect_pads (clearance 0.508))
+    (min_thickness 0.254) (filled_areas_thickness no)
+    (fill yes (thermal_gap 0.508) (thermal_bridge_width 0.508))
+    (polygon
+      (pts
+        (xy 124.968 66.04)
+        (xy 56.896 66.04)
+        (xy 56.896 37.084)
+        (xy 124.968 37.084)
+      )
+    )
+  )
+  (zone (net 0) (net_name "") (layer "B.Cu") (hatch edge 0.508)
+    (connect_pads (clearance 0.508))
+    (min_thickness 0.254) (filled_areas_thickness no)
+    (fill yes (thermal_gap 0.508) (thermal_bridge_width 0.508))
+    (polygon
+      (pts
+        (xy 124.968 66.04)
+        (xy 56.896 66.04)
+        (xy 56.896 37.084)
+        (xy 124.968 37.084)
+      )
+    )
+  )
 )

Commit message: mod graphic
Parts:
- added G***: LOGO, PolyuRobotics:Club_logo, F.Cu at (112.4, 38.7)
- added G***: LOGO, PolyuRobotics:Club_logo, B.Cu at (88.4, 39.1)
- J11, J12: value Termination Resistor -> resistor
Connections:
- J1 pad 3: unconnected-(J1-Pad3) -> GND
- J10 pad 3: unconnected-(J10-Pad3) -> GND
- J2 pad 3: unconnected-(J2-Pad3) -> GND
- J3 pad 3: unconnected-(J3-Pad3) -> GND
- J4 pad 3: unconnected-(J4-Pad3) -> GND
- J5 pad 3: unconnected-(J5-Pad3) -> GND
- J6 pad 3: unconnected-(J6-Pad3) -> GND
- J7 pad 3: unconnected-(J7-Pad3) -> GND
- J8 pad 3: unconnected-(J8-Pad3) -> GND
- J9 pad 3: unconnected-(J9-Pad3) -> GND
Routing:
- added copper zone on B.Cu, net GND
- added copper zone on F.Cu, net GND
- removed copper zone on B.Cu, net (none)
- removed copper zone on F.Cu, net (none)
