File: canbus_board/canbus_board.kicad_sch (KiCad schematic)
At the start: 14 parts, among them J1 mx3.0_2x2, J10 mx3.0_2x2, J11 resistor, J12 resistor, J2 mx3.0_2x2, J3 mx3.0_2x2, J4 mx3.0_2x2, J5 mx3.0_2x2, J6 mx3.0_2x2, J7 mx3.0_2x2, J8 mx3.0_2x2, J9 mx3.0_2x2

Commit message: mod graphic
Connections:
- net GND: now reaches J4.3 (Pin_3)
- net GND: now also J1.3 (Pin_3), J10.3 (Pin_3), J2.3 (Pin_3), J3.3 (Pin_3), J5.3 (Pin_3), J6.3 (Pin_3), J7.3 (Pin_3), J8.3 (Pin_3), J9.3 (Pin_3)
- no-connect marks 20 -> 10
Changed lines of the file:
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@@
   (junction (at 144.78 67.31) (diameter 0) (color 0 0 0 0)
   )
+  (junction (at 175.26 38.1) (diameter 0) (color 0 0 0 0)
+  )
   (junction (at 113.03 67.31) (diameter 0) (color 0 0 0 0)
   )
+  (junction (at 99.06 38.1) (diameter 0) (color 0 0 0 0)
+  )
+  (junction (at 132.08 38.1) (diameter 0) (color 0 0 0 0)
+  )
   (junction (at 172.72 67.31) (diameter 0) (color 0 0 0 0)
   )
@@
   (junction (at 132.08 72.39) (diameter 0) (color 0 0 0 0)
   )
+  (junction (at 147.32 38.1) (diameter 0) (color 0 0 0 0)
+  )
   (junction (at 99.06 72.39) (diameter 0) (color 0 0 0 0)
   )
   (junction (at 68.58 67.31) (diameter 0) (color 0 0 0 0)
   )
+  (junction (at 83.82 38.1) (diameter 0) (color 0 0 0 0)
+  )
   (junction (at 115.57 72.39) (diameter 0) (color 0 0 0 0)
   )
@@
   (junction (at 203.2 67.31) (diameter 0) (color 0 0 0 0)
   )
+  (junction (at 71.12 38.1) (diameter 0) (color 0 0 0 0)
+  )
   (junction (at 71.12 72.39) (diameter 0) (color 0 0 0 0)
   )
+  (junction (at 55.88 38.1) (diameter 0) (color 0 0 0 0)
+  )
   (junction (at 96.52 67.31) (diameter 0) (color 0 0 0 0)
   )
   (junction (at 205.74 72.39) (diameter 0) (color 0 0 0 0)
   )
+  (junction (at 115.57 38.1) (diameter 0) (color 0 0 0 0)
+  )
   (junction (at 160.02 67.31) (diameter 0) (color 0 0 0 0)
   )
   (junction (at 175.26 72.39) (diameter 0) (color 0 0 0 0)
   )
+  (junction (at 162.56 38.1) (diameter 0) (color 0 0 0 0)
+  )
   (junction (at 162.56 72.39) (diameter 0) (color 0 0 0 0)
   )
   (no_connect (at 144.78 44.45))
-  (no_connect (at 132.08 44.45))
   (no_connect (at 129.54 44.45))
-  (no_connect (at 115.57 44.45))
   (no_connect (at 113.03 44.45))
-  (no_connect (at 99.06 44.45))
   (no_connect (at 96.52 44.45))
-  (no_connect (at 83.82 44.45))
-  (no_connect (at 162.56 44.45))
   (no_connect (at 160.02 44.45))
-  (no_connect (at 147.32 44.45))
-  (no_connect (at 191.77 44.45))
   (no_connect (at 189.23 44.45))
-  (no_connect (at 175.26 44.45))
   (no_connect (at 172.72 44.45))
   (no_connect (at 81.28 44.45))
-  (no_connect (at 71.12 44.45))
   (no_connect (at 68.58 44.45))
-  (no_connect (at 55.88 44.45))
   (no_connect (at 53.34 44.45))
   (wire (pts (xy 162.56 72.39) (xy 175.26 72.39))
@@
     (stroke (width 0) (type default) (color 0 0 0 0))
   )
+  (wire (pts (xy 191.77 44.45) (xy 191.77 38.1))
+    (stroke (width 0) (type default) (color 0 0 0 0))
+  )
+  (wire (pts (xy 55.88 38.1) (xy 34.925 38.1))
+    (stroke (width 0) (type default) (color 0 0 0 0))
+  )
   (wire (pts (xy 144.78 57.15) (xy 144.78 67.31))
     (stroke (width 0) (type default) (color 0 0 0 0))
   )
+  (wire (pts (xy 99.06 38.1) (xy 83.82 38.1))
+    (stroke (width 0) (type default) (color 0 0 0 0))
+  )
   (wire (pts (xy 189.23 57.15) (xy 189.23 67.31))
     (stroke (width 0) (type default) (color 0 0 0 0))
@@
     (stroke (width 0) (type default) (color 0 0 0 0))
   )
+  (wire (pts (xy 147.32 38.1) (xy 147.32 44.45))
+    (stroke (width 0) (type default) (color 0 0 0 0))
+  )
+  (wire (pts (xy 83.82 38.1) (xy 71.12 38.1))
+    (stroke (width 0) (type default) (color 0 0 0 0))
+  )
+  (wire (pts (xy 147.32 38.1) (xy 162.56 38.1))
+    (stroke (width 0) (type default) (color 0 0 0 0))
+  )
+  (wire (pts (xy 115.57 38.1) (xy 115.57 44.45))
+    (stroke (width 0) (type default) (color 0 0 0 0))
+  )
   (wire (pts (xy 205.74 72.39) (xy 219.71 72.39))
     (stroke (width 0) (type default) (color 0 0 0 0))
   )
+  (wire (pts (xy 34.925 38.1) (xy 34.925 57.15))
+    (stroke (width 0) (type default) (color 0 0 0 0))
+  )
   (wire (pts (xy 113.03 67.31) (xy 129.54 67.31))
     (stroke (width 0) (type default) (color 0 0 0 0))
@@
     (stroke (width 0) (type default) (color 0 0 0 0))
   )
+  (wire (pts (xy 175.26 38.1) (xy 191.77 38.1))
+    (stroke (width 0) (type default) (color 0 0 0 0))
+  )
+  (wire (pts (xy 162.56 38.1) (xy 175.26 38.1))
+    (stroke (width 0) (type default) (color 0 0 0 0))
+  )
   (wire (pts (xy 99.06 72.39) (xy 115.57 72.39))
     (stroke (width 0) (type default) (color 0 0 0 0))
@@
     (stroke (width 0) (type default) (color 0 0 0 0))
   )
+  (wire (pts (xy 71.12 38.1) (xy 55.88 38.1))
+    (stroke (width 0) (type default) (color 0 0 0 0))
+  )
+  (wire (pts (xy 175.26 38.1) (xy 175.26 44.45))
+    (stroke (width 0) (type default) (color 0 0 0 0))
+  )
+  (wire (pts (xy 132.08 44.45) (xy 132.08 38.1))
+    (stroke (width 0) (type default) (color 0 0 0 0))
+  )
   (wire (pts (xy 175.26 72.39) (xy 191.77 72.39))
     (stroke (width 0) (type default) (color 0 0 0 0))
   )
+  (wire (pts (xy 115.57 38.1) (xy 132.08 38.1))
+    (stroke (width 0) (type default) (color 0 0 0 0))
+  )
   (wire (pts (xy 81.28 57.15) (xy 81.28 67.31))
     (stroke (width 0) (type default) (color 0 0 0 0))
@@
     (stroke (width 0) (type default) (color 0 0 0 0))
   )
+  (wire (pts (xy 132.08 38.1) (xy 147.32 38.1))
+    (stroke (width 0) (type default) (color 0 0 0 0))
+  )
   (wire (pts (xy 205.74 50.8) (xy 205.74 72.39))
     (stroke (width 0) (type default) (color 0 0 0 0))
@@
     (stroke (width 0) (type default) (color 0 0 0 0))
   )
+  (wire (pts (xy 71.12 38.1) (xy 71.12 44.45))
+    (stroke (width 0) (type default) (color 0 0 0 0))
+  )
   (wire (pts (xy 83.82 72.39) (xy 99.06 72.39))
     (stroke (width 0) (type default) (color 0 0 0 0))
   )
+  (wire (pts (xy 99.06 38.1) (xy 99.06 44.45))
+    (stroke (width 0) (type default) (color 0 0 0 0))
+  )
   (wire (pts (xy 68.58 67.31) (xy 81.28 67.31))
     (stroke (width 0) (type default) (color 0 0 0 0))
@@
     (stroke (width 0) (type default) (color 0 0 0 0))
   )
+  (wire (pts (xy 83.82 38.1) (xy 83.82 44.45))
+    (stroke (width 0) (type default) (color 0 0 0 0))
+  )
+  (wire (pts (xy 55.88 38.1) (xy 55.88 44.45))
+    (stroke (width 0) (type default) (color 0 0 0 0))
+  )
   (wire (pts (xy 68.58 57.15) (xy 68.58 67.31))
     (stroke (width 0) (type default) (color 0 0 0 0))
   )
   (wire (pts (xy 53.34 67.31) (xy 68.58 67.31))
+    (stroke (width 0) (type default) (color 0 0 0 0))
+  )
+  (wire (pts (xy 115.57 38.1) (xy 99.06 38.1))
+    (stroke (width 0) (type default) (color 0 0 0 0))
+  )
+  (wire (pts (xy 162.56 38.1) (xy 162.56 44.45))
     (stroke (width 0) (type default) (color 0 0 0 0))
   )
@@
     (pin "4")
   )
+  (symbol (lib_id "power:GND") (at 34.925 57.15 0) (unit 1)
+    (in_bom yes) (on_board yes) (fields_autoplaced)
+    (property "Reference" "#PWR0101" (id 0) (at 34.925 63.5 0)
+      (effects (font (size 1.27 1.27)) hide)
+    )
+    (property "Value" "GND" (id 1) (at 34.925 62.23 0))
+    (property "Footprint" "" (id 2) (at 34.925 57.15 0)
+      (effects (font (size 1.27 1.27)) hide)
+    )
+    (property "Datasheet" "" (id 3) (at 34.925 57.15 0)
+      (effects (font (size 1.27 1.27)) hide)
+    )
+    (pin "1")
+  )
   (symbol (lib_id "Device:R_Small") (at 203.2 57.15 0) (unit 1)
     (in_bom yes) (on_board yes)
@@
   )
   (symbol_instances
+    (path "/5ceea8f2-f416-4c6d-9821-df752bd8836c"
+      (reference "#PWR0101") (unit 1) (value "GND") (footprint "")
+    )
     (path "/cf0a08fc-a7e1-4e2e-b77b-d5d82ed08115"
       (reference "J1") (unit 1) (value "mx3.0_2x2") (footprint "Connector_Molex:Molex_Micro-Fit_3.0_43045-0412_2x02_P3.00mm_Vertical")
