File: XT60_CAN/XT60_CAN.kicad_pcb (KiCad board)
At the start: 2 copper layers, 141 x 54.6 mm, 28 parts, among them J1 XT60_IN, J10 mx3.0_2x2, J11 mx3.0_2x2, J12 mx3.0_2x2, J13 mx3.0_2x2, J14 mx3.0_2x2, J15 XT60_CH4, J16 XT60_CH5, J17 resistor, J18 resistor, J19 DC step down power, J2 XT60_CH1, J20 DC step down power, J3 mx3.0_2x2, J4 mx3.0_2x2, J5 mx3.0_2x2, J6 mx3.0_2x2, J7 mx3.0_2x2, J8 XT60_CH2, J9 XT60_CH3, U1 DCDC_StepDown_LM2596

Commit message: graphics
Parts:
- added G***: LOGO, PolyuRobotics:Club_logo, F.Cu at (183.4, 85.9)
- added G***: LOGO, PolyuRobotics:Raymond, B.Cu at (90.9, 49.3)
Other:
- board text added: "BATT input"
- board text added: "DC 12V"
- board text added: "GND"
- board text added: "IGGG can bus power divider by SamsonChau 2022-2-2"
- board text added: "VCC"
- board text added: "Vin"

Commit message: power_board
Parts:
- removed J10, J11, J12, J13, J14, J7: mx3.0_2x2, Connector_Molex:Molex_Micro-Fit_3.0_43045-0412_2x02_P3.00mm_Vertical
- removed J17, J18: resistor, Connector_PinHeader_2.54mm:PinHeader_1x02_P2.54mm_Vertical
- added C1: 10v 100uF, Capacitor_SMD:C_Elec_5x5.4, F.Cu at (128.3, 73.7)
- added C2: 16v 220uF, Capacitor_SMD:C_Elec_6.3x7.7, F.Cu at (150.7, 73.7)
- added C3: 25v 100uF, Capacitor_SMD:C_Elec_6.3x7.7, F.Cu at (174.0, 73.7)
- added C4: 50v 47uF, Capacitor_SMD:C_Elec_6.3x7.7, F.Cu at (84.1, 29.7)
- added C5: 50v 47uF, Capacitor_SMD:C_Elec_6.3x7.7, F.Cu at (73.9, 41.1)
- added C6: 50v 47uF, Capacitor_SMD:C_Elec_6.3x7.7, F.Cu at (84.1, 41.1)
- added D1: SMBJ5CA, Diode_SMD:D_SMB, F.Cu at (128.3, 66.0)
- added D2: SMBJ9CA, Diode_SMD:D_SMB, F.Cu at (151.1, 66.0)
- added D3: SMBJ12CA, Diode_SMD:D_SMB, F.Cu at (174.5, 66.0)
- added D4: SMBJ24CA, Diode_SMD:D_SMB, F.Cu at (73.9, 29.7)
- added D5: 5v_led, LED_SMD:LED_0805_2012Metric_Pad1.15x1.40mm_HandSolder, F.Cu at (135.9, 66.0)
- added D6: 9v_led, LED_SMD:LED_0805_2012Metric_Pad1.15x1.40mm_HandSolder, F.Cu at (158.4, 68.6)
- added D7: 12v_led, LED_SMD:LED_0805_2012Metric_Pad1.15x1.40mm_HandSolder, F.Cu at (184.2, 68.6)
- added F6: 3557-2, PolyuRobotics:FUSE_3557-2, F.Cu at (87.6, 58.4)
- added F7: 3557-2, PolyuRobotics:FUSE_3557-2, F.Cu at (100.3, 58.4)
- added F8: 3557-2, PolyuRobotics:FUSE_3557-2, F.Cu at (113.0, 58.4)
- added R3: 33k, Resistor_SMD:R_0805_2012Metric_Pad1.20x1.40mm_HandSolder, F.Cu at (184.2, 73.7)
- added U2: MP1584, PolyuRobotics:DC-DC-mp1584_module, F.Cu at (168.1, 37.3)
- added U3: MP1584, PolyuRobotics:DC-DC-mp1584_module, F.Cu at (122.4, 37.3)
- F1, F2, F3, F4, F5: value Fuse -> 3557-2; footprint Fuse_custom:Keystone_3557-2 -> PolyuRobotics:FUSE_3557-2
- J19, J20: value DC step down power -> +5V
- J3, J5: value mx3.0_2x2 -> +9V; footprint Connector_Molex:Molex_Micro-Fit_3.0_43045-0412_2x02_P3.00mm_Vertical -> Connector_Molex:Molex_Micro-Fit_3.0_43045-0212_2x01_P3.00mm_Vertical
- J4, J6: value mx3.0_2x2 -> +12V; footprint Connector_Molex:Molex_Micro-Fit_3.0_43045-0412_2x02_P3.00mm_Vertical -> Connector_Molex:Molex_Micro-Fit_3.0_43045-0212_2x01_P3.00mm_Vertical
- R1: value 120R -> 10k
- R2: value 120R -> 22k
- U1: value DCDC_StepDown_LM2596 -> MP1584; footprint mid_DCDC2:YAAJ_DCDC_StepDown_LM2596 -> PolyuRobotics:DC-DC-mp1584_module
- moved F5 86.7 mm to (74.9, 58.4), turned to 90 degrees
- moved F4 75.5 mm to (62.2, 58.4), turned to 90 degrees
- moved U1 71.6 mm to (144.9, 37.3), turned to -90 degrees
- moved F1 64.4 mm to (114.3, 35.3)
- moved J16 58.6 mm to (113.0, 84.9)
- moved R1 57.5 mm to (135.9, 71.1), turned to 90 degrees
- moved G*** 56.5 mm to (173.7, 30.2)
- moved J4 48.7 mm to (183.1, 82.3), turned to 0 degrees
- moved J15 47.3 mm to (100.3, 84.9)
- moved F2 43.4 mm to (105.4, 35.3)
- moved F3 42.6 mm to (96.0, 35.3)
- moved J3 38.4 mm to (148.1, 82.3), turned to 0 degrees
- moved J20 38.1 mm to (126.2, 82.5), turned to 0 degrees
- moved J6 37.9 mm to (171.5, 82.3), turned to 0 degrees
- moved J5 37.8 mm to (159.1, 82.3), turned to 0 degrees
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Connections:
- F1 pad 1: +24V -> Net-(F1-Pad1)
- F1 pad 2: Net-(F1-Pad2) -> +24V
- F2 pad 1: +24V -> Net-(F2-Pad1)
- F2 pad 2: Net-(F2-Pad2) -> +24V
- F3 pad 1: +24V -> Net-(F3-Pad1)
- F3 pad 2: Net-(F3-Pad2) -> +24V
- F4 pad 1: +24V -> Net-(F4-Pad1)
- F4 pad 2: Net-(F4-Pad2) -> +24V
- F5 pad 1: +24V -> Net-(F5-Pad1)
- F5 pad 2: Net-(F5-Pad2) -> +24V
- J1 pad 1: +24V -> GNDPWR
- J1 pad 2: GND -> +24V
- J15 pad 1: Net-(F4-Pad2) -> GNDPWR
- J15 pad 2: GNDPWR -> Net-(F7-Pad1)
- J16 pad 1: Net-(F5-Pad2) -> GNDPWR
- J16 pad 2: GNDPWR -> Net-(F8-Pad1)
- J19 pad 1: VCC -> +5V
- J2 pad 1: Net-(F1-Pad2) -> GNDPWR
- J2 pad 2: GNDPWR -> Net-(F4-Pad1)
- J20 pad 1: VCC -> +5V
- J3 pad 1: /CAN_P -> +9V
- J3 pad 2: /CAN_N -> GND
- J4 pad 1: /CAN_P -> +12V
- J4 pad 2: /CAN_N -> GND
- J5 pad 1: /CAN_P -> +9V
- J5 pad 2: /CAN_N -> GND
- J6 pad 1: /CAN_P -> +12V
- J6 pad 2: /CAN_N -> GND
- J8 pad 1: Net-(F2-Pad2) -> GNDPWR
- J8 pad 2: GNDPWR -> Net-(F5-Pad1)
- J9 pad 1: Net-(F3-Pad2) -> GNDPWR
- J9 pad 2: GNDPWR -> Net-(F6-Pad1)
- R1 pad 1: Net-(R1-Pad1) -> +5V
- R1 pad 2: /CAN_P -> Net-(D5-Pad2)
- R2 pad 1: Net-(J18-Pad2) -> +9V
- R2 pad 2: /CAN_P -> Net-(D6-Pad2)
Routing:
- net /CAN_P: track 200.2 -> 0.00 mm, vias 1 -> 0
- net /CAN_N: track 173.4 -> 0.00 mm
- net Net-(F1-Pad1): track 0.00 -> 132.8 mm
- net Net-(F3-Pad1): track 0.00 -> 83.2 mm
- net Net-(F2-Pad1): track 0.00 -> 54.0 mm
- net +5V: track 0.00 -> 47.2 mm
- net +12V: track 0.00 -> 46.4 mm
- net +9V: track 0.00 -> 45.7 mm
- net VCC: track 28.5 -> 0.00 mm
- net Net-(F8-Pad1): track 0.00 -> 16.6 mm
- net Net-(F7-Pad1): track 0.00 -> 16.6 mm
- net Net-(F6-Pad1): track 0.00 -> 16.6 mm
- net Net-(F5-Pad1): track 0.00 -> 16.6 mm
- net Net-(F4-Pad1): track 0.00 -> 15.0 mm
- net Net-(F1-Pad2): track 12.6 -> 0.00 mm
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- removed copper zone on B.Cu, net GND
- removed copper zone on F.Cu, net GND
- removed copper zone on B.Cu, net GNDPWR
- removed copper zone on F.Cu, net GNDPWR
Other:
- board outline removed
- board text removed: "DC 12V"
- board text removed: "GND"
- board text removed: "VCC"
- board text removed: "Vin"

Commit message: power_board
Parts:
- removed the G*** at (90.9, 49.3)
- moved D6 4.36 mm to (159.5, 64.4)
- moved R2 4.36 mm to (159.5, 69.5)
- moved D2 3.98 mm to (151.6, 62.1)
- moved D3 3.98 mm to (175.0, 62.1)
- moved D5 3.98 mm to (136.4, 62.1)
- moved J19 3.98 mm to (136.9, 78.6)
- moved J20 3.98 mm to (126.7, 78.6)
- moved J3 3.98 mm to (148.6, 78.3)
- moved J5 3.98 mm to (159.7, 78.3)
- moved J6 3.98 mm to (172.0, 78.4)
- moved R1 3.98 mm to (136.4, 67.2)
- moved C1 3.98 mm to (128.8, 69.7)
- moved C2 3.98 mm to (151.3, 69.7)
- moved C3 3.98 mm to (174.5, 69.7)
- moved D1 3.98 mm to (128.8, 62.1)
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Routing:
- net +24V: track 202.5 -> 199.8 mm
- net +12V: track 46.4 -> 45.2 mm
- net Net-(F2-Pad1): track 54.0 -> 53.4 mm
Other:
- board outline added: 132.1 x 68.6 mm
- board text added: "10k"
- board text added: "10v 100uF"
- board text added: "12V Fulse"
- board text added: "16v 220uF"
- board text added: "22k"
- board text added: "24V->12V"
- board text added: "24V->5V"
- board text added: "24V->9V"
- board text added: "25v 100uF"
- board text added: "33k"
- board text added: "50V 47uF"
- board text added: "5V Fulse"
- board text added: "9V Fulse"
- board text added: "SMBJ12CA"
- board text added: "SMBJ24CA"
- board text added: "SMBJ5CA"
- board text added: "SMBJ9CA"

Commit message: terminal
Parts:
- removed J19, J20: +5V, Connector_Molex:Molex_Micro-Fit_3.0_43045-0212_2x01_P3.00mm_Vertical
- added J10: +12v, TerminalBlock:TerminalBlock_Altech_AK300-2_P5.00mm, F.Cu at (182.1, 82.8)
- added J7: +9v, TerminalBlock:TerminalBlock_Altech_AK300-2_P5.00mm, F.Cu at (148.1, 82.8)
- J3: value +9V -> +5v; footprint Connector_Molex:Molex_Micro-Fit_3.0_43045-0212_2x01_P3.00mm_Vertical -> TerminalBlock:TerminalBlock_Altech_AK300-2_P5.00mm
- J4: value +12V -> +9v; footprint Connector_Molex:Molex_Micro-Fit_3.0_43045-0212_2x01_P3.00mm_Vertical -> TerminalBlock:TerminalBlock_Altech_AK300-2_P5.00mm
- J5: value +9V -> +12v; footprint Connector_Molex:Molex_Micro-Fit_3.0_43045-0212_2x01_P3.00mm_Vertical -> TerminalBlock:TerminalBlock_Altech_AK300-2_P5.00mm
- J6: value +12V -> +5v; footprint Connector_Molex:Molex_Micro-Fit_3.0_43045-0212_2x01_P3.00mm_Vertical -> TerminalBlock:TerminalBlock_Altech_AK300-2_P5.00mm
- moved J6 35.6 mm to (136.7, 82.8)
- moved J4 24.0 mm to (159.5, 82.8)
- moved J3 23.7 mm to (125.3, 82.8)
- moved J5 11.9 mm to (170.7, 82.8)
Connections:
- J3 pad 1: +9V -> +5V
- J4 pad 1: +12V -> +9V
- J5 pad 1: +9V -> +12V
- J6 pad 1: +12V -> +5V
Routing:
- net +12V: track 45.2 -> 61.3 mm
- net +5V: track 47.2 -> 59.0 mm
- net +9V: track 45.7 -> 56.6 mm

Commit message: terminal
Parts:
- added G***: LOGO, PolyuRobotics:Club_logo, B.Cu at (158.8, 62.2)
- moved R3 4.95 mm to (188.0, 68.8)
- moved D7 4.95 mm to (188.0, 63.8)
- moved C3 4.95 mm to (179.3, 68.6)
- moved D3 4.95 mm to (179.8, 61.0)
- moved U2 4.95 mm to (173.5, 32.2)
- moved J10 4.82 mm to (186.7, 81.3)
- moved D2 4.04 mm to (155.6, 61.2)
- moved D6 4.04 mm to (163.5, 63.5)
- moved R2 4.04 mm to (163.5, 68.6)
- moved U1 4.04 mm to (149.3, 32.4)
- moved C2 4.04 mm to (155.2, 68.8)
- moved J5 3.84 mm to (174.2, 81.3)
- moved J1 3.56 mm to (66.0, 40.6)
- moved G*** 3.07 mm to (180.6, 28.8)
- moved D1 3.04 mm to (131.7, 61.2)
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Connections:
- J1 pad 1: GNDPWR -> GND
- J15 pad 1: GNDPWR -> GND
- J16 pad 1: GNDPWR -> GND
- J2 pad 1: GNDPWR -> GND
- J8 pad 1: GNDPWR -> GND
- J9 pad 1: GNDPWR -> GND
- U1 pad IN1-: GNDPWR -> GND
- U1 pad IN2-: GNDPWR -> GND
- U1 pad OUT1-: GNDPWR -> GND
- U1 pad OUT2-: GNDPWR -> GND
- U2 pad IN1-: GNDPWR -> GND
- U2 pad IN2-: GNDPWR -> GND
- U2 pad OUT1-: GNDPWR -> GND
- U2 pad OUT2-: GNDPWR -> GND
- U3 pad IN1-: GNDPWR -> GND
- U3 pad IN2-: GNDPWR -> GND
- U3 pad OUT1-: GNDPWR -> GND
- U3 pad OUT2-: GNDPWR -> GND
Routing:
- net Net-(F1-Pad1): track 132.5 -> 15.9 mm
- net +24V: track 199.8 -> 225.5 mm
- net Net-(F2-Pad1): track 53.4 -> 61.3 mm
- net Net-(F3-Pad1): track 83.2 -> 87.4 mm
- net +9V: track 56.6 -> 55.0 mm
- net +12V: track 61.3 -> 60.7 mm
- net GND: vias 0 -> 56
- net (no net): vias 0 -> 4
- added copper zone on B.Cu, net GND
- added copper zone on F.Cu, net GND
Other:
- board size 132.1 x 68.6 mm -> 141 x 67.6 mm
- board text added: "12V GND"
- board text added: "5V GND"
- board text added: "9V GND"
