File: POS_card/POS_card.kicad_sch (KiCad schematic)
At the start: 27 parts

Commit message: POS_CARD
Parts:
- added C1, C2: 22pF, symbol Device:C_Small
- added C10, C15, C17: 100nf, symbol Device:C_Small
- added C21, C23, C3: 100nF, symbol Device:C_Small
- added D1: User_LED, symbol Device:LED_Small
- added D2: power, symbol Device:LED_Small
- added J1: molex3.0 2x2, symbol Connector_Generic:Conn_02x02_Counter_Clockwise
- added J3: SWD, symbol Connector_Generic:Conn_01x04
- added J6: Encoder1, symbol Connector_Generic:Conn_01x05
- added J7: Encoder2, symbol Connector_Generic:Conn_01x05
- added JP1: Term., symbol Jumper:Jumper_2_Bridged
- added Q1, Q2, Q3, Q4, Q5, Q6: BSS138, Package_TO_SOT_SMD:SOT-23, symbol Transistor_FET:BSS138
- added R1, R10, R12, R13, R14, R15, R16, R17, R20, R24, R26, R5, R6, R7, R8, R9: 10k, symbol Device:R_Small
- added R11: 120, symbol Device:R_Small
- added R18: 3.3k, symbol Device:R_Small
- added R22, R25: 100, symbol Device:R_Small
- added R4: 6k8, symbol Device:R_Small
- added SW1, SW2: SW_Push, symbol Switch:SW_Push
- added U2: MCP2517FD-xSL, Package_SO:SOIC-14_3.9x8.7mm_P1.27mm, symbol Interface_CAN_LIN:MCP2517FD-xSL
- added U3: MCP2562-E-SN, Package_SO:SOIC-8_3.9x4.9mm_P1.27mm, symbol Interface_CAN_LIN:MCP2562-E-SN
- added U?: LSM6DS3, Package_LGA:LGA-14_3x2.5mm_P0.5mm_LayoutBorder3x4y, symbol Sensor_Motion:LSM6DS3
- added Y1: 40MHz, symbol Device:Crystal_GND23_Small
- J2: renamed from J?; value Conn_01x04 -> UART
- gave numbers to parts that had none: 26
Connections:
- net +3V3: now also U1.44 (VREG_VIN), C10.1, C3.1, Q1.1 (G), Q2.1 (G), Q3.1 (G), Q4.1 (G), Q5.1 (G), Q6.1 (G), R1.1, R12.1, R13.1, R14.1, R24.1, R26.1, R4.1, R5.1, R6.1, R7.1, U2.14 (VDD), U3.5 (Vio)
- net GND: now also C1.2, C10.2, C15.2, C17.2, C2.2, C21.2, C23.2, C3.2, D1.1 (K), D2.1 (K), J3.1 (Pin_1), J6.5 (Pin_5), J7.5 (Pin_5), R22.2, R25.2, U2.7 (VSS), U3.2 (VSS), Y1.2, Y1.3
- net GPIO20: now also U1.31 (GPIO20), Q4.2 (S), R12.2; no longer J2.3 (Pin_3)
- net GPIO21: now also U1.32 (GPIO21)
- net SWCLK: now also J3.2 (Pin_2)
- net SWD: now also J3.3 (Pin_3)
- net VBUS: now also C15.1, C17.1, J3.4 (Pin_4), J6.1 (Pin_1), J7.1 (Pin_1), R10.1, R15.1, R16.1, R17.1, R20.1, R8.1, R9.1, U3.3 (VDD)
- net SPI1_RX: now reaches U1.11 (GPIO8)
- net SPI1_RX: now also U2.12 (SDO)
- net SPI1_SCK: now reaches U1.13 (GPIO10)
- net SPI1_SCK: now also U2.10 (SCK)
- net SPI1_TX: now reaches U1.14 (GPIO11)
- net SPI1_TX: now also U2.11 (SDI)
- net GPIO15: now reaches U1.18 (GPIO15)
- net GPIO15: now also Q1.2 (S), R5.2
- net GPIO0: now reaches U1.2 (GPIO0)
- net GPIO0: now also R18.1
- net GPIO16: now reaches U1.27 (GPIO16)
- net GPIO16: now also Q2.2 (S), R6.2
- net GPIO17: now reaches U1.28 (GPIO17)
- net GPIO17: now also Q3.2 (S), R7.2
- net GPIO18: now reaches U1.29 (GPIO18)
- net GPIO18: now also Q5.2 (S), R13.2
- net GPIO1: now reaches U1.3 (GPIO1)
- net GPIO1: now also C21.1, R24.2, SW1.2
- net GPIO19: now reaches U1.30 (GPIO19)
- net GPIO19: now also Q6.2 (S), R14.2
- net GPIO22: now reaches U1.34 (GPIO22)
- net GPIO22: now also J2.3 (Pin_3)
- net GPIO2: now reaches U1.4 (GPIO2)
- net GPIO2: now also C23.1, R26.2, SW2.2
- net STBY: now reaches U1.5 (GPIO3)
- net STBY: now also U3.8 (STBY)
- net SOF: now reaches U1.6 (GPIO4)
- net SOF: now also U2.3 (CLKO/SOF)
- net IRQ: now reaches U1.7 (GPIO5)
- net IRQ: now also U2.4 (~{INT})
- net CSn: now reaches U1.8 (GPIO6)
- net CSn: now also U2.13 (nCS)
- net RUN: no longer names the net of U1.26 (RUN)
- net RUN: now also R1.2
- new net: C1.1, U2.5 (OSC2), Y1.1
- new net: J1.1 (Pin_1), JP1.1 (A), U3.7 (CANH)
- new net: J1.2 (Pin_2), R11.1, U3.6 (CANL)
- new net: D1.2 (A), R18.2
- new net: JP1.2 (B), R11.2
- new net: R22.1, SW1.1
- new net: C2.1, U2.6 (OSC1), Y1.4
- new net: D2.2 (A), R20.2
- new net: R25.1, SW2.1
- new net CANRx: U2.2 (RXCAN), U3.4 (RXD)
- new net CANTx: R4.2, U2.1 (TXCAN), U3.1 (TXD)
- new net Encoder1_A: J6.2 (Pin_2), Q1.3 (D), R8.2
- new net Encoder1_B: J6.3 (Pin_3), Q2.3 (D), R9.2
- new net Encoder1_X: J6.4 (Pin_4), Q3.3 (D), R10.2
- new net Encoder2_A: J7.2 (Pin_2), Q5.3 (D), R16.2
- new net Encoder2_B: J7.3 (Pin_3), Q6.3 (D), R17.2
- new net Encoder2_X: J7.4 (Pin_4), Q4.3 (D), R15.2
- no-connect marks 1 -> 17
Other:
- company: (none) -> POLYU ROBOCON 2020 ~ 2022  by Samson Chau
- title: (none) -> POS CARD
- moved on the sheet: C11, C12, C13, C14, C16, C18, C19, C20, C4, C5, C6, C7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

Commit message: POS_update
Parts:
- removed U?: LSM6DS3, Package_LGA:LGA-14_3x2.5mm_P0.5mm_LayoutBorder3x4y, symbol Sensor_Motion:LSM6DS3
- C1, C10, C11, C12, C13, C14, C15, C16, C17, C18, C19, C2, C21, C3, C4, C5, C6, C7, C8, C9: footprint (none) -> Capacitor_SMD:C_0402_1005Metric
- C20, C22: footprint (none) -> Capacitor_SMD:C_0603_1608Metric
- C23: footprint (none) -> Capacitor_SMD:C_0402_1005Metric_Pad0.74x0.62mm_HandSolder
- D1, D2: footprint (none) -> LED_SMD:LED_0402_1005Metric
- J1: footprint (none) -> Connector_Molex:Molex_Micro-Fit_3.0_43045-0412_2x02_P3.00mm_Vertical
- J2, J3: footprint (none) -> Connector_PinHeader_2.54mm:PinHeader_1x04_P2.54mm_Vertical
- J4: footprint (none) -> Connector_USB:USB_Micro-B_Molex-105017-0001
- J5: footprint (none) -> Connector_PinHeader_2.54mm:PinHeader_1x02_P2.54mm_Vertical
- J6, J7: footprint (none) -> Connector_JST:JST_PH_B5B-PH-K_1x05_P2.00mm_Vertical
- JP1: footprint (none) -> TestPoint:TestPoint_Bridge_Pitch2.0mm_Drill0.7mm
- R1, R10, R11, R12, R13, R14, R15, R16, R17, R18, R19, R2, R20, R21, R22, R23, R24, R25, R26, R3, R4, R5, R6, R7, R8, R9: footprint (none) -> Resistor_SMD:R_0402_1005Metric
- SW1, SW2: footprint (none) -> Button_Switch_SMD:SW_Push_1P1T_NO_6x6mm_H9.5mm
- Y1: value 40MHz -> ASEAIG-40MHZ-C-S-T; footprint (none) -> Crystal:Crystal_SMD_TXC_7M-4Pin_3.2x2.5mm
- Y2: footprint (none) -> Crystal:Crystal_SMD_HC49-SD
