File: solenoid_board/F446RE_sch.kicad_sch (KiCad schematic)
At the start: 30 parts

Commit message: add
Parts:
- removed D6: (no value), symbol Device:D_Schottky
- added D26: LED1, LED_SMD:LED_0805_2012Metric_Pad1.15x1.40mm_HandSolder, symbol Device:LED_Small
- added D27: LED2, LED_SMD:LED_0805_2012Metric_Pad1.15x1.40mm_HandSolder, symbol Device:LED_Small
- added D28: LED3, LED_SMD:LED_0805_2012Metric_Pad1.15x1.40mm_HandSolder, symbol Device:LED_Small
- added R56, R57, R58: 470R, Resistor_SMD:R_0805_2012Metric_Pad1.20x1.40mm_HandSolder, symbol Device:R_Small
- added R59, R60: (no value), symbol Device:R_Small
- added SW11: (no value), symbol Switch:SW_DIP_x04
- C1: value (none) -> 16v100uF; footprint (none) -> Capacitor_SMD:C_Elec_6.3x7.7
- C2: value (none) -> 16v 47uF; footprint (none) -> Capacitor_SMD:C_Elec_6.3x7.7
- C3: value (none) -> 50v 47uF; footprint (none) -> Capacitor_SMD:C_Elec_6.3x7.7
- C4: value (none) -> 16v 100uF; footprint (none) -> Capacitor_SMD:C_Elec_6.3x7.7
- D3: value (none) -> power_led; footprint (none) -> LED_SMD:LED_0805_2012Metric_Pad1.15x1.40mm_HandSolder
- D4, D5: value (none) -> can_led; footprint (none) -> LED_SMD:LED_0805_2012Metric_Pad1.15x1.40mm_HandSolder
- D7: value (none) -> SMBJ24CA; footprint (none) -> Diode_SMD:D_SMB_Handsoldering
- D8: value (none) -> SMBJ9VCA; footprint (none) -> Diode_SMD:D_SMB_Handsoldering
- J11, J15, J3, J7: value (none) -> CAN1; footprint (none) -> Connector_Molex:Molex_Micro-Fit_3.0_43045-0412_2x02_P3.00mm_Vertical
- J12, J16, J4, J8: value (none) -> CAN2; footprint (none) -> Connector_Molex:Molex_Micro-Fit_3.0_43045-0412_2x02_P3.00mm_Vertical
- J19: value (none) -> I2C3; footprint (none) -> Connector_Molex:Molex_Nano-Fit_105309-xx04_1x04_P2.50mm_Vertical
- J20: value (none) -> UART4; footprint (none) -> Connector_Molex:Molex_Nano-Fit_105309-xx04_1x04_P2.50mm_Vertical
- J21: value (none) -> xt60 male; footprint (none) -> PolyuRobotics:XT60PW-M20
- M3, M4: value (none) -> TJA1050_Module; footprint (none) -> PolyuRobotics:TJA1050_CAN_Module
- R3, R4, R5: value (none) -> 10K; footprint (none) -> Resistor_SMD:R_0805_2012Metric_Pad1.20x1.40mm_HandSolder
- R6, R7: value (none) -> 4.7k; footprint (none) -> Resistor_SMD:R_0805_2012Metric_Pad1.20x1.40mm_HandSolder
- U1: value (none) -> NUCLEO-F446RE; footprint (none) -> PolyuRobotics:NUCLEO-F446RE
- U2: value (none) -> MP1584; footprint (none) -> PolyuRobotics:DC-DC-mp1584_module
Connections:
- net +24V: now also C3.1, U2.IN1+ (VIN+), U2.IN2+ (VIN+)
- net +5V: now also SW11.2, SW11.4; no longer M3.1 (VCC), M4.1 (VCC), R4.1, R5.1
- net CAN1+: now also SW11.3
- net CAN1-: now also R60.2
- net CAN2+: now also SW11.1
- net CAN2-: now also R59.2
- net GND: now also D26.1 (K), D27.1 (K), D28.1 (K)
- net PC7: now also R56.1
- net PC8: now also R57.1
- net PC9: now also R58.1
- new net: D27.2 (A), R57.2
- new net: D28.2 (A), R58.2
- new net: D26.2 (A), R56.2
- new net: R59.1, SW11.8
- new net: R60.1, SW11.6
- new net CAN1_VCC: M3.1 (VCC), R4.1, SW11.5
- new net CAN2_VCC: M4.1 (VCC), R5.1, SW11.7
Other:
- note added: "LED and User button"
- moved on the sheet: C3, C4, D3, D7, D8, J19, J20, J21, R3, R6, R7
