File: solenoid_board/24_in_GPIO.kicad_sch (KiCad schematic)
At the start: 64 parts, among them J12 PORT, U11 EL357N

Commit message: solenoid board
Parts:
- D31: footprint (none) -> Diode_SMD:D_1206_3216Metric
- D33, D34, D35, D39, D40, D41, D42: renamed from D?; footprint (none) -> Diode_SMD:D_1206_3216Metric
- J12: footprint TerminalBlock_Phoenix:TerminalBlock_Phoenix_MKDS-3-3-5.08_1x03_P5.08mm_Horizontal -> (none)
- J13, J14, J15, J16, J17, J18, J19: renamed from J?; footprint TerminalBlock_Phoenix:TerminalBlock_Phoenix_MKDS-3-3-5.08_1x03_P5.08mm_Horizontal -> (none)
- gave numbers to parts that had none: 42
Connections:
- net PB0: no longer R74.2, R75.2, R76.2, R89.2, R90.2, R91.2, R92.2
- new net PB7: R92.2
- new net PC0: R75.2
- new net PC1: R74.2
- new net PC14: R91.2
- new net PC15: R90.2
- new net PC2: R76.2
- new net PC3: R89.2

Commit message: test
Parts:
- J12, J13, J14, J15, J16, J17, J18, J19: footprint (none) -> TerminalBlock_Phoenix:TerminalBlock_Phoenix_PT-1,5-3-3.5-H_1x03_P3.50mm_Horizontal
Changed lines of the file:
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@@
     (property "Reference" "J16" (id 0) (at 111.125 30.48 0))
     (property "Value" "PORT" (id 1) (at 111.125 33.02 0))
-    (property "Footprint" "" (id 2) (at 111.125 39.37 0)
+    (property "Footprint" "TerminalBlock_Phoenix:TerminalBlock_Phoenix_PT-1,5-3-3.5-H_1x03_P3.50mm_Horizontal" (id 2) (at 111.125 39.37 0)
       (effects (font (size 1.27 1.27)) hide)
     )
@@
     (property "Reference" "J13" (id 0) (at 24.13 59.69 0))
     (property "Value" "PORT" (id 1) (at 24.13 62.23 0))
-    (property "Footprint" "" (id 2) (at 24.13 68.58 0)
+    (property "Footprint" "TerminalBlock_Phoenix:TerminalBlock_Phoenix_PT-1,5-3-3.5-H_1x03_P3.50mm_Horizontal" (id 2) (at 24.13 68.58 0)
       (effects (font (size 1.27 1.27)) hide)
     )
@@
     (property "Reference" "J12" (id 0) (at 24.13 30.48 0))
     (property "Value" "PORT" (id 1) (at 24.13 33.02 0))
-    (property "Footprint" "" (id 2) (at 24.13 39.37 0)
+    (property "Footprint" "TerminalBlock_Phoenix:TerminalBlock_Phoenix_PT-1,5-3-3.5-H_1x03_P3.50mm_Horizontal" (id 2) (at 24.13 39.37 0)
       (effects (font (size 1.27 1.27)) hide)
     )
@@
     (property "Reference" "J18" (id 0) (at 111.76 87.63 0))
     (property "Value" "PORT" (id 1) (at 111.76 90.17 0))
-    (property "Footprint" "" (id 2) (at 111.76 96.52 0)
+    (property "Footprint" "TerminalBlock_Phoenix:TerminalBlock_Phoenix_PT-1,5-3-3.5-H_1x03_P3.50mm_Horizontal" (id 2) (at 111.76 96.52 0)
       (effects (font (size 1.27 1.27)) hide)
     )
@@
     (property "Reference" "J14" (id 0) (at 24.765 86.995 0))
     (property "Value" "PORT" (id 1) (at 24.765 89.535 0))
-    (property "Footprint" "" (id 2) (at 24.765 95.885 0)
+    (property "Footprint" "TerminalBlock_Phoenix:TerminalBlock_Phoenix_PT-1,5-3-3.5-H_1x03_P3.50mm_Horizontal" (id 2) (at 24.765 95.885 0)
       (effects (font (size 1.27 1.27)) hide)
     )
@@
     (property "Reference" "J17" (id 0) (at 111.125 58.42 0))
     (property "Value" "PORT" (id 1) (at 111.125 60.96 0))
-    (property "Footprint" "" (id 2) (at 111.125 67.31 0)
+    (property "Footprint" "TerminalBlock_Phoenix:TerminalBlock_Phoenix_PT-1,5-3-3.5-H_1x03_P3.50mm_Horizontal" (id 2) (at 111.125 67.31 0)
       (effects (font (size 1.27 1.27)) hide)
     )
@@
     (property "Reference" "J19" (id 0) (at 111.76 116.84 0))
     (property "Value" "PORT" (id 1) (at 111.76 119.38 0))
-    (property "Footprint" "" (id 2) (at 111.76 125.73 0)
+    (property "Footprint" "TerminalBlock_Phoenix:TerminalBlock_Phoenix_PT-1,5-3-3.5-H_1x03_P3.50mm_Horizontal" (id 2) (at 111.76 125.73 0)
       (effects (font (size 1.27 1.27)) hide)
     )
@@
     (property "Reference" "J15" (id 0) (at 24.765 114.935 0))
     (property "Value" "PORT" (id 1) (at 24.765 117.475 0))
-    (property "Footprint" "" (id 2) (at 24.765 123.825 0)
-      (effects (font (size 1.27 1.27)) hide)
-    )
+    (property "Footprint" "TerminalBlock_Phoenix:TerminalBlock_Phoenix_PT-1,5-3-3.5-H_1x03_P3.50mm_Horizontal" (id 2) (at 24.765 123.825 0)
+      (effects (font (size 1.27 1.27)) hide)
+    )

Commit message: test
Connections:
- net PB0: now also R92.2; no longer R64.2
- net PB7: now also R64.2; no longer R92.2
- net PC0: now also R90.2; no longer R75.2
- net PC1: now also R91.2; no longer R74.2
- net PC14: now also R74.2; no longer R91.2
- net PC15: now also R75.2; no longer R90.2
Changed lines of the file:
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@@
     (stroke (width 0) (type default) (color 0 0 0 0))
-  )
-  (global_label "PB7" (shape input) (at 175.26 125.73 0) (fields_autoplaced)
-    (effects (font (size 1.27 1.27)) (justify left))
-    (property "Intersheet References" "${INTERSHEET_REFS}" (id 0) (at 181.4226 125.6506 0)
-      (effects (font (size 1.27 1.27)) (justify left) hide)
-    )
   )
   (global_label "PC3" (shape input) (at 174.625 39.37 0) (fields_autoplaced)
@@
     )
   )
-  (global_label "PC1" (shape input) (at 87.63 68.58 0) (fields_autoplaced)
+  (global_label "PB0" (shape input) (at 175.26 125.73 0) (fields_autoplaced)
     (effects (font (size 1.27 1.27)) (justify left))
-    (property "Intersheet References" "${INTERSHEET_REFS}" (id 0) (at 93.7926 68.5006 0)
+    (property "Intersheet References" "${INTERSHEET_REFS}" (id 0) (at 181.4226 125.6506 0)
       (effects (font (size 1.27 1.27)) (justify left) hide)
     )
   )
-  (global_label "PB0" (shape input) (at 87.63 39.37 0) (fields_autoplaced)
+  (global_label "PC1" (shape input) (at 175.26 96.52 0) (fields_autoplaced)
     (effects (font (size 1.27 1.27)) (justify left))
-    (property "Intersheet References" "${INTERSHEET_REFS}" (id 0) (at 93.7926 39.2906 0)
+    (property "Intersheet References" "${INTERSHEET_REFS}" (id 0) (at 181.4226 96.4406 0)
       (effects (font (size 1.27 1.27)) (justify left) hide)
     )
   )
-  (global_label "PC0" (shape input) (at 88.265 95.885 0) (fields_autoplaced)
+  (global_label "PC0" (shape input) (at 174.625 67.31 0) (fields_autoplaced)
     (effects (font (size 1.27 1.27)) (justify left))
-    (property "Intersheet References" "${INTERSHEET_REFS}" (id 0) (at 94.4276 95.8056 0)
+    (property "Intersheet References" "${INTERSHEET_REFS}" (id 0) (at 180.7876 67.2306 0)
+      (effects (font (size 1.27 1.27)) (justify left) hide)
+    )
+  )
+  (global_label "PC15" (shape input) (at 88.265 95.885 0) (fields_autoplaced)
+    (effects (font (size 1.27 1.27)) (justify left))
+    (property "Intersheet References" "${INTERSHEET_REFS}" (id 0) (at 95.6371 95.8056 0)
+      (effects (font (size 1.27 1.27)) (justify left) hide)
+    )
+  )
+  (global_label "PB7" (shape input) (at 87.63 39.37 0) (fields_autoplaced)
+    (effects (font (size 1.27 1.27)) (justify left))
+    (property "Intersheet References" "${INTERSHEET_REFS}" (id 0) (at 93.7926 39.2906 0)
       (effects (font (size 1.27 1.27)) (justify left) hide)
     )
@@
     )
   )
-  (global_label "PC15" (shape input) (at 174.625 67.31 0) (fields_autoplaced)
+  (global_label "PC14" (shape input) (at 87.63 68.58 0) (fields_autoplaced)
     (effects (font (size 1.27 1.27)) (justify left))
-    (property "Intersheet References" "${INTERSHEET_REFS}" (id 0) (at 181.9971 67.2306 0)
+    (property "Intersheet References" "${INTERSHEET_REFS}" (id 0) (at 95.0021 68.5006 0)
       (effects (font (size 1.27 1.27)) (justify left) hide)
     )
-  )
-  (global_label "PC14" (shape input) (at 175.26 96.52 0) (fields_autoplaced)
-    (effects (font (size 1.27 1.27)) (justify left))
-    (property "Intersheet References" "${INTERSHEET_REFS}" (id 0) (at 182.6321 96.4406 0)
-      (effects (font (size 1.27 1.27)) (justify left) hide)
-    )
