File: solenoid_board/24_out_GPIO.kicad_sch (KiCad schematic)
At the start: 120 parts, among them J1 mx2.54, J10 mx2.54, J13 mx2.54, J14 mx2.54, J17 mx2.54, J18 mx2.54, J2 mx2.54, J5 mx2.54, J6 mx2.54, J9 mx2.54, Q1 IRF540NSTRLPBF, Q10 IRF540NSTRLPBF, Q2 IRF540NSTRLPBF, Q3 IRF540NSTRLPBF, Q4 IRF540NSTRLPBF, Q5 IRF540NSTRLPBF, Q6 IRF540NSTRLPBF, Q7 IRF540NSTRLPBF, Q8 IRF540NSTRLPBF, Q9 IRF540NSTRLPBF, SW1 SW_Push, SW10 SW_Push, SW2 SW_Push, SW3 SW_Push, SW4 SW_Push, SW5 SW_Push, SW6 SW_Push, SW7 SW_Push, SW8 SW_Push, SW9 SW_Push, U10 4N35, U11 4N35, U12 4N35, U3 4N35, U4 4N35, U5 4N35, U6 4N35, U7 4N35, U8 4N35, U9 4N35

Commit message: add
Parts:
- removed D10, D17, D23: indictor, symbol Device:LED_Small
- removed D14, D20, D26: 1N4001, Diode_THT:D_DO-41_SOD81_P10.16mm_Horizontal, symbol Diode:1N4001
- added C15, C16, C17, C18, C19, C20, C21, C22, C23, C24: 100nF, Capacitor_SMD:C_0805_2012Metric_Pad1.18x1.45mm_HandSolder, symbol Device:C_Small
- added D10, D17, D23: 1N4001, Diode_THT:D_DO-41_SOD81_P10.16mm_Horizontal, symbol Diode:1N4001
- added D14, D20, D6: indictor, LED_SMD:LED_0805_2012Metric_Pad1.15x1.40mm_HandSolder, symbol Device:LED_Small
- C10, C11, C12, C13, C14, C5, C6, C7, C8, C9: footprint (none) -> Capacitor_SMD:C_0805_2012Metric_Pad1.18x1.45mm_HandSolder
- D1, D15, D16, D2, D21, D22, D9: footprint (none) -> LED_SMD:LED_0805_2012Metric_Pad1.15x1.40mm_HandSolder
- J1, J10, J13, J14, J17, J18, J2, J5, J6, J9: footprint (none) -> Connector_PinHeader_2.54mm:PinHeader_1x02_P2.54mm_Vertical
- R1, R10, R11, R12, R13, R14, R15, R16, R17, R18, R19, R2, R20, R21, R22, R23, R24, R25, R26, R27, R28, R29, R30, R31, R32, R33, R34, R35, R36, R37, R38, R39, R40, R41, R42, R43, R44, R45, R46, R47, R48, R49, R50, R51, R52, R53, R54, R55, R8, R9: footprint (none) -> Resistor_SMD:R_0805_2012Metric_Pad1.20x1.40mm_HandSolder
- SW1, SW10, SW2, SW3, SW4, SW5, SW6, SW7, SW8, SW9: footprint (none) -> Button_Switch_SMD:SW_SPST_TL3305A
Connections:
- net GND: now also C16.2, C17.2, C18.2, C22.2, C23.2, C24.2; no longer C13.2, C14.2, C6.2, C7.2, C8.2, C9.2
- net GNDPWR: now also D14.1 (K), D20.1 (K), D6.1 (K)
- net VCC: now also D10.1 (K), D17.1 (K), D23.1 (K)
- net at J6.2 (Pin_2), Q4.2: now also D13.2 (A)
- net at J10.2 (Pin_2), Q6.2: now also D18.2 (A); no longer D19.2 (A)
- net PC6: now reaches R29.1, SW5.2
- net PC6: now also C13.2
- net at R29.2, U7.1: now also C16.1; no longer C9.1
- net at R42.2, SW9.1: now also C20.1
- net at R43.2, SW10.1: now also C21.1
- net PC15: now reaches R46.1, SW10.2
- net PC15: now also C21.2
- net at R28.2, SW7.1: now also C15.1
- net at R31.2, U9.1: now also C18.1; no longer C11.1
- net at J9.2 (Pin_2), Q5.2: now also D17.2 (A); no longer D18.2 (A)
- net at R30.2, U8.1: now also C17.1; no longer C10.1
- net at R49.1: now also D22.2 (A)
- net PC3: now reaches R11.1, SW2.2
- net PC3: now also C7.2
- net at R11.2, U4.1: now also C10.1; no longer C6.1
- net at R48.1: now also D21.2 (A); no longer D22.2 (A)
- net at J2.2 (Pin_2), Q2.2: now also D10.2 (A); no longer D12.2 (A)
- net at R47.1: now also D20.2 (A); no longer D21.2 (A)
- net at D9.2 (A): now also R17.1; no longer R16.1
- net at J13.2 (Pin_2), Q7.2: now also D19.2 (A)
- net at R45.2, U11.1: now also C23.1; no longer C13.1
- net PC5: now reaches R13.1, SW4.2
- net PC5: now also C9.2
- net at R13.2, U6.1: now also C12.1; no longer C8.1
- net at R26.2, SW5.1: now also C13.1
- net at J18.2 (Pin_2), Q10.2: now also D25.2 (A)
- net at R34.1: now also D16.2 (A)
- net at R8.2, SW3.1: now also C8.1
- net at R46.2, U12.1: now also C24.1; no longer C14.1
- net at R33.1: now also D15.2 (A); no longer D16.2 (A)
- net at R1.2, SW1.1: now also C6.1
- net at R2.2, SW2.1: now also C7.1
- net at R32.1: now also D14.2 (A); no longer D15.2 (A)
- net at J14.2 (Pin_2), Q8.2: now also D23.2 (A); no longer D24.2 (A)
- net at R44.2, U10.1: now also C22.1; no longer C12.1
- net at J5.2 (Pin_2), Q3.2: now also D12.2 (A); no longer D13.2 (A)
- net PC2: now reaches R10.1, SW1.2
- net PC2: now also C6.2
- net at R12.2, U5.1: now also C11.1; no longer C7.1
- net PC4: now reaches R12.1, SW3.2
- net PC4: now also C8.2
- net at J17.2 (Pin_2), Q9.2: now also D24.2 (A); no longer D25.2 (A)
- net at R27.2, SW6.1: now also C14.1
- net PC11: now reaches R31.1, SW7.2
- net PC11: now also C15.2
- net at R41.2, SW8.1: now also C19.1
- net PC12: now reaches R44.1, SW8.2
- net PC12: now also C19.2
- net at R9.2, SW4.1: now also C9.1
- net PC10: now reaches R30.1, SW6.2
- net PC10: now also C14.2
- net PC14: now reaches R45.1, SW9.2
- net PC14: now also C20.2
- new net: D6.2 (A), R16.1
Other:
- moved on the sheet: R1, SW1

Commit message: solenoid board
Parts:
- removed C11, C12, C13, C14, C15, C16, C17, C18, C19, C20, C21, C22, C23, C24: 100nF, Capacitor_SMD:C_0805_2012Metric_Pad1.18x1.45mm_HandSolder, symbol Device:C_Small
- removed D13, D17, D18, D23, D24, D25: 1N4001, Diode_THT:D_DO-41_SOD81_P10.16mm_Horizontal, symbol Diode:1N4001
- removed D15, D16, D2, D20, D21, D22, D9: indictor, LED_SMD:LED_0805_2012Metric_Pad1.15x1.40mm_HandSolder, symbol Device:LED_Small
- removed J13, J14, J17, J18, J2: mx2.54, Connector_PinHeader_2.54mm:PinHeader_1x02_P2.54mm_Vertical, symbol Connector_Generic:Conn_01x02
- removed Q1, Q10, Q2, Q3, Q4, Q5, Q6, Q7, Q8, Q9: IRF540NSTRLPBF, PolyuRobotics:IRF540NSTRLPBF, symbol PolyuRobotics:IRF540NSTRLPBF
- removed U10, U11, U12, U3, U4, U5, U6, U7, U8, U9: 4N35, Package_DIP:DIP-6_W7.62mm, symbol Isolator:4N35
- added C1, C2, C3, C4: 100nF, Capacitor_SMD:C_0805_2012Metric_Pad1.18x1.45mm_HandSolder, symbol Device:C_Small
- added D13, D15, D16, D2, D22, D24, D25, D3, D5, D7: SS24, Diode_SMD:D_SMB, symbol Diode:1N5822
- added D17, D18, D23, D26, D27, D4, D8: indictor, LED_SMD:LED_0805_2012Metric_Pad1.15x1.40mm_HandSolder, symbol Device:LED_Small
- added D20, D21, D28, D29, D30, D9: 1N4001, Diode_THT:D_DO-41_SOD81_P10.16mm_Horizontal, symbol Diode:1N4001
- added J11, J3, J4, J7, J8: mx2.54, Connector_PinHeader_2.54mm:PinHeader_1x02_P2.54mm_Vertical, symbol Connector_Generic:Conn_01x02
- added Q1: AOD4184A, PolyuRobotics:DPAK228P994X240-4N, symbol PolyuRobotics:AOD4184A
- added Q10, Q2, Q3, Q4, Q5, Q6, Q7, Q8, Q9: ~, PolyuRobotics:DPAK228P994X240-4N, symbol PolyuRobotics:AOD4184A
- added R3, R4: 1k, Resistor_SMD:R_0805_2012Metric_Pad1.20x1.40mm_HandSolder, symbol Device:R_Small
- added R5, R7: 470R, Resistor_SMD:R_0805_2012Metric_Pad1.20x1.40mm_HandSolder, symbol Device:R_Small
- added R56, R57: 100R, Resistor_SMD:R_0805_2012Metric_Pad1.20x1.40mm_HandSolder, symbol Device:R_Small
- added R58, R59, R60: 10k, Resistor_SMD:R_0805_2012Metric_Pad1.20x1.40mm_HandSolder, symbol Device:R_Small
- added R6: 10K, Resistor_SMD:R_0805_2012Metric_Pad1.20x1.40mm_HandSolder, symbol Device:R_Small
- added U1: EL357N, PolyuRobotics:EL357N, symbol PolyuRobotics:EL357N
- added U10, U2, U3, U4, U5, U6, U7, U8, U9: ~, PolyuRobotics:EL357N, symbol PolyuRobotics:EL357N
- R11, R12, R31: value 470R -> ~
- R13: value 470R -> 3.3K
- R17: value 3.3K -> 100R
- R21: value 100R -> 10k
- R25: value 10k -> 1k
- R28, R8: value 1k -> 470R
- R32, R33, R49: value 3.3K -> ~
- R35, R36, R52: value 100R -> 3.3K
- R38, R39, R55: value 10k -> 100R
- R41, R42: value 1k -> 10k
- R44, R45: value 470R -> 1k
- R47, R48: value 3.3K -> 470R
- R50, R51: value 100R -> ~
- R53, R54: value 10k -> 3.3K
- R9: value 1k -> ~
Connections:
- net +5V: now also R25.1, R44.1, R45.1, R3.1, R4.1; no longer R28.1, R41.1, R42.1, R8.1, R9.1
- net GND: now also R11.1, R12.1, R31.1, R32.1, R33.1, R49.1, R50.1, R51.1, R9.1, R6.1, U1.2, U10.2, U2.2, U3.2, U4.2, U5.2, U6.2, U7.2, U8.2, U9.2; no longer C10.2, C5.2
- net GNDPWR: now also R21.1, R41.1, R42.1, D17.1 (K), D18.1 (K), D23.1 (K), D26.1 (K), D27.1 (K), D4.1 (K), D8.1 (K), Q1.3, Q10.3, Q2.3, Q3.3, Q4.3, Q5.3, Q6.3, Q7.3, Q8.3, Q9.3, R58.1, R59.1, R60.1; no longer R25.1, R38.1, R39.1, R53.1, R54.1, R55.1
- net PC10: now also C8.2, R46.1, SW8.2; no longer R30.1, SW6.2
- net PC11: now also C5.2, R29.1, SW6.2; no longer R31.1, SW7.2
- net PC12: now also C9.2, R47.1, SW9.2; no longer R44.1, SW8.2
- net VCC: now also D13.1 (K), D15.1 (K), D16.1 (K), D2.1 (K), D22.1 (K), D24.1 (K), D25.1 (K), D3.1 (K), D5.1 (K), D7.1 (K), U1.4, U10.4, U2.4, U3.4, U4.4, U5.4, U6.4, U7.4, U8.4, U9.4; no longer D10.1 (K), D11.1 (K), D12.1 (K), D19.1 (K), J1.1 (Pin_1), J10.1 (Pin_1), J5.1 (Pin_1), J6.1 (Pin_1), J9.1 (Pin_1)
- net at R18.2, R22.2: now also Q1.1
- net at D19.2 (A): now also J6.2 (Pin_2), Q5.4
- net at SW9.1: now also C9.1, R44.2; no longer R42.2
- net at SW6.1: now also C5.1, R26.2; no longer R27.2
- net at R45.2: now also C10.1, SW10.1
- net at R48.2: now also R51.2, U10.1; no longer R51.1
- net at R12.2: now also R8.2, U4.1
- net at R16.2, R20.1: now also U4.3
- net at D11.2 (A), J1.2 (Pin_2): now also Q1.4
- net at R2.2, SW2.1: now also C1.1; no longer C7.1
- net at R20.2, R24.2: now also Q4.1
- net at D12.2 (A), J5.2 (Pin_2): now also Q4.4
- net at D10.2 (A): now also J4.2 (Pin_2), Q3.4
- net PA4: now reaches R48.1
- net PA4: now also C10.2, SW10.2
- net at R15.2, R19.1: now also U3.3
- net at R19.2, R23.2: now also Q3.1
- net at R11.2: now also R7.2, U3.1; no longer C10.1
- net at R15.1: now also D6.2 (A)
- net at R28.2: now also R31.2, U5.1; no longer SW7.1
- net at SW8.1: now also C8.1, R43.2; no longer R41.2
- net at R29.2: now also R32.2, U6.1
- net at R35.1: now also D17.2 (A); no longer R32.2
- net at R46.2: now also R49.2, U8.1
- net at R37.2, R40.2: now also Q5.1
- net at J10.2 (Pin_2): now also D29.2 (A), Q9.4
- net at D14.2 (A): now also R34.1; no longer R32.1
- net at R35.2: now also R38.1, U6.3; no longer R38.2
- net at R30.2: now also R33.2, U7.1
- net at R36.1: now also D18.2 (A); no longer R33.2
- net at R47.2: now also R50.2, U9.1; no longer R50.1
- net at R53.2: now also R56.1, U9.3; no longer R50.2
- net at R21.2: now also R17.2, Q2.1; no longer R25.2
- net at R36.2: now also R39.1, U7.3; no longer R39.2
- net at R17.1: now also R13.2, U2.3
- net at R52.1: now also D23.2 (A); no longer R49.2
- net at R52.2: now also R55.1, U8.3; no longer R55.2
- net at J9.2 (Pin_2): now also D28.2 (A), Q8.4
- net at R34.2, R37.1: now also U5.3
- net at R14.2, R18.1: now also U1.3
- net at SW5.1: now also R25.2, C4.1; no longer R26.2
- net at R54.2: now also R57.1, U10.3; no longer R51.2
- net at R16.1: now also D8.2 (A); no longer D6.2 (A)
- net at R10.2: now also R6.2, U1.1; no longer C5.1
- removed net PC14: R45.1, SW9.2
- removed net PC15: R46.1, SW10.2
- net PC2 renamed PB1
- removed net PC3: C7.2, R11.1, SW2.2
- removed net PC4: C8.2, R12.1, SW3.2
- removed net PC5: C9.2, R13.1, SW4.2
- net PC6 renamed PA6
- net PA6: now also R28.1, C4.2; no longer R29.1
- new net: D22.2 (A), D28.1 (K), J9.1 (Pin_1)
- new net: C3.1, R4.2, SW4.1
- new net: D11.1 (K), D2.2 (A), J1.1 (Pin_1)
- new net: D4.2 (A), R13.1
- new net: D25.2 (A), D30.1 (K), J11.1 (Pin_1)
- new net: D30.2 (A), J11.2 (Pin_2), Q10.4
- new net: D15.2 (A), D20.1 (K), J7.1 (Pin_1)
- new net: D3.2 (A), D9.1 (K), J3.1 (Pin_1)
- new net: Q8.1, R55.2, R58.2
- new net: Q6.1, R38.2, R41.2
- new net: D13.2 (A), D19.1 (K), J6.1 (Pin_1)
- new net: Q9.1, R56.2, R59.2
- new net: D20.2 (A), J7.2 (Pin_2), Q6.4
- new net: D27.2 (A), R54.1
- new net: C2.1, R3.2, SW3.1
- new net: D10.1 (K), D5.2 (A), J4.1 (Pin_1)
- new net: Q10.1, R57.2, R60.2
- new net: D16.2 (A), D21.1 (K), J8.1 (Pin_1)
- new net: D21.2 (A), J8.2 (Pin_2), Q7.4
- new net: D26.2 (A), R53.1
- new net: D12.1 (K), D7.2 (A), J5.1 (Pin_1)
- new net: C7.1, R27.2, SW7.1
- new net: D9.2 (A), J3.2 (Pin_2), Q2.4
- new net: D24.2 (A), D29.1 (K), J10.1 (Pin_1)
- new net: Q7.1, R39.2, R42.2
- new net: R5.2, R9.2, U2.1
- new net PA5: C7.2, R30.1, SW7.2
- new net PA7: C3.2, R8.1, SW4.2
- new net PA9: C2.2, R7.1, SW3.2
- new net PB2: C1.2, R5.1, SW2.2
- no-connect marks 10 -> 0
Other:
- moved on the sheet: D1, J1, R10, R14, R18, R22

Commit message: solenoid board
Parts:
- removed J1, J10, J11, J3, J4, J5, J6, J7, J8, J9: mx2.54, Connector_PinHeader_2.54mm:PinHeader_1x02_P2.54mm_Vertical, symbol Connector_Generic:Conn_01x02
- added J1, J10, J11, J3, J4, J5, J6, J7, J8, J9: (no value), symbol Connector:Screw_Terminal_01x02
- Q10, Q2, Q3, Q4, Q5, Q6, Q7, Q8, Q9: value ~ -> AOD4184A
- R11, R12, R31, R32, R33, R49, R50, R51, R9: value ~ -> 10K
- U10, U2, U3, U4, U5, U6, U7, U8, U9: value ~ -> EL357N
Connections:
- net at D22.2 (A), D28.1 (K): now also J9.1 (Pin_1)
- net at D11.1 (K), D2.2 (A): now also J1.1 (Pin_1)
- net at D11.2 (A), Q1.4: now also J1.2 (Pin_2)
- net at D25.2 (A), D30.1 (K): now also J11.1 (Pin_1)
- net at D30.2 (A), Q10.4: now also J11.2 (Pin_2)
- net at D19.2 (A), Q5.4: now also J6.2 (Pin_2)
- net at D15.2 (A), D20.1 (K): now also J7.1 (Pin_1)
- net at D3.2 (A), D9.1 (K): now also J3.1 (Pin_1)
- net at D13.2 (A), D19.1 (K): now also J6.1 (Pin_1)
- net at D29.2 (A), Q9.4: now also J10.2 (Pin_2)
- net at D20.2 (A), Q6.4: now also J7.2 (Pin_2)
- net at D10.1 (K), D5.2 (A): now also J4.1 (Pin_1)
- net at D12.2 (A), Q4.4: now also J5.2 (Pin_2)
- net at D16.2 (A), D21.1 (K): now also J8.1 (Pin_1)
- net at D21.2 (A), Q7.4: now also J8.2 (Pin_2)
- net at D28.2 (A), Q8.4: now also J9.2 (Pin_2)
- net at D12.1 (K), D7.2 (A): now also J5.1 (Pin_1)
- net at D10.2 (A), Q3.4: now also J4.2 (Pin_2)
- net at D9.2 (A), Q2.4: now also J3.2 (Pin_2)
- net at D24.2 (A), D29.1 (K): now also J10.1 (Pin_1)

Commit message: test
Parts:
- J1, J10, J11, J3, J4, J5, J6, J7, J8, J9: value (none) -> output; footprint (none) -> TerminalBlock_Phoenix:TerminalBlock_Phoenix_PT-1,5-2-5.0-H_1x02_P5.00mm_Horizontal
Connections:
- net VCC renamed +24V

Commit message: test
Connections:
- net PA5: now also C5.2, R29.1, SW6.2; no longer C7.2, R30.1, SW7.2
- net PA7: now also C6.2, R10.1, SW1.2; no longer C3.2, R8.1, SW4.2
- net PA9: now also C1.2, R5.1, SW2.2; no longer C2.2, R7.1, SW3.2
- net PB1: now also C3.2, R8.1, SW4.2; no longer C6.2, R10.1, SW1.2
- net PB2: now also C2.2, R7.1, SW3.2; no longer C1.2, R5.1, SW2.2
- net PC11: now also C7.2, R30.1, SW7.2; no longer C5.2, R29.1, SW6.2
Changed lines of the file:
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@@
     )
   )
-  (global_label "PA9" (shape input) (at 40.64 127 180) (fields_autoplaced)
+  (global_label "PA9" (shape input) (at 38.735 83.82 180) (fields_autoplaced)
     (effects (font (size 1.27 1.27)) (justify right))
-    (property "Intersheet References" "${INTERSHEET_REFS}" (id 0) (at 34.6588 126.9206 0)
-      (effects (font (size 1.27 1.27)) (justify right) hide)
-    )
-  )
-  (global_label "PA5" (shape input) (at 128.905 88.9 180) (fields_autoplaced)
-    (effects (font (size 1.27 1.27)) (justify right))
-    (property "Intersheet References" "${INTERSHEET_REFS}" (id 0) (at 122.9238 88.8206 0)
-      (effects (font (size 1.27 1.27)) (justify right) hide)
-    )
-  )
-  (global_label "PB1" (shape input) (at 34.925 43.815 180) (fields_autoplaced)
-    (effects (font (size 1.27 1.27)) (justify right))
-    (property "Intersheet References" "${INTERSHEET_REFS}" (id 0) (at 28.7624 43.7356 0)
+    (property "Intersheet References" "${INTERSHEET_REFS}" (id 0) (at 32.7538 83.7406 0)
       (effects (font (size 1.27 1.27)) (justify right) hide)
     )
@@
     )
   )
+  (global_label "PB1" (shape input) (at 41.91 168.91 180) (fields_autoplaced)
+    (effects (font (size 1.27 1.27)) (justify right))
+    (property "Intersheet References" "${INTERSHEET_REFS}" (id 0) (at 35.7474 168.8306 0)
+      (effects (font (size 1.27 1.27)) (justify right) hide)
+    )
+  )
   (global_label "PC12" (shape input) (at 212.725 91.44 180) (fields_autoplaced)
     (effects (font (size 1.27 1.27)) (justify right))
@@
     )
   )
-  (global_label "PB2" (shape input) (at 38.735 83.82 180) (fields_autoplaced)
+  (global_label "PC11" (shape input) (at 128.905 88.9 180) (fields_autoplaced)
     (effects (font (size 1.27 1.27)) (justify right))
-    (property "Intersheet References" "${INTERSHEET_REFS}" (id 0) (at 32.5724 83.7406 0)
+    (property "Intersheet References" "${INTERSHEET_REFS}" (id 0) (at 121.5329 88.8206 0)
       (effects (font (size 1.27 1.27)) (justify right) hide)
     )
@@
     )
   )
-  (global_label "PC11" (shape input) (at 128.27 132.715 180) (fields_autoplaced)
+  (global_label "PA7" (shape input) (at 34.925 43.815 180) (fields_autoplaced)
     (effects (font (size 1.27 1.27)) (justify right))
-    (property "Intersheet References" "${INTERSHEET_REFS}" (id 0) (at 120.8979 132.6356 0)
+    (property "Intersheet References" "${INTERSHEET_REFS}" (id 0) (at 28.9438 43.7356 0)
       (effects (font (size 1.27 1.27)) (justify right) hide)
     )
   )
-  (global_label "PA7" (shape input) (at 41.91 168.91 180) (fields_autoplaced)
+  (global_label "PA5" (shape input) (at 128.27 132.715 180) (fields_autoplaced)
     (effects (font (size 1.27 1.27)) (justify right))
-    (property "Intersheet References" "${INTERSHEET_REFS}" (id 0) (at 35.9288 168.8306 0)
+    (property "Intersheet References" "${INTERSHEET_REFS}" (id 0) (at 122.2888 132.6356 0)
+      (effects (font (size 1.27 1.27)) (justify right) hide)
+    )
+  )
+  (global_label "PB2" (shape input) (at 40.64 127 180) (fields_autoplaced)
+    (effects (font (size 1.27 1.27)) (justify right))
+    (property "Intersheet References" "${INTERSHEET_REFS}" (id 0) (at 34.4774 126.9206 0)
       (effects (font (size 1.27 1.27)) (justify right) hide)
     )
@@
   (symbol (lib_id "power:+24V") (at 245.11 120.015 0) (unit 1)
     (in_bom yes) (on_board yes) (fields_autoplaced)
-    (property "Reference" "#PWR?" (id 0) (at 245.11 123.825 0)
+    (property "Reference" "#PWR0145" (id 0) (at 245.11 123.825 0)
       (effects (font (size 1.27 1.27)) hide)
     )
@@
   (symbol (lib_id "power:+24V") (at 243.84 30.48 0) (unit 1)
     (in_bom yes) (on_board yes) (fields_autoplaced)
-    (property "Reference" "#PWR?" (id 0) (at 243.84 34.29 0)
+    (property "Reference" "#PWR0147" (id 0) (at 243.84 34.29 0)
       (effects (font (size 1.27 1.27)) hide)
     )
@@
   (symbol (lib_id "power:+24V") (at 161.29 70.485 0) (unit 1)
     (in_bom yes) (on_board yes) (fields_autoplaced)
-    (property "Reference" "#PWR?" (id 0) (at 161.29 74.295 0)
+    (property "Reference" "#PWR0107" (id 0) (at 161.29 74.295 0)
       (effects (font (size 1.27 1.27)) hide)
     )
@@
   (symbol (lib_id "power:+24V") (at 67.31 25.4 0) (unit 1)
     (in_bom yes) (on_board yes) (fields_autoplaced)
-    (property "Reference" "#PWR?" (id 0) (at 67.31 29.21 0)
+    (property "Reference" "#PWR0115" (id 0) (at 67.31 29.21 0)
       (effects (font (size 1.27 1.27)) hide)
     )
@@
   (symbol (lib_id "power:+24V") (at 73.025 108.585 0) (unit 1)
     (in_bom yes) (on_board yes) (fields_autoplaced)
-    (property "Reference" "#PWR?" (id 0) (at 73.025 112.395 0)
+    (property "Reference" "#PWR0129" (id 0) (at 73.025 112.395 0)
       (effects (font (size 1.27 1.27)) hide)
     )
@@
   (symbol (lib_id "power:+24V") (at 245.11 73.025 0) (unit 1)
     (in_bom yes) (on_board yes) (fields_autoplaced)
-    (property "Reference" "#PWR?" (id 0) (at 245.11 76.835 0)
+    (property "Reference" "#PWR0141" (id 0) (at 245.11 76.835 0)
       (effects (font (size 1.27 1.27)) hide)
     )
@@
   (symbol (lib_id "power:+24V") (at 71.12 65.405 0) (unit 1)
     (in_bom yes) (on_board yes) (fields_autoplaced)
-    (property "Reference" "#PWR?" (id 0) (at 71.12 69.215 0)
+    (property "Reference" "#PWR0139" (id 0) (at 71.12 69.215 0)
       (effects (font (size 1.27 1.27)) hide)
     )
@@
   (symbol (lib_id "power:+24V") (at 74.295 150.495 0) (unit 1)
     (in_bom yes) (on_board yes) (fields_autoplaced)
-    (property "Reference" "#PWR?" (id 0) (at 74.295 154.305 0)
+    (property "Reference" "#PWR0122" (id 0) (at 74.295 154.305 0)
       (effects (font (size 1.27 1.27)) hide)
     )
@@
   (symbol (lib_id "power:+24V") (at 160.02 28.575 0) (unit 1)
     (in_bom yes) (on_board yes) (fields_autoplaced)
-    (property "Reference" "#PWR?" (id 0) (at 160.02 32.385 0)
+    (property "Reference" "#PWR0106" (id 0) (at 160.02 32.385 0)
       (effects (font (size 1.27 1.27)) hide)
     )
@@
   (symbol (lib_id "power:+24V") (at 160.655 114.3 0) (unit 1)
     (in_bom yes) (on_board yes) (fields_autoplaced)
-    (property "Reference" "#PWR?" (id 0) (at 160.655 118.11 0)
-      (effects (font (size 1.27 1.27)) hide)
-    )
+    (property "Reference" "#PWR0110" (id 0) (at 160.655 118.11 0)
+      (effects (font (size 1.27 1.27)) hide)
+    )
