File: solenoid_board/solenoid_board.kicad_sch (KiCad schematic)
At the start: 0 parts

Commit message: solenoid board
Parts:
- added J2: Conn_02x13_Odd_Even, Connector_IDC:IDC-Header_2x13_P2.54mm_Vertical, symbol Connector_Generic:Conn_02x13_Odd_Even
Connections:
- new net +5V: J2.13 (Pin_13), J2.14 (Pin_14)
- new net GND: J2.10 (Pin_10), J2.8 (Pin_8)
- new net PA15: J2.12 (Pin_12)
- new net PA4: J2.21 (Pin_21)
- new net PA5: J2.11 (Pin_11)
- new net PA6: J2.9 (Pin_9)
- new net PA7: J2.7 (Pin_7)
- new net PA8: J2.4 (Pin_4)
- new net PA9: J2.5 (Pin_5)
- new net PB0: J2.23 (Pin_23)
- new net PB1: J2.1 (Pin_1)
- new net PB2: J2.3 (Pin_3)
- new net PB3: J2.2 (Pin_2)
- new net PB4: J2.6 (Pin_6)
- new net PB7: J2.16 (Pin_16)
- new net PC0: J2.26 (Pin_26)
- new net PC1: J2.25 (Pin_25)
- new net PC10: J2.17 (Pin_17)
- new net PC11: J2.15 (Pin_15)
- new net PC12: J2.19 (Pin_19)
- new net PC14: J2.18 (Pin_18)
- new net PC15: J2.20 (Pin_20)
- new net PC2: J2.22 (Pin_22)
- new net PC3: J2.24 (Pin_24)
Other:
- removed sheet MCU
- sheet 24_in_GPIO: file untitled.kicad_sch -> 24_in_GPIO.kicad_sch
- note added: "Extension plug"

Commit message: test
Parts:
- added J20: 5V in, Connector_BarrelJack:BarrelJack_GCT_DCJ200-10-A_Horizontal, symbol Connector:Barrel_Jack_MountingPin
- added J21: XT60-M, PolyuRobotics:XT60PW-M20, symbol Connector_Generic:Conn_01x02
Connections:
- net +5V: now also J20.1
- net GND: now also J20.2
- new net +24V: J21.1 (Pin_1)
- new net GNDPWR: J21.2 (Pin_2)

Commit message: test
Parts:
- removed J20: 5V in, Connector_BarrelJack:BarrelJack_GCT_DCJ200-10-A_Horizontal, symbol Connector:Barrel_Jack_MountingPin
- J21: footprint PolyuRobotics:XT60PW-M20 -> (none)
Connections:
- net +24V: now also J21.2 (Pin_2); no longer J21.1 (Pin_1)
- net GNDPWR: now also J21.1 (Pin_1); no longer J21.2 (Pin_2)
Other:
- moved on the sheet: J21
Changed lines of the file:
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@@
     )
-  )
-  (symbol (lib_id "Connector:Barrel_Jack_MountingPin") (at 130.175 106.68 0) (unit 1)
-    (in_bom yes) (on_board yes) (fields_autoplaced)
-    (property "Reference" "J20" (id 0) (at 130.175 97.155 0))
-    (property "Value" "5V in" (id 1) (at 130.175 99.695 0))
-    (property "Footprint" "Connector_BarrelJack:BarrelJack_GCT_DCJ200-10-A_Horizontal" (id 2) (at 131.445 107.696 0)
-      (effects (font (size 1.27 1.27)) hide)
-    )
-    (property "Datasheet" "~" (id 3) (at 131.445 107.696 0)
-      (effects (font (size 1.27 1.27)) hide)
-    )
-    (pin "1")
-    (pin "2")
-    (pin "MP")
   )
   (symbol (lib_id "power:GNDPWR") (at 125.73 84.455 0) (unit 1)
@@
     )
     (property "Datasheet" "" (id 3) (at 125.73 81.915 0)
-      (effects (font (size 1.27 1.27)) hide)
-    )
-    (pin "1")
-  )
-  (symbol (lib_id "power:GND") (at 137.795 109.22 0) (unit 1)
-    (in_bom yes) (on_board yes) (fields_autoplaced)
-    (property "Reference" "#PWR0187" (id 0) (at 137.795 115.57 0)
-      (effects (font (size 1.27 1.27)) hide)
-    )
-    (property "Value" "GND" (id 1) (at 137.795 113.665 0))
-    (property "Footprint" "" (id 2) (at 137.795 109.22 0)
-      (effects (font (size 1.27 1.27)) hide)
-    )
-    (property "Datasheet" "" (id 3) (at 137.795 109.22 0)
       (effects (font (size 1.27 1.27)) hide)
     )
@@
     (pin "9")
   )
-  (symbol (lib_id "Connector_Generic:Conn_01x02") (at 130.81 81.915 0) (unit 1)
+  (symbol (lib_id "Connector_Generic:Conn_01x02") (at 120.65 84.455 180) (unit 1)
     (in_bom yes) (on_board yes) (fields_autoplaced)
-    (property "Reference" "J21" (id 0) (at 133.985 81.9149 0)
-      (effects (font (size 1.27 1.27)) (justify left))
-    )
-    (property "Value" "XT60-M" (id 1) (at 133.985 84.4549 0)
-      (effects (font (size 1.27 1.27)) (justify left))
-    )
-    (property "Footprint" "PolyuRobotics:XT60PW-M20" (id 2) (at 130.81 81.915 0)
-      (effects (font (size 1.27 1.27)) hide)
-    )
-    (property "Datasheet" "~" (id 3) (at 130.81 81.915 0)
+    (property "Reference" "J21" (id 0) (at 120.65 74.93 0))
+    (property "Value" "XT60-M" (id 1) (at 120.65 77.47 0))
+    (property "Footprint" "" (id 2) (at 120.65 84.455 0)
+      (effects (font (size 1.27 1.27)) hide)
+    )
+    (property "Datasheet" "~" (id 3) (at 120.65 84.455 0)
       (effects (font (size 1.27 1.27)) hide)
     )
     (pin "1")
     (pin "2")
-  )
-  (symbol (lib_id "power:+5V") (at 137.795 104.14 0) (unit 1)
-    (in_bom yes) (on_board yes) (fields_autoplaced)
-    (property "Reference" "#PWR0189" (id 0) (at 137.795 107.95 0)
-      (effects (font (size 1.27 1.27)) hide)
-    )
-    (property "Value" "+5V" (id 1) (at 137.795 98.425 0))
-    (property "Footprint" "" (id 2) (at 137.795 104.14 0)
-      (effects (font (size 1.27 1.27)) hide)
-    )
-    (property "Datasheet" "" (id 3) (at 137.795 104.14 0)
-      (effects (font (size 1.27 1.27)) hide)
-    )
-    (pin "1")
   )
   (sheet (at 107.315 24.765) (size 34.29 33.02) (fields_autoplaced)
@@
       (reference "#PWR0105") (unit 1) (value "+5V") (footprint "")
     )
+    (path "/dd00c030-9b8d-4d40-8d8f-4fd3b5efd5ca/e80b2b35-b6c0-4d41-bba7-6bc814b6444d"
+      (reference "#PWR0106") (unit 1) (value "+24V") (footprint "")
+    )
+    (path "/dd00c030-9b8d-4d40-8d8f-4fd3b5efd5ca/4b355d96-1c0b-4ff4-91f0-4fd5a7144671"
+      (reference "#PWR0107") (unit 1) (value "+24V") (footprint "")
+    )
     (path "/dd00c030-9b8d-4d40-8d8f-4fd3b5efd5ca/a699054f-e794-4026-95df-b546858c36d7"
       (reference "#PWR0108") (unit 1) (value "+5V") (footprint "")
@@
       (reference "#PWR0109") (unit 1) (value "GNDPWR") (footprint "")
     )
+    (path "/dd00c030-9b8d-4d40-8d8f-4fd3b5efd5ca/f5a71fa9-e4d6-4ba5-9e60-1e546211d93a"
+      (reference "#PWR0110") (unit 1) (value "+24V") (footprint "")
+    )
     (path "/dd00c030-9b8d-4d40-8d8f-4fd3b5efd5ca/498b6f1d-80e5-4a3b-8ba3-0c7a767b2c24"
       (reference "#PWR0111") (unit 1) (value "GND") (footprint "")
@@
       (reference "#PWR0114") (unit 1) (value "GNDPWR") (footprint "")
     )
+    (path "/dd00c030-9b8d-4d40-8d8f-4fd3b5efd5ca/74ff4524-eb61-4791-972c-bc786077f68d"
+      (reference "#PWR0115") (unit 1) (value "+24V") (footprint "")
+    )
     (path "/dd00c030-9b8d-4d40-8d8f-4fd3b5efd5ca/af81da96-1b40-4946-89e9-b8f63ae7eb79"
       (reference "#PWR0116") (unit 1) (value "GNDPWR") (footprint "")
@@
       (reference "#PWR0121") (unit 1) (value "+5V") (footprint "")
     )
+    (path "/dd00c030-9b8d-4d40-8d8f-4fd3b5efd5ca/e1fcac5b-38a3-4e13-9305-7b74c4f4617b"
+      (reference "#PWR0122") (unit 1) (value "+24V") (footprint "")
+    )
     (path "/dd00c030-9b8d-4d40-8d8f-4fd3b5efd5ca/4b20ccc5-c858-414e-960c-dfde9d9620ce"
       (reference "#PWR0123") (unit 1) (value "+5V") (footprint "")
@@
       (reference "#PWR0128") (unit 1) (value "GNDPWR") (footprint "")
     )
+    (path "/dd00c030-9b8d-4d40-8d8f-4fd3b5efd5ca/89bfb9bf-45dd-43c5-b761-f525139d48ba"
+      (reference "#PWR0129") (unit 1) (value "+24V") (footprint "")
+    )
     (path "/dd00c030-9b8d-4d40-8d8f-4fd3b5efd5ca/52132b2c-213b-41b0-90b0-689d8f5877e9"
       (reference "#PWR0130") (unit 1) (value "GNDPWR") (footprint "")
@@
       (reference "#PWR0138") (unit 1) (value "GNDPWR") (footprint "")
     )
+    (path "/dd00c030-9b8d-4d40-8d8f-4fd3b5efd5ca/d22ab3b3-7dd4-44ab-ab4f-363a34dc95db"
+      (reference "#PWR0139") (unit 1) (value "+24V") (footprint "")
+    )
     (path "/dd00c030-9b8d-4d40-8d8f-4fd3b5efd5ca/6c3f638b-cb14-4517-868e-6007fa9a3c7b"
       (reference "#PWR0140") (unit 1) (value "+5V") (footprint "")
     )
+    (path "/dd00c030-9b8d-4d40-8d8f-4fd3b5efd5ca/b594805f-074a-41d9-8a5f-b9d922339e49"
+      (reference "#PWR0141") (unit 1) (value "+24V") (footprint "")
+    )
     (path "/dd00c030-9b8d-4d40-8d8f-4fd3b5efd5ca/77e21c41-6018-4d2d-81a0-9796cd954bd0"
       (reference "#PWR0142") (unit 1) (value "GND") (footprint "")
@@
       (reference "#PWR0144") (unit 1) (value "GNDPWR") (footprint "")
     )
+    (path "/dd00c030-9b8d-4d40-8d8f-4fd3b5efd5ca/1ac7b23b-fd1b-4663-9f43-9f20e97e49b0"
+      (reference "#PWR0145") (unit 1) (value "+24V") (footprint "")
+    )
     (path "/dd00c030-9b8d-4d40-8d8f-4fd3b5efd5ca/a637c436-2f2f-42c6-94be-3ebe5d53a5ae"
       (reference "#PWR0146") (unit 1) (value "GND") (footprint "")
     )
+    (path "/dd00c030-9b8d-4d40-8d8f-4fd3b5efd5ca/2c012b80-b65f-4bc3-9f29-880a981b2dad"
+      (reference "#PWR0147") (unit 1) (value "+24V") (footprint "")
+    )
     (path "/dd00c030-9b8d-4d40-8d8f-4fd3b5efd5ca/4c008c9c-0b07-41f5-9b43-492542fef116"
       (reference "#PWR0148") (unit 1) (value "GNDPWR") (footprint "")
@@
       (reference "#PWR0186") (unit 1) (value "+24V") (footprint "")
     )
-    (path "/909b6f57-c767-4999-aebc-a22e874b7f96"
-      (reference "#PWR0187") (unit 1) (value "GND") (footprint "")
-    )
     (path "/36cad135-112c-4600-939d-93f9eed314a3"
       (reference "#PWR0188") (unit 1) (value "GNDPWR") (footprint "")
     )
-    (path "/f8c7401f-e334-4a21-8966-3cb30a833a3f"
-      (reference "#PWR0189") (unit 1) (value "+5V") (footprint "")
-    )
-    (path "/dd00c030-9b8d-4d40-8d8f-4fd3b5efd5ca/1ac7b23b-fd1b-4663-9f43-9f20e97e49b0"
-      (reference "#PWR?") (unit 1) (value "+24V") (footprint "")
-    )
-    (path "/dd00c030-9b8d-4d40-8d8f-4fd3b5efd5ca/2c012b80-b65f-4bc3-9f29-880a981b2dad"
-      (reference "#PWR?") (unit 1) (value "+24V") (footprint "")
-    )
-    (path "/dd00c030-9b8d-4d40-8d8f-4fd3b5efd5ca/4b355d96-1c0b-4ff4-91f0-4fd5a7144671"
-      (reference "#PWR?") (unit 1) (value "+24V") (footprint "")
-    )
-    (path "/dd00c030-9b8d-4d40-8d8f-4fd3b5efd5ca/74ff4524-eb61-4791-972c-bc786077f68d"
-      (reference "#PWR?") (unit 1) (value "+24V") (footprint "")
-    )
-    (path "/dd00c030-9b8d-4d40-8d8f-4fd3b5efd5ca/89bfb9bf-45dd-43c5-b761-f525139d48ba"
-      (reference "#PWR?") (unit 1) (value "+24V") (footprint "")
-    )
-    (path "/dd00c030-9b8d-4d40-8d8f-4fd3b5efd5ca/b594805f-074a-41d9-8a5f-b9d922339e49"
-      (reference "#PWR?") (unit 1) (value "+24V") (footprint "")
-    )
-    (path "/dd00c030-9b8d-4d40-8d8f-4fd3b5efd5ca/d22ab3b3-7dd4-44ab-ab4f-363a34dc95db"
-      (reference "#PWR?") (unit 1) (value "+24V") (footprint "")
-    )
-    (path "/dd00c030-9b8d-4d40-8d8f-4fd3b5efd5ca/e1fcac5b-38a3-4e13-9305-7b74c4f4617b"
-      (reference "#PWR?") (unit 1) (value "+24V") (footprint "")
-    )
-    (path "/dd00c030-9b8d-4d40-8d8f-4fd3b5efd5ca/e80b2b35-b6c0-4d41-bba7-6bc814b6444d"
-      (reference "#PWR?") (unit 1) (value "+24V") (footprint "")
-    )
-    (path "/dd00c030-9b8d-4d40-8d8f-4fd3b5efd5ca/f5a71fa9-e4d6-4ba5-9e60-1e546211d93a"
-      (reference "#PWR?") (unit 1) (value "+24V") (footprint "")
-    )
     (path "/dd00c030-9b8d-4d40-8d8f-4fd3b5efd5ca/7279863c-ff9f-41e2-868a-ae542af3f597"
       (reference "C1") (unit 1) (value "100nF") (footprint "Capacitor_SMD:C_0805_2012Metric_Pad1.18x1.45mm_HandSolder")
@@
       (reference "J19") (unit 1) (value "PORT") (footprint "TerminalBlock_Phoenix:TerminalBlock_Phoenix_PT-1,5-3-3.5-H_1x03_P3.50mm_Horizontal")
     )
-    (path "/299ed31b-8320-42e3-a997-78990b515eff"
-      (reference "J20") (unit 1) (value "5V in") (footprint "Connector_BarrelJack:BarrelJack_GCT_DCJ200-10-A_Horizontal")
-    )
     (path "/ec870b96-a94e-4dc6-9900-ce74b92f8bb5"
-      (reference "J21") (unit 1) (value "XT60-M") (footprint "PolyuRobotics:XT60PW-M20")
+      (reference "J21") (unit 1) (value "XT60-M") (footprint "Connector_AMASS:AMASS_XT60-M_1x02_P7.20mm_Vertical")
     )
     (path "/dd00c030-9b8d-4d40-8d8f-4fd3b5efd5ca/35634533-6645-4c4a-9e5c-2f43c1ab9439"
