File: solenoid_board/solenoid_board.kicad_pcb (KiCad board)
At the start: 2 copper layers, 150 parts, among them J1 mx2.54, J10 mx2.54, J11 CAN1, J12 CAN2, J13 mx2.54, J14 mx2.54, J15 CAN1, J16 CAN2, J17 mx2.54, J18 mx2.54, J19 I2C3, J2 mx2.54, J20 UART4, J21 xt60 male, J3 CAN1, J4 CAN2, J5 mx2.54, J6 mx2.54, J7 CAN1, J8 CAN2, J9 mx2.54, M3 TJA1050_Module, M4 TJA1050_Module, Q1 IRF540NSTRLPBF, Q10 IRF540NSTRLPBF, Q2 IRF540NSTRLPBF, Q3 IRF540NSTRLPBF, Q4 IRF540NSTRLPBF, Q5 IRF540NSTRLPBF, Q6 IRF540NSTRLPBF, Q7 IRF540NSTRLPBF, Q8 IRF540NSTRLPBF, Q9 IRF540NSTRLPBF, SW1 SW_Push, SW10 SW_Push, SW2 SW_Push, SW3 SW_Push, SW4 SW_Push, SW5 SW_Push, SW6 SW_Push, SW7 SW_Push, SW8 SW_Push, SW9 SW_Push, U1 NUCLEO-F446RE, U10 4N35, U11 4N35, U12 4N35, U2 MP1584, U3 4N35, U4 4N35, U5 4N35, U6 4N35, U7 4N35, U8 4N35, U9 4N35

Commit message: add
Parts:
- added C15: 100nF, Capacitor_SMD:C_0805_2012Metric_Pad1.18x1.45mm_HandSolder, F.Cu at (72.8, 165.9)
- added C16: 100nF, Capacitor_SMD:C_0805_2012Metric_Pad1.18x1.45mm_HandSolder, F.Cu at (137.8, 134.7)
- added C17: 100nF, Capacitor_SMD:C_0805_2012Metric_Pad1.18x1.45mm_HandSolder, F.Cu at (136.7, 171.2)
- added C18: 100nF, Capacitor_SMD:C_0805_2012Metric_Pad1.18x1.45mm_HandSolder, F.Cu at (55.0, 168.2)
- added C19: 100nF, Capacitor_SMD:C_0805_2012Metric_Pad1.18x1.45mm_HandSolder, F.Cu at (100.5, 166.6)
- added C20: 100nF, Capacitor_SMD:C_0805_2012Metric_Pad1.18x1.45mm_HandSolder, F.Cu at (44.5, 165.6)
- added C21: 100nF, Capacitor_SMD:C_0805_2012Metric_Pad1.18x1.45mm_HandSolder, F.Cu at (127.9, 166.3)
- added C22: 100nF, Capacitor_SMD:C_0805_2012Metric_Pad1.18x1.45mm_HandSolder, F.Cu at (86.2, 171.7)
- added C23: 100nF, Capacitor_SMD:C_0805_2012Metric_Pad1.18x1.45mm_HandSolder, F.Cu at (26.3, 168.0)
- added C24: 100nF, Capacitor_SMD:C_0805_2012Metric_Pad1.18x1.45mm_HandSolder, F.Cu at (109.3, 170.0)
- added D27: LED2, LED_SMD:LED_0805_2012Metric_Pad1.15x1.40mm_HandSolder, F.Cu at (99.6, 115.6)
- added D28: LED3, LED_SMD:LED_0805_2012Metric_Pad1.15x1.40mm_HandSolder, F.Cu at (97.0, 115.6)
- added R56: 470R, Resistor_SMD:R_0805_2012Metric_Pad1.20x1.40mm_HandSolder, F.Cu at (102.1, 111.5)
- added R57: 470R, Resistor_SMD:R_0805_2012Metric_Pad1.20x1.40mm_HandSolder, F.Cu at (99.6, 111.5)
- added R58: 470R, Resistor_SMD:R_0805_2012Metric_Pad1.20x1.40mm_HandSolder, F.Cu at (97.0, 111.5)
- added R59: 120R, Resistor_SMD:R_0805_2012Metric_Pad1.20x1.40mm_HandSolder, F.Cu at (129.6, 67.4)
- added R60: 120R, Resistor_SMD:R_0805_2012Metric_Pad1.20x1.40mm_HandSolder, F.Cu at (129.6, 72.6)
- added SW11: SW_DIP_x04, Button_Switch_THT:SW_DIP_SPSTx04_Slide_9.78x12.34mm_W7.62mm_P2.54mm, F.Cu at (117.6, 67.6)
- D10, D17, D23: value indictor -> 1N4001; footprint LED_SMD:LED_0805_2012Metric_Pad1.15x1.40mm_HandSolder -> Diode_THT:D_DO-41_SOD81_P10.16mm_Horizontal
- D14, D20: value 1N4001 -> indictor; footprint Diode_THT:D_DO-41_SOD81_P10.16mm_Horizontal -> LED_SMD:LED_0805_2012Metric_Pad1.15x1.40mm_HandSolder
- D26: value 1N4001 -> LED1; footprint Diode_THT:D_DO-41_SOD81_P10.16mm_Horizontal -> LED_SMD:LED_0805_2012Metric_Pad1.15x1.40mm_HandSolder
- D6: value ss24 -> indictor; footprint Diode_SMD:D_SMB_Handsoldering -> LED_SMD:LED_0805_2012Metric_Pad1.15x1.40mm_HandSolder
- J19, J20: footprint Connector_PinHeader_2.54mm:PinHeader_1x04_P2.54mm_Vertical -> Connector_Molex:Molex_Nano-Fit_105309-xx04_1x04_P2.50mm_Vertical
- moved J13 257.3 mm to (55.6, 193.0), turned to 90 degrees
- moved R40 250.0 mm to (58.8, 187.9), turned to 90 degrees
- moved R37 250.0 mm to (55.0, 186.0), turned to 0 degrees
- moved R34 244.3 mm to (55.0, 182.2), turned to 180 degrees
- moved D24 240.0 mm to (35.8, 190.2), turned to 0 degrees
- moved Q7 235.7 mm to (67.7, 179.0), turned to 90 degrees
- moved D20 232.2 mm to (86.9, 188.4), turned to 180 degrees
- moved D19 231.8 mm to (71.5, 193.0), turned to 180 degrees
- moved D21 230.6 mm to (30.7, 181.3), turned to 180 degrees
- moved D16 230.3 mm to (58.8, 183.5), turned to 90 degrees
- moved U9 227.5 mm to (58.8, 171.4), turned to -90 degrees
- moved R31 223.2 mm to (59.1, 168.2), turned to 180 degrees
- moved R28 222.1 mm to (59.4, 164.4), turned to 0 degrees
- moved J2 219.8 mm to (54.7, 155.3), turned to 90 degrees
- moved R19 210.3 mm to (54.7, 150.7), turned to 0 degrees
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Connections:
- C13 pad 2: GND -> PC6
- C14 pad 2: GND -> PC10
- C3 pad 1: Net-(C3-Pad1) -> +24V
- C6 pad 2: GND -> PC2
- C7 pad 2: GND -> PC3
- C8 pad 2: GND -> PC4
- C9 pad 2: GND -> PC5
- D10 pad 1: GNDPWR -> VCC
- D14 pad 1: VCC -> GNDPWR
- D17 pad 1: GNDPWR -> VCC
- D20 pad 1: VCC -> GNDPWR
- D23 pad 1: GNDPWR -> VCC
- D26 pad 1: VCC -> GND
- D6 pad 1: Net-(C3-Pad1) -> GNDPWR
- D6 pad 2: +24V -> Net-(D6-Pad2)
- J10 pad 2: Net-(D19-Pad2) -> Net-(D18-Pad2)
- J13 pad 2: Net-(D20-Pad2) -> Net-(D19-Pad2)
- J14 pad 2: Net-(D24-Pad2) -> Net-(D23-Pad2)
- J17 pad 2: Net-(D25-Pad2) -> Net-(D24-Pad2)
- J18 pad 2: Net-(D26-Pad2) -> Net-(D25-Pad2)
- J2 pad 2: Net-(D12-Pad2) -> Net-(D10-Pad2)
- J5 pad 2: Net-(D13-Pad2) -> Net-(D12-Pad2)
- J6 pad 2: Net-(D14-Pad2) -> Net-(D13-Pad2)
- J9 pad 2: Net-(D18-Pad2) -> Net-(D17-Pad2)
- M3 pad 1: +5V -> /MCU/CAN1_VCC
- M4 pad 1: +5V -> /MCU/CAN2_VCC
- Q10 pad 2: Net-(D26-Pad2) -> Net-(D25-Pad2)
- Q2 pad 2: Net-(D12-Pad2) -> Net-(D10-Pad2)
- Q3 pad 2: Net-(D13-Pad2) -> Net-(D12-Pad2)
- Q4 pad 2: Net-(D14-Pad2) -> Net-(D13-Pad2)
- Q5 pad 2: Net-(D18-Pad2) -> Net-(D17-Pad2)
- Q6 pad 2: Net-(D19-Pad2) -> Net-(D18-Pad2)
- Q7 pad 2: Net-(D20-Pad2) -> Net-(D19-Pad2)
- Q8 pad 2: Net-(D24-Pad2) -> Net-(D23-Pad2)
- Q9 pad 2: Net-(D25-Pad2) -> Net-(D24-Pad2)
- R1 pad 2: Net-(R1-Pad2) -> Net-(C6-Pad1)
- R10 pad 1: Net-(R10-Pad1) -> PC2
- R11 pad 1: Net-(R11-Pad1) -> PC3
- R11 pad 2: Net-(C6-Pad1) -> Net-(C10-Pad1)
- R12 pad 1: Net-(R12-Pad1) -> PC4
- R12 pad 2: Net-(C7-Pad1) -> Net-(C11-Pad1)
- R13 pad 1: Net-(R13-Pad1) -> PC5
- R13 pad 2: Net-(C8-Pad1) -> Net-(C12-Pad1)
- R16 pad 1: Net-(D9-Pad2) -> Net-(D6-Pad2)
- R17 pad 1: Net-(D10-Pad2) -> Net-(D9-Pad2)
- R2 pad 2: Net-(R2-Pad2) -> Net-(C7-Pad1)
- R26 pad 2: Net-(R26-Pad2) -> Net-(C13-Pad1)
- R27 pad 2: Net-(R27-Pad2) -> Net-(C14-Pad1)
- R29 pad 1: Net-(R29-Pad1) -> PC6
- R29 pad 2: Net-(C9-Pad1) -> Net-(C16-Pad1)
- R30 pad 1: Net-(R30-Pad1) -> PC10
- R30 pad 2: Net-(C10-Pad1) -> Net-(C17-Pad1)
- R31 pad 1: Net-(R31-Pad1) -> PC11
- R31 pad 2: Net-(C11-Pad1) -> Net-(C18-Pad1)
- R32 pad 1: Net-(D15-Pad2) -> Net-(D14-Pad2)
- R33 pad 1: Net-(D16-Pad2) -> Net-(D15-Pad2)
- R34 pad 1: Net-(D17-Pad2) -> Net-(D16-Pad2)
- R4 pad 1: +5V -> /MCU/CAN1_VCC
- R44 pad 1: Net-(R44-Pad1) -> PC12
- R44 pad 2: Net-(C12-Pad1) -> Net-(C22-Pad1)
- R45 pad 1: Net-(R45-Pad1) -> PC14
- R45 pad 2: Net-(C13-Pad1) -> Net-(C23-Pad1)
- R46 pad 1: Net-(R46-Pad1) -> PC15
- R46 pad 2: Net-(C14-Pad1) -> Net-(C24-Pad1)
- R47 pad 1: Net-(D21-Pad2) -> Net-(D20-Pad2)
- R48 pad 1: Net-(D22-Pad2) -> Net-(D21-Pad2)
- R49 pad 1: Net-(D23-Pad2) -> Net-(D22-Pad2)
- R5 pad 1: +5V -> /MCU/CAN2_VCC
- R8 pad 2: Net-(R8-Pad2) -> Net-(C8-Pad1)
- R9 pad 2: Net-(R9-Pad2) -> Net-(C9-Pad1)
- SW1 pad 1: Net-(R1-Pad2) -> Net-(C6-Pad1)
- SW1 pad 2: Net-(R10-Pad1) -> PC2
- SW10 pad 2: Net-(R46-Pad1) -> PC15
- SW2 pad 1: Net-(R2-Pad2) -> Net-(C7-Pad1)
- SW2 pad 2: Net-(R11-Pad1) -> PC3
- SW3 pad 1: Net-(R8-Pad2) -> Net-(C8-Pad1)
- SW3 pad 2: Net-(R12-Pad1) -> PC4
- SW4 pad 1: Net-(R9-Pad2) -> Net-(C9-Pad1)
- SW4 pad 2: Net-(R13-Pad1) -> PC5
- SW5 pad 1: Net-(R26-Pad2) -> Net-(C13-Pad1)
- SW5 pad 2: Net-(R29-Pad1) -> PC6
- SW6 pad 1: Net-(R27-Pad2) -> Net-(C14-Pad1)
- SW6 pad 2: Net-(R30-Pad1) -> PC10
- SW7 pad 2: Net-(R31-Pad1) -> PC11
- SW8 pad 2: Net-(R44-Pad1) -> PC12
- SW9 pad 2: Net-(R45-Pad1) -> PC14
- U10 pad 1: Net-(C12-Pad1) -> Net-(C22-Pad1)
- U11 pad 1: Net-(C13-Pad1) -> Net-(C23-Pad1)
- U12 pad 1: Net-(C14-Pad1) -> Net-(C24-Pad1)
- U2 pad IN1+: Net-(C3-Pad1) -> +24V
- U2 pad IN2+: Net-(C3-Pad1) -> +24V
- U4 pad 1: Net-(C6-Pad1) -> Net-(C10-Pad1)
- U5 pad 1: Net-(C7-Pad1) -> Net-(C11-Pad1)
- U6 pad 1: Net-(C8-Pad1) -> Net-(C12-Pad1)
- U7 pad 1: Net-(C9-Pad1) -> Net-(C16-Pad1)
- U8 pad 1: Net-(C10-Pad1) -> Net-(C17-Pad1)
- U9 pad 1: Net-(C11-Pad1) -> Net-(C18-Pad1)

Commit message: solenoid board
Parts:
- removed C11, C12, C13, C14, C15, C16, C17, C18, C19, C20, C21, C22, C23, C24: 100nF, Capacitor_SMD:C_0805_2012Metric_Pad1.18x1.45mm_HandSolder
- removed J13, J14, J17, J18: mx2.54, Connector_PinHeader_2.54mm:PinHeader_1x02_P2.54mm_Vertical
- removed J15: CAN1, Connector_Molex:Molex_Micro-Fit_3.0_43045-0412_2x02_P3.00mm_Vertical
- removed J16: CAN2, Connector_Molex:Molex_Micro-Fit_3.0_43045-0412_2x02_P3.00mm_Vertical
- removed J19: I2C3, Connector_Molex:Molex_Nano-Fit_105309-xx04_1x04_P2.50mm_Vertical
- removed J20: UART4, Connector_Molex:Molex_Nano-Fit_105309-xx04_1x04_P2.50mm_Vertical
- removed J21: xt60 male, PolyuRobotics:XT60PW-M20
- removed M3, M4: TJA1050_Module, PolyuRobotics:TJA1050_CAN_Module
- removed SW11: SW_DIP_x04, Button_Switch_THT:SW_DIP_SPSTx04_Slide_9.78x12.34mm_W7.62mm_P2.54mm
- removed U12: 4N35, Package_DIP:DIP-6_W7.62mm
- added D29: 1N4001, Diode_THT:D_DO-41_SOD81_P10.16mm_Horizontal, F.Cu at (51.4, 39.0)
- added D30: 1N4001, Diode_THT:D_DO-41_SOD81_P10.16mm_Horizontal, F.Cu at (51.4, 26.3)
- added D32: Signal, LED_SMD:LED_0805_2012Metric_Pad1.15x1.40mm_HandSolder, F.Cu at (69.3, 79.5)
- added R61: 4K7, Resistor_SMD:R_0805_2012Metric_Pad1.20x1.40mm_HandSolder, F.Cu at (69.2, 82.5)
- added R62: 10K, Resistor_SMD:R_0805_2012Metric_Pad1.20x1.40mm_HandSolder, F.Cu at (51.9, 99.8)
- added R63: 4K7, Resistor_SMD:R_0805_2012Metric_Pad1.20x1.40mm_HandSolder, F.Cu at (60.0, 92.7)
- added R64: 200R, Resistor_SMD:R_0805_2012Metric_Pad1.20x1.40mm_HandSolder, F.Cu at (51.9, 96.9)
- C1: value 16v100uF -> 100nF; footprint Capacitor_SMD:C_Elec_6.3x7.7 -> Capacitor_SMD:C_0805_2012Metric_Pad1.18x1.45mm_HandSolder
- C2: value 16v 47uF -> 100nF; footprint Capacitor_SMD:C_Elec_6.3x7.7 -> Capacitor_SMD:C_0805_2012Metric_Pad1.18x1.45mm_HandSolder
- C3: value 50v 47uF -> 100nF; footprint Capacitor_SMD:C_Elec_6.3x7.7 -> Capacitor_SMD:C_0805_2012Metric_Pad1.18x1.45mm_HandSolder
- C4: value 16v 100uF -> 100nF; footprint Capacitor_SMD:C_Elec_6.3x7.7 -> Capacitor_SMD:C_0805_2012Metric_Pad1.18x1.45mm_HandSolder
- D13, D24, D25: value 1N4001 -> SS24; footprint Diode_THT:D_DO-41_SOD81_P10.16mm_Horizontal -> Diode_SMD:D_SMB
- D15, D16, D2, D22: value indictor -> SS24; footprint LED_SMD:LED_0805_2012Metric_Pad1.15x1.40mm_HandSolder -> Diode_SMD:D_SMB
- D17, D18, D23: value 1N4001 -> indictor; footprint Diode_THT:D_DO-41_SOD81_P10.16mm_Horizontal -> LED_SMD:LED_0805_2012Metric_Pad1.15x1.40mm_HandSolder
- D20, D21, D9: value indictor -> 1N4001; footprint LED_SMD:LED_0805_2012Metric_Pad1.15x1.40mm_HandSolder -> Diode_THT:D_DO-41_SOD81_P10.16mm_Horizontal
- D26: value LED1 -> indictor
- D27: value LED2 -> indictor
- D28: value LED3 -> 1N4001; footprint LED_SMD:LED_0805_2012Metric_Pad1.15x1.40mm_HandSolder -> Diode_THT:D_DO-41_SOD81_P10.16mm_Horizontal
- D3: value power_led -> SS24; footprint LED_SMD:LED_0805_2012Metric_Pad1.15x1.40mm_HandSolder -> Diode_SMD:D_SMB
- D4: value can_led -> indictor
- D5: value can_led -> SS24; footprint LED_SMD:LED_0805_2012Metric_Pad1.15x1.40mm_HandSolder -> Diode_SMD:D_SMB
- D7: value SMBJ24CA -> SS24; footprint Diode_SMD:D_SMB_Handsoldering -> Diode_SMD:D_SMB
- D8: value SMBJ9VCA -> indictor; footprint Diode_SMD:D_SMB_Handsoldering -> LED_SMD:LED_0805_2012Metric_Pad1.15x1.40mm_HandSolder
- J11, J3, J7: value CAN1 -> mx2.54; footprint Connector_Molex:Molex_Micro-Fit_3.0_43045-0412_2x02_P3.00mm_Vertical -> Connector_PinHeader_2.54mm:PinHeader_1x02_P2.54mm_Vertical
- J12: value CAN2 -> PORT; footprint Connector_Molex:Molex_Micro-Fit_3.0_43045-0412_2x02_P3.00mm_Vertical -> TerminalBlock_Phoenix:TerminalBlock_Phoenix_MKDS-3-3-5.08_1x03_P5.08mm_Horizontal
- J2: value mx2.54 -> Conn_02x13_Odd_Even; footprint Connector_PinHeader_2.54mm:PinHeader_1x02_P2.54mm_Vertical -> Connector_IDC:IDC-Header_2x13_P2.54mm_Vertical
- J4, J8: value CAN2 -> mx2.54; footprint Connector_Molex:Molex_Micro-Fit_3.0_43045-0412_2x02_P3.00mm_Vertical -> Connector_PinHeader_2.54mm:PinHeader_1x02_P2.54mm_Vertical
- Q1: value IRF540NSTRLPBF -> AOD4184A; footprint PolyuRobotics:IRF540NSTRLPBF -> PolyuRobotics:DPAK228P994X240-4N
- Q10, Q2, Q3, Q4, Q5, Q6, Q7, Q8, Q9: value IRF540NSTRLPBF -> ~; footprint PolyuRobotics:IRF540NSTRLPBF -> PolyuRobotics:DPAK228P994X240-4N
- R11, R12, R31: value 470R -> ~
- R13: value 470R -> 3.3K
- R17: value 3.3K -> 100R
- R21: value 100R -> 10k
- R25: value 10k -> 1k
- R28, R8: value 1k -> 470R
- R3, R4: value 10K -> 1k
- R32, R33, R49: value 3.3K -> ~
- R35, R36, R52: value 100R -> 3.3K
- R38, R39, R55: value 10k -> 100R
- R41, R42: value 1k -> 10k
- R44, R45: value 470R -> 1k
- R47, R48: value 3.3K -> 470R
- R5: value 10K -> 470R
- R50, R51: value 100R -> ~
- R53, R54: value 10k -> 3.3K
- R56, R57: value 470R -> 100R
- R58: value 470R -> 10k
- R59, R60: value 120R -> 10k
- R6: value 4.7k -> 10K
- R7: value 4.7k -> 470R
- R9: value 1k -> ~
- U1: value NUCLEO-F446RE -> EL357N; footprint PolyuRobotics:NUCLEO-F446RE -> PolyuRobotics:EL357N
- U10, U3, U4, U5, U6, U7, U8, U9: value 4N35 -> ~; footprint Package_DIP:DIP-6_W7.62mm -> PolyuRobotics:EL357N
- U11: value 4N35 -> EL357N; footprint Package_DIP:DIP-6_W7.62mm -> PolyuRobotics:EL357N
- U2: value MP1584 -> ~; footprint PolyuRobotics:DC-DC-mp1584_module -> PolyuRobotics:EL357N
- moved R51 205.4 mm to (148.6, 20.1)
- moved R48 191.0 mm to (143.1, 30.2), turned to 0 degrees
- moved R37 190.8 mm to (143.8, 17.1)
- moved D24 173.9 mm to (141.1, 51.8)
- moved D20 170.8 mm to (79.3, 17.8), turned to 0 degrees
- moved J2 169.0 mm to (192.9, 58.0), turned to -90 degrees
- moved R50 164.7 mm to (137.7, 33.2)
- moved D19 163.7 mm to (51.4, 30.5), turned to 0 degrees
- moved D21 160.6 mm to (51.4, 22.0), turned to 0 degrees
- moved Q10 158.7 mm to (81.6, 26.3), turned to 0 degrees
- moved R40 158.2 mm to (118.6, 41.5), turned to 0 degrees
- moved R44 157.8 mm to (147.6, 23.0)
- moved Q6 157.3 mm to (89.9, 35.4), turned to 0 degrees
- moved U8 156.8 mm to (132.7, 17.5), turned to 0 degrees
- moved R42 156.8 mm to (128.4, 41.8)
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Connections:
- C1 pad 1: VCC -> Net-(C1-Pad1)
- C1 pad 2: GND -> PB2
- C10 pad 2: GND -> PA4
- C2 pad 1: +5V -> Net-(C2-Pad1)
- C2 pad 2: GND -> PA9
- C3 pad 1: +24V -> Net-(C3-Pad1)
- C3 pad 2: GND -> PA7
- C4 pad 1: VCC -> Net-(C4-Pad1)
- C4 pad 2: GND -> PA6
- C5 pad 2: GND -> PC11
- C6 pad 2: PC2 -> PB1
- C7 pad 2: PC3 -> PA5
- C8 pad 2: PC4 -> PC10
- C9 pad 2: PC5 -> PC12
- D10 pad 1: VCC -> Net-(D10-Pad1)
- D11 pad 1: VCC -> Net-(D11-Pad1)
- D12 pad 1: VCC -> Net-(D12-Pad1)
- D15 pad 1: GNDPWR -> VCC
- D16 pad 1: GNDPWR -> VCC
- D17 pad 1: VCC -> GNDPWR
- D18 pad 1: VCC -> GNDPWR
- D19 pad 1: VCC -> Net-(D13-Pad2)
- D2 pad 1: GNDPWR -> VCC
- D2 pad 2: Net-(D2-Pad2) -> Net-(D11-Pad1)
- D20 pad 1: GNDPWR -> Net-(D15-Pad2)
- D21 pad 1: GNDPWR -> Net-(D16-Pad2)
- D22 pad 1: GNDPWR -> VCC
- D23 pad 1: VCC -> GNDPWR
- D26 pad 1: GND -> GNDPWR
- D27 pad 1: GND -> GNDPWR
- D28 pad 1: GND -> Net-(D22-Pad2)
- D3 pad 1: GND -> VCC
- D4 pad 1: GND -> GNDPWR
- D5 pad 1: GND -> VCC
- D5 pad 2: Net-(D5-Pad2) -> Net-(D10-Pad1)
- D7 pad 1: +24V -> VCC
- D7 pad 2: GND -> Net-(D12-Pad1)
- D8 pad 1: VCC -> GNDPWR
- D8 pad 2: GND -> Net-(D8-Pad2)
- D9 pad 1: GNDPWR -> Net-(D3-Pad2)
- J1 pad 1: VCC -> Net-(D11-Pad1)
- J10 pad 1: VCC -> Net-(D24-Pad2)
- J10 pad 2: Net-(D18-Pad2) -> Net-(D29-Pad2)
- J11 pad 1: /MCU/CAN1+ -> Net-(D25-Pad2)
- J11 pad 2: /MCU/CAN1- -> Net-(D30-Pad2)
- J12 pad 1: /MCU/CAN2+ -> GNDPWR
- J12 pad 2: /MCU/CAN2- -> Net-(J12-Pad2)
- J12 pad 3: GND -> +24V
- J2 pad 1: VCC -> PB1
- J2 pad 2: Net-(D10-Pad2) -> PB3
- J3 pad 1: /MCU/CAN1+ -> Net-(D3-Pad2)
- J3 pad 2: /MCU/CAN1- -> Net-(D9-Pad2)
- J4 pad 1: /MCU/CAN2+ -> Net-(D10-Pad1)
- J4 pad 2: /MCU/CAN2- -> Net-(D10-Pad2)
- J5 pad 1: VCC -> Net-(D12-Pad1)
- J6 pad 1: VCC -> Net-(D13-Pad2)
- J6 pad 2: Net-(D13-Pad2) -> Net-(D19-Pad2)
- J7 pad 1: /MCU/CAN1+ -> Net-(D15-Pad2)
- J7 pad 2: /MCU/CAN1- -> Net-(D20-Pad2)
- J8 pad 1: /MCU/CAN2+ -> Net-(D16-Pad2)
- J8 pad 2: /MCU/CAN2- -> Net-(D21-Pad2)
- J9 pad 1: VCC -> Net-(D22-Pad2)
- J9 pad 2: Net-(D17-Pad2) -> Net-(D28-Pad2)
- R10 pad 1: PC2 -> PB1
- R10 pad 2: Net-(C5-Pad1) -> Net-(R10-Pad2)
- R11 pad 1: PC3 -> GND
- R11 pad 2: Net-(C10-Pad1) -> Net-(R11-Pad2)
- R12 pad 1: PC4 -> GND
- R12 pad 2: Net-(C11-Pad1) -> Net-(R12-Pad2)
- R13 pad 1: PC5 -> Net-(D4-Pad2)
- R13 pad 2: Net-(C12-Pad1) -> Net-(R13-Pad2)
- R15 pad 1: Net-(D2-Pad2) -> Net-(D6-Pad2)
- R16 pad 1: Net-(D6-Pad2) -> Net-(D8-Pad2)
- R17 pad 1: Net-(D9-Pad2) -> Net-(R13-Pad2)
- R17 pad 2: Net-(R17-Pad2) -> Net-(Q2-Pad1)
- R19 pad 2: Net-(Q2-Pad1) -> Net-(Q3-Pad1)
- R2 pad 2: Net-(C7-Pad1) -> Net-(C1-Pad1)
- R20 pad 2: Net-(Q3-Pad1) -> Net-(Q4-Pad1)
- R21 pad 1: Net-(R17-Pad2) -> GNDPWR
- R21 pad 2: Net-(Q4-Pad1) -> Net-(Q2-Pad1)
- R23 pad 2: Net-(Q2-Pad1) -> Net-(Q3-Pad1)
- R24 pad 2: Net-(Q3-Pad1) -> Net-(Q4-Pad1)
- R25 pad 1: GNDPWR -> +5V
- R25 pad 2: Net-(Q4-Pad1) -> Net-(C4-Pad1)
- R26 pad 2: Net-(C13-Pad1) -> Net-(C5-Pad1)
- R27 pad 2: Net-(C14-Pad1) -> Net-(C7-Pad1)
- R28 pad 1: +5V -> PA6
- R28 pad 2: Net-(C15-Pad1) -> Net-(R28-Pad2)
- R29 pad 1: PC6 -> PC11
- R29 pad 2: Net-(C16-Pad1) -> Net-(R29-Pad2)
- R3 pad 1: VCC -> +5V
- R3 pad 2: Net-(D3-Pad2) -> Net-(C2-Pad1)
- R30 pad 1: PC10 -> PA5
- R30 pad 2: Net-(C17-Pad1) -> Net-(R30-Pad2)
- R31 pad 1: PC11 -> GND
- R31 pad 2: Net-(C18-Pad1) -> Net-(R28-Pad2)
- R32 pad 1: Net-(D14-Pad2) -> GND
- R32 pad 2: Net-(R32-Pad2) -> Net-(R29-Pad2)
- R33 pad 1: Net-(D15-Pad2) -> GND
- R33 pad 2: Net-(R33-Pad2) -> Net-(R30-Pad2)
- R34 pad 1: Net-(D16-Pad2) -> Net-(D14-Pad2)
- R35 pad 1: Net-(R32-Pad2) -> Net-(D17-Pad2)
- R35 pad 2: Net-(Q5-Pad1) -> Net-(R35-Pad2)
- R36 pad 1: Net-(R33-Pad2) -> Net-(D18-Pad2)
- R36 pad 2: Net-(Q6-Pad1) -> Net-(R36-Pad2)
- R37 pad 2: Net-(Q7-Pad1) -> Net-(Q5-Pad1)
- R38 pad 1: GNDPWR -> Net-(R35-Pad2)
- R38 pad 2: Net-(Q5-Pad1) -> Net-(Q6-Pad1)
- R39 pad 1: GNDPWR -> Net-(R36-Pad2)
- R39 pad 2: Net-(Q6-Pad1) -> Net-(Q7-Pad1)
- R4 pad 1: /MCU/CAN1_VCC -> +5V
- R4 pad 2: Net-(D4-Pad2) -> Net-(C3-Pad1)
- R40 pad 2: Net-(Q7-Pad1) -> Net-(Q5-Pad1)
- R41 pad 1: +5V -> GNDPWR
- R41 pad 2: Net-(C19-Pad1) -> Net-(Q6-Pad1)
- R42 pad 1: +5V -> GNDPWR
- R42 pad 2: Net-(C20-Pad1) -> Net-(Q7-Pad1)
- R43 pad 2: Net-(C21-Pad1) -> Net-(C8-Pad1)
- R44 pad 1: PC12 -> +5V
- R44 pad 2: Net-(C22-Pad1) -> Net-(C9-Pad1)
- R45 pad 1: PC14 -> +5V
- R45 pad 2: Net-(C23-Pad1) -> Net-(C10-Pad1)
- R46 pad 1: PC15 -> PC10
- R46 pad 2: Net-(C24-Pad1) -> Net-(R46-Pad2)
- R47 pad 1: Net-(D20-Pad2) -> PC12
- R48 pad 1: Net-(D21-Pad2) -> PA4
- R49 pad 1: Net-(D22-Pad2) -> GND
- R49 pad 2: Net-(R49-Pad2) -> Net-(R46-Pad2)
- R5 pad 1: /MCU/CAN2_VCC -> PB2
- R5 pad 2: Net-(D5-Pad2) -> Net-(R5-Pad2)
- R50 pad 1: Net-(R47-Pad2) -> GND
- R50 pad 2: Net-(Q8-Pad1) -> Net-(R47-Pad2)
- R51 pad 1: Net-(R48-Pad2) -> GND
- R51 pad 2: Net-(Q9-Pad1) -> Net-(R48-Pad2)
- R52 pad 1: Net-(R49-Pad2) -> Net-(D23-Pad2)
- R52 pad 2: Net-(Q10-Pad1) -> Net-(R52-Pad2)
- R53 pad 1: GNDPWR -> Net-(D26-Pad2)
- R53 pad 2: Net-(Q8-Pad1) -> Net-(R53-Pad2)
- R54 pad 1: GNDPWR -> Net-(D27-Pad2)
- R54 pad 2: Net-(Q9-Pad1) -> Net-(R54-Pad2)
- R55 pad 1: GNDPWR -> Net-(R52-Pad2)
- R55 pad 2: Net-(Q10-Pad1) -> Net-(Q8-Pad1)
- R56 pad 1: /MCU/PC7 -> Net-(R53-Pad2)
- R56 pad 2: Net-(D26-Pad2) -> Net-(Q9-Pad1)
- R57 pad 1: /MCU/PC8 -> Net-(R54-Pad2)
- R57 pad 2: Net-(D27-Pad2) -> Net-(Q10-Pad1)
- R58 pad 1: /MCU/PC9 -> GNDPWR
- R58 pad 2: Net-(D28-Pad2) -> Net-(Q8-Pad1)
- R59 pad 1: Net-(R59-Pad1) -> GNDPWR
- R59 pad 2: /MCU/CAN2- -> Net-(Q9-Pad1)
- R6 pad 1: +3V3 -> GND
- R6 pad 2: /MCU/PA8 -> Net-(R10-Pad2)
- R60 pad 1: Net-(SW11-Pad6) -> GNDPWR
- R60 pad 2: /MCU/CAN1- -> Net-(Q10-Pad1)
- R7 pad 1: +3V3 -> PA9
- R7 pad 2: /MCU/PB4 -> Net-(R11-Pad2)
- R8 pad 1: +5V -> PA7
- R8 pad 2: Net-(C8-Pad1) -> Net-(R12-Pad2)
- R9 pad 1: +5V -> GND
- R9 pad 2: Net-(C9-Pad1) -> Net-(R5-Pad2)
- SW1 pad 2: PC2 -> PB1
- SW10 pad 1: Net-(C21-Pad1) -> Net-(C10-Pad1)
- SW10 pad 2: PC15 -> PA4
- SW2 pad 1: Net-(C7-Pad1) -> Net-(C1-Pad1)
- SW2 pad 2: PC3 -> PB2
- SW3 pad 1: Net-(C8-Pad1) -> Net-(C2-Pad1)
- SW3 pad 2: PC4 -> PA9
- SW4 pad 1: Net-(C9-Pad1) -> Net-(C3-Pad1)
- SW4 pad 2: PC5 -> PA7
- SW5 pad 1: Net-(C13-Pad1) -> Net-(C4-Pad1)
- SW5 pad 2: PC6 -> PA6
- SW6 pad 1: Net-(C14-Pad1) -> Net-(C5-Pad1)
- SW6 pad 2: PC10 -> PC11
- SW7 pad 1: Net-(C15-Pad1) -> Net-(C7-Pad1)
- SW7 pad 2: PC11 -> PA5
- SW8 pad 1: Net-(C19-Pad1) -> Net-(C8-Pad1)
- SW8 pad 2: PC12 -> PC10
- SW9 pad 1: Net-(C20-Pad1) -> Net-(C9-Pad1)
- SW9 pad 2: PC14 -> PC12
- U10 pad 1: Net-(C22-Pad1) -> Net-(R48-Pad2)
- U10 pad 3: unconnected-(U10-Pad3) -> Net-(R54-Pad2)
- U10 pad 4: Net-(R47-Pad2) -> VCC
- U11 pad 1: Net-(C23-Pad1) -> Net-(D31-Pad1)
- U11 pad 2: GND -> Net-(D32-Pad2)
- U11 pad 3: unconnected-(U11-Pad3) -> GND
- U11 pad 4: Net-(R48-Pad2) -> Net-(R63-Pad2)
- U3 pad 1: Net-(C5-Pad1) -> Net-(R11-Pad2)
- U3 pad 3: unconnected-(U3-Pad3) -> Net-(R15-Pad2)
- U3 pad 4: Net-(R14-Pad2) -> VCC
- U4 pad 1: Net-(C10-Pad1) -> Net-(R12-Pad2)
- U4 pad 3: unconnected-(U4-Pad3) -> Net-(R16-Pad2)
- U4 pad 4: Net-(R15-Pad2) -> VCC
- U5 pad 1: Net-(C11-Pad1) -> Net-(R28-Pad2)
- U5 pad 3: unconnected-(U5-Pad3) -> Net-(R34-Pad2)
- U5 pad 4: Net-(R16-Pad2) -> VCC
- U6 pad 1: Net-(C12-Pad1) -> Net-(R29-Pad2)
- U6 pad 3: unconnected-(U6-Pad3) -> Net-(R35-Pad2)
- U6 pad 4: Net-(R17-Pad2) -> VCC
- U7 pad 1: Net-(C16-Pad1) -> Net-(R30-Pad2)
- U7 pad 3: unconnected-(U7-Pad3) -> Net-(R36-Pad2)
- U7 pad 4: Net-(R32-Pad2) -> VCC
- U8 pad 1: Net-(C17-Pad1) -> Net-(R46-Pad2)
- U8 pad 3: unconnected-(U8-Pad3) -> Net-(R52-Pad2)
- U8 pad 4: Net-(R33-Pad2) -> VCC
- U9 pad 1: Net-(C18-Pad1) -> Net-(R47-Pad2)
- U9 pad 3: unconnected-(U9-Pad3) -> Net-(R53-Pad2)
- U9 pad 4: Net-(R34-Pad2) -> VCC

Commit message: solenoid board
Parts:
- added D31: CD4148W, Diode_SMD:D_1206_3216Metric, F.Cu at (199.0, 101.3)
- added D33: CD4148W, Diode_SMD:D_1206_3216Metric, F.Cu at (227.3, 64.8)
- added D34: CD4148W, Diode_SMD:D_1206_3216Metric, F.Cu at (199.0, 104.7)
- added D35: CD4148W, Diode_SMD:D_1206_3216Metric, F.Cu at (216.3, 88.9)
- added D36: Signal, LED_SMD:LED_0805_2012Metric_Pad1.15x1.40mm_HandSolder, F.Cu at (204.2, 101.2)
- added D37: Signal, LED_SMD:LED_0805_2012Metric_Pad1.15x1.40mm_HandSolder, F.Cu at (198.6, 111.0)
- added D38: Signal, LED_SMD:LED_0805_2012Metric_Pad1.15x1.40mm_HandSolder, F.Cu at (221.5, 88.7)
- added D39: CD4148W, Diode_SMD:D_1206_3216Metric, F.Cu at (188.6, 120.3)
- added D40: CD4148W, Diode_SMD:D_1206_3216Metric, F.Cu at (199.0, 98.0)
- added D41: CD4148W, Diode_SMD:D_1206_3216Metric, F.Cu at (226.1, 69.8)
- added D42: CD4148W, Diode_SMD:D_1206_3216Metric, F.Cu at (204.7, 98.0)
- added D43: Signal, LED_SMD:LED_0805_2012Metric_Pad1.15x1.40mm_HandSolder, F.Cu at (209.9, 97.8)
- added D44: Signal, LED_SMD:LED_0805_2012Metric_Pad1.15x1.40mm_HandSolder, F.Cu at (204.2, 104.2)
- added D45: Signal, LED_SMD:LED_0805_2012Metric_Pad1.15x1.40mm_HandSolder, F.Cu at (198.6, 108.0)
- added D46: Signal, LED_SMD:LED_0805_2012Metric_Pad1.15x1.40mm_HandSolder, F.Cu at (215.9, 92.1)
- added J13: PORT, TerminalBlock_Phoenix:TerminalBlock_Phoenix_PT-1,5-3-3.5-H_1x03_P3.50mm_Horizontal, F.Cu at (143.8, 56.5)
- added J14: PORT, TerminalBlock_Phoenix:TerminalBlock_Phoenix_PT-1,5-3-3.5-H_1x03_P3.50mm_Horizontal, F.Cu at (157.8, 56.5)
- added J15: PORT, TerminalBlock_Phoenix:TerminalBlock_Phoenix_PT-1,5-3-3.5-H_1x03_P3.50mm_Horizontal, F.Cu at (171.8, 56.5)
- added J16: PORT, TerminalBlock_Phoenix:TerminalBlock_Phoenix_PT-1,5-3-3.5-H_1x03_P3.50mm_Horizontal, F.Cu at (185.7, 56.5)
- added J17: PORT, TerminalBlock_Phoenix:TerminalBlock_Phoenix_PT-1,5-3-3.5-H_1x03_P3.50mm_Horizontal, F.Cu at (199.7, 56.5)
- added J18: PORT, TerminalBlock_Phoenix:TerminalBlock_Phoenix_PT-1,5-3-3.5-H_1x03_P3.50mm_Horizontal, F.Cu at (213.7, 56.5)
- added J19: PORT, TerminalBlock_Phoenix:TerminalBlock_Phoenix_PT-1,5-3-3.5-H_1x03_P3.50mm_Horizontal, F.Cu at (227.6, 56.5)
- added R65: 4K7, Resistor_SMD:R_0805_2012Metric_Pad1.20x1.40mm_HandSolder, F.Cu at (236.2, 64.8)
- added R66: 4K7, Resistor_SMD:R_0805_2012Metric_Pad1.20x1.40mm_HandSolder, F.Cu at (224.2, 94.6)
- added R67: 4K7, Resistor_SMD:R_0805_2012Metric_Pad1.20x1.40mm_HandSolder, F.Cu at (198.5, 116.9)
- added R68: 10K, Resistor_SMD:R_0805_2012Metric_Pad1.20x1.40mm_HandSolder, F.Cu at (231.1, 64.8)
- added R69: 10K, Resistor_SMD:R_0805_2012Metric_Pad1.20x1.40mm_HandSolder, F.Cu at (231.0, 86.2)
- added R70: 10K, Resistor_SMD:R_0805_2012Metric_Pad1.20x1.40mm_HandSolder, F.Cu at (219.4, 95.1)
- added R71: 4K7, Resistor_SMD:R_0805_2012Metric_Pad1.20x1.40mm_HandSolder, F.Cu at (218.5, 101.0)
- added R72: 4K7, Resistor_SMD:R_0805_2012Metric_Pad1.20x1.40mm_HandSolder, F.Cu at (219.4, 98.0)
- added R73: 4K7, Resistor_SMD:R_0805_2012Metric_Pad1.20x1.40mm_HandSolder, F.Cu at (213.7, 101.0)
- added R74: 200R, Resistor_SMD:R_0805_2012Metric_Pad1.20x1.40mm_HandSolder, F.Cu at (214.6, 98.0)
- added R75: 200R, Resistor_SMD:R_0805_2012Metric_Pad1.20x1.40mm_HandSolder, F.Cu at (229.6, 83.3)
- added R76: 200R, Resistor_SMD:R_0805_2012Metric_Pad1.20x1.40mm_HandSolder, F.Cu at (193.8, 120.1)
- added R77: 4K7, Resistor_SMD:R_0805_2012Metric_Pad1.20x1.40mm_HandSolder, F.Cu at (198.6, 119.9)
- added R78: 4K7, Resistor_SMD:R_0805_2012Metric_Pad1.20x1.40mm_HandSolder, F.Cu at (226.3, 90.1)
- added R79: 4K7, Resistor_SMD:R_0805_2012Metric_Pad1.20x1.40mm_HandSolder, F.Cu at (214.7, 95.1)
- added R80: 4K7, Resistor_SMD:R_0805_2012Metric_Pad1.20x1.40mm_HandSolder, F.Cu at (204.2, 107.2)
- added R81: 10K, Resistor_SMD:R_0805_2012Metric_Pad1.20x1.40mm_HandSolder, F.Cu at (221.5, 91.7)
- added R82: 10K, Resistor_SMD:R_0805_2012Metric_Pad1.20x1.40mm_HandSolder, F.Cu at (209.0, 101.1)
- added R83: 10K, Resistor_SMD:R_0805_2012Metric_Pad1.20x1.40mm_HandSolder, F.Cu at (208.1, 110.2)
- added R84: 10K, Resistor_SMD:R_0805_2012Metric_Pad1.20x1.40mm_HandSolder, F.Cu at (203.3, 116.1)
- added R85: 4K7, Resistor_SMD:R_0805_2012Metric_Pad1.20x1.40mm_HandSolder, F.Cu at (233.7, 69.8)
- added R86: 4K7, Resistor_SMD:R_0805_2012Metric_Pad1.20x1.40mm_HandSolder, F.Cu at (208.9, 107.2)
- added R87: 4K7, Resistor_SMD:R_0805_2012Metric_Pad1.20x1.40mm_HandSolder, F.Cu at (226.3, 87.1)
- added R88: 4K7, Resistor_SMD:R_0805_2012Metric_Pad1.20x1.40mm_HandSolder, F.Cu at (209.0, 104.1)
- added R89: 200R, Resistor_SMD:R_0805_2012Metric_Pad1.20x1.40mm_HandSolder, F.Cu at (198.5, 114.0)
- added R90: 200R, Resistor_SMD:R_0805_2012Metric_Pad1.20x1.40mm_HandSolder, F.Cu at (203.3, 110.2)
- added R91: 200R, Resistor_SMD:R_0805_2012Metric_Pad1.20x1.40mm_HandSolder, F.Cu at (203.3, 113.1)
- added R92: 200R, Resistor_SMD:R_0805_2012Metric_Pad1.20x1.40mm_HandSolder, F.Cu at (213.7, 103.9)
- added U12: EL357N, PolyuRobotics:EL357N, F.Cu at (190.4, 131.4)
- added U13: EL357N, PolyuRobotics:EL357N, F.Cu at (165.6, 120.4)
- added U14: EL357N, PolyuRobotics:EL357N, F.Cu at (200.7, 77.5)
- added U15: EL357N, PolyuRobotics:EL357N, F.Cu at (208.3, 93.9)
- added U16: EL357N, PolyuRobotics:EL357N, F.Cu at (217.5, 84.8)
- added U17: EL357N, PolyuRobotics:EL357N, F.Cu at (173.7, 120.4)
- added U18: EL357N, PolyuRobotics:EL357N, F.Cu at (200.2, 93.9)
- J1, J10, J11, J3, J4, J5, J6, J7, J8, J9: value mx2.54 -> output; footprint Connector_PinHeader_2.54mm:PinHeader_1x02_P2.54mm_Vertical -> TerminalBlock_Phoenix:TerminalBlock_Phoenix_PT-1,5-2-5.0-H_1x02_P5.00mm_Horizontal
- J12: footprint TerminalBlock_Phoenix:TerminalBlock_Phoenix_MKDS-3-3-5.08_1x03_P5.08mm_Horizontal -> TerminalBlock_Phoenix:TerminalBlock_Phoenix_PT-1,5-3-3.5-H_1x03_P3.50mm_Horizontal
- Q10, Q2, Q3, Q4, Q5, Q6, Q7, Q8, Q9: value ~ -> AOD4184A
- R11, R12, R31, R32, R33, R49, R50, R51, R9: value ~ -> 10K
- U10, U2, U3, U4, U5, U6, U7, U8, U9: value ~ -> EL357N
- moved J1 169.9 mm to (232.4, 121.4), turned to 0 degrees
- moved Q2 156.8 mm to (190.8, 146.4)
- moved U8 146.2 mm to (181.8, 155.2)
- moved Q6 144.6 mm to (182.4, 146.4)
- moved Q10 141.3 mm to (174.1, 133.1)
- moved U10 140.6 mm to (207.1, 132.7)
- moved U9 138.7 mm to (207.1, 128.6)
- moved R9 134.7 mm to (210.2, 136.5)
- moved U5 134.6 mm to (165.6, 155.2)
- moved U7 134.3 mm to (199.0, 136.9)
- moved Q3 132.5 mm to (148.6, 135.5)
- moved U4 130.2 mm to (173.7, 155.2)
- moved R51 130.1 mm to (197.3, 140.7)
- moved J11 129.4 mm to (235.0, 104.9)
- moved R31 128.9 mm to (202.1, 143.6)
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
Commit message: test
Parts:
- added J20: 5V in, Connector_BarrelJack:BarrelJack_GCT_DCJ200-10-A_Horizontal, F.Cu at (245.1, 46.4)
- added J21: XT60-M, PolyuRobotics:XT60PW-M20, F.Cu at (121.2, 50.2)
- D13, D15, D16, D2, D22, D24, D25, D3, D5, D7, R13, R14, R15, R16, R17, R18, R19, R20, R21, R22, R23, R24, R34, R35, R36, R37, R38, R39, R40, R41, R42, R52, R53, R54, R55, R56, R57, R58, R59, R60: moved to B.Cu
- moved SW10 184.1 mm to (238.8, 76.2), turned to 90 degrees
- moved SW9 148.4 mm to (226.1, 76.2), turned to 90 degrees
- moved SW8 142.5 mm to (213.4, 76.2), turned to 90 degrees
- moved R60 141.8 mm to (242.6, 78.1), turned to 90 degrees
- moved D25 140.3 mm to (227.3, 90.8), turned to -90 degrees
- moved R53 138.1 mm to (229.9, 70.5), turned to -90 degrees
- moved R45 135.4 mm to (238.8, 67.9)
- moved D27 130.8 mm to (233.0, 69.2), turned to 90 degrees
- moved R54 129.1 mm to (242.6, 70.5), turned to -90 degrees
- moved R57 126.6 mm to (242.6, 74.3), turned to -90 degrees
- moved R46 124.7 mm to (216.5, 69.2), turned to 90 degrees
- moved R59 124.6 mm to (229.9, 78.1), turned to 90 degrees
- moved C7 123.2 mm to (200.7, 69.8)
- moved SW6 123.0 mm to (188.0, 76.2), turned to 90 degrees
- moved SW7 119.4 mm to (200.7, 76.2), turned to 90 degrees
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Connections:
- D13 pad 1: VCC -> +24V
- D15 pad 1: VCC -> +24V
- D16 pad 1: VCC -> +24V
- D2 pad 1: VCC -> +24V
- D22 pad 1: VCC -> +24V
- D24 pad 1: VCC -> +24V
- D25 pad 1: VCC -> +24V
- D3 pad 1: VCC -> +24V
- D5 pad 1: VCC -> +24V
- D7 pad 1: VCC -> +24V
- U1 pad 4: VCC -> +24V
- U10 pad 4: VCC -> +24V
- U2 pad 4: VCC -> +24V
- U3 pad 4: VCC -> +24V
- U4 pad 4: VCC -> +24V
- U5 pad 4: VCC -> +24V
- U6 pad 4: VCC -> +24V
- U7 pad 4: VCC -> +24V
- U8 pad 4: VCC -> +24V
- U9 pad 4: VCC -> +24V
Other:
- board outline added: 152.4 x 64.8 mm

Commit message: test
Parts:
- R10, R28, R29, R30, R46, R47, R48, R5, R7, R8: moved to B.Cu
- R13, R14, R15, R16, R34, R35, R36, R52, R53, R54: moved to F.Cu
- moved R16 13.5 mm to (156.2, 78.7), turned to 90 degrees
- moved R54 13.3 mm to (232.4, 79.1), turned to 90 degrees
- moved R14 13.1 mm to (118.1, 78.7), turned to 90 degrees
- moved R15 13.1 mm to (143.5, 78.7), turned to 90 degrees
- moved R34 13.1 mm to (168.9, 78.7), turned to 90 degrees
- moved R35 13.1 mm to (181.6, 78.7), turned to 90 degrees
- moved R53 13.1 mm to (219.7, 78.7), turned to 90 degrees
- moved R13 12.9 mm to (130.8, 78.7), turned to 90 degrees
- moved R36 12.9 mm to (194.3, 78.7), turned to 90 degrees
- moved R52 12.7 mm to (207.0, 78.7)
- moved D17 10.3 mm to (184.2, 79.4)
- moved D26 10.3 mm to (222.2, 79.4)
- moved D27 10.3 mm to (234.9, 79.4)
- moved J20 10.3 mm to (248.9, 55.9), turned to 180 degrees
- moved D18 10.2 mm to (196.8, 79.1), turned to 90 degrees
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Routing:
- net +24V: track 0.00 -> 307.5 mm
- net Net-(D20-Pad2): track 0.00 -> 22.0 mm
- net Net-(D10-Pad2): track 0.00 -> 21.6 mm
- net Net-(D21-Pad2): track 0.00 -> 21.6 mm
- net Net-(D30-Pad2): track 0.00 -> 21.6 mm
- net Net-(D28-Pad2): track 0.00 -> 21.6 mm
- net Net-(D9-Pad2): track 0.00 -> 21.6 mm
- net Net-(D29-Pad2): track 0.00 -> 21.6 mm
- net Net-(D12-Pad2): track 0.00 -> 21.6 mm
- net Net-(D19-Pad2): track 0.00 -> 21.6 mm
- net Net-(D11-Pad2): track 0.00 -> 20.8 mm
- net Net-(R13-Pad2): track 0.00 -> 15.3 mm, vias 0 -> 1
- net Net-(R35-Pad2): track 0.00 -> 15.2 mm, vias 0 -> 1
- net Net-(R54-Pad2): track 0.00 -> 14.9 mm, vias 0 -> 1
- net Net-(R16-Pad2): track 0.00 -> 14.8 mm, vias 0 -> 1
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Other:
- board size 152.4 x 64.8 mm -> 151.1 x 63.5 mm
