File: Power_connector/Power_connector.kicad_sch (KiCad schematic)
At the start: 64 parts, among them J1 XT60_F, J10 XT60_F, J11 XT60_F, J12 XT60_F, J13 XT60_F, J14 XT60_F, J2 XT60_Male, J3 XT60_F, J4 E_Stop, J5 XT60_F, J6 XT60_F, J7 XT60_F, J8 XT60_F, J9 XT60_F, Q1 IRFS7530, Q2 IRFS7530

Commit message: new shield
Parts:
- D10, D11, D12, D13, D14, D15, D3, D5, D7, D8, D9: footprint (none) -> LED_SMD:LED_0805_2012Metric
- D4: value (none) -> indicator; footprint (none) -> LED_SMD:LED_0805_2012Metric
- J2: footprint PolyuRobotics:XT60PW-M20 -> (none)
- R10, R11, R12, R13, R14, R15, R16, R17, R18, R2, R6: footprint (none) -> Resistor_SMD:R_0805_2012Metric
- R4: value (none) -> 10M; footprint (none) -> Resistor_SMD:R_0805_2012Metric
Changed lines of the file:
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@@
       (effects (font (size 1.27 1.27)) (justify right))
     )
-    (property "Footprint" "" (id 2) (at 125.095 74.295 90)
+    (property "Footprint" "LED_SMD:LED_0805_2012Metric" (id 2) (at 125.095 74.295 90)
       (effects (font (size 1.27 1.27)) hide)
     )
@@
     (property "Reference" "R10" (id 0) (at 207.645 67.945 90))
     (property "Value" "10M" (id 1) (at 208.28 69.85 90))
-    (property "Footprint" "" (id 2) (at 206.375 71.755 0)
+    (property "Footprint" "Resistor_SMD:R_0805_2012Metric" (id 2) (at 206.375 71.755 0)
       (effects (font (size 1.27 1.27)) hide)
     )
@@
       (effects (font (size 1.27 1.27)) (justify right))
     )
-    (property "Footprint" "" (id 2) (at 237.49 74.295 90)
+    (property "Footprint" "LED_SMD:LED_0805_2012Metric" (id 2) (at 237.49 74.295 90)
       (effects (font (size 1.27 1.27)) hide)
     )
@@
       (effects (font (size 1.27 1.27)) (justify right))
     )
-    (property "Footprint" "" (id 2) (at 208.915 100.33 90)
+    (property "Footprint" "LED_SMD:LED_0805_2012Metric" (id 2) (at 208.915 100.33 90)
       (effects (font (size 1.27 1.27)) hide)
     )
@@
       (effects (font (size 1.27 1.27)) (justify right))
     )
-    (property "Footprint" "" (id 2) (at 180.975 100.965 90)
+    (property "Footprint" "LED_SMD:LED_0805_2012Metric" (id 2) (at 180.975 100.965 90)
       (effects (font (size 1.27 1.27)) hide)
     )
@@
       (effects (font (size 1.27 1.27)) (justify right))
     )
-    (property "Footprint" "" (id 2) (at 125.095 100.33 90)
+    (property "Footprint" "LED_SMD:LED_0805_2012Metric" (id 2) (at 125.095 100.33 90)
       (effects (font (size 1.27 1.27)) hide)
     )
@@
       (effects (font (size 1.27 1.27)) (justify right))
     )
-    (property "Footprint" "" (id 2) (at 265.43 100.33 90)
+    (property "Footprint" "LED_SMD:LED_0805_2012Metric" (id 2) (at 265.43 100.33 90)
       (effects (font (size 1.27 1.27)) hide)
     )
@@
     (property "Reference" "R15" (id 0) (at 179.705 94.615 90))
     (property "Value" "10M" (id 1) (at 180.34 96.52 90))
-    (property "Footprint" "" (id 2) (at 178.435 98.425 0)
+    (property "Footprint" "Resistor_SMD:R_0805_2012Metric" (id 2) (at 178.435 98.425 0)
       (effects (font (size 1.27 1.27)) hide)
     )
@@
     (in_bom yes) (on_board yes)
     (property "Reference" "R4" (id 0) (at 148.59 67.945 90))
-    (property "Value" "" (id 1) (at 149.225 69.85 90))
-    (property "Footprint" "" (id 2) (at 147.32 71.755 0)
+    (property "Value" "10M" (id 1) (at 149.225 69.85 90))
+    (property "Footprint" "Resistor_SMD:R_0805_2012Metric" (id 2) (at 147.32 71.755 0)
       (effects (font (size 1.27 1.27)) hide)
     )
@@
     (property "Reference" "R6" (id 0) (at 179.705 68.58 90))
     (property "Value" "10M" (id 1) (at 180.34 70.485 90))
-    (property "Footprint" "" (id 2) (at 178.435 72.39 0)
+    (property "Footprint" "Resistor_SMD:R_0805_2012Metric" (id 2) (at 178.435 72.39 0)
       (effects (font (size 1.27 1.27)) hide)
     )
@@
     (property "Reference" "J2" (id 0) (at 121.92 24.765 0))
     (property "Value" "XT60_Male" (id 1) (at 114.935 29.845 0))
-    (property "Footprint" "PolyuRobotics:XT60PW-M20" (id 2) (at 121.92 30.48 0)
+    (property "Footprint" "" (id 2) (at 121.92 30.48 0)
       (effects (font (size 1.27 1.27)) hide)
     )
@@
     (property "Reference" "R12" (id 0) (at 264.16 67.945 90))
     (property "Value" "10M" (id 1) (at 264.795 69.85 90))
-    (property "Footprint" "" (id 2) (at 262.89 71.755 0)
+    (property "Footprint" "Resistor_SMD:R_0805_2012Metric" (id 2) (at 262.89 71.755 0)
       (effects (font (size 1.27 1.27)) hide)
     )
@@
     (property "Reference" "R17" (id 0) (at 236.22 93.98 90))
     (property "Value" "10M" (id 1) (at 236.855 95.885 90))
-    (property "Footprint" "" (id 2) (at 234.95 97.79 0)
+    (property "Footprint" "Resistor_SMD:R_0805_2012Metric" (id 2) (at 234.95 97.79 0)
       (effects (font (size 1.27 1.27)) hide)
     )
@@
       (effects (font (size 1.27 1.27)) (justify right))
     )
-    (property "Value" "" (id 1) (at 152.4 75.5014 90)
-      (effects (font (size 1.27 1.27)) (justify right))
-    )
-    (property "Footprint" "" (id 2) (at 149.86 74.295 90)
+    (property "Value" "indicator" (id 1) (at 152.4 75.5014 90)
+      (effects (font (size 1.27 1.27)) (justify right))
+    )
+    (property "Footprint" "LED_SMD:LED_0805_2012Metric" (id 2) (at 149.86 74.295 90)
       (effects (font (size 1.27 1.27)) hide)
     )
@@
     (property "Reference" "R16" (id 0) (at 207.645 93.98 90))
     (property "Value" "10M" (id 1) (at 208.28 95.885 90))
-    (property "Footprint" "" (id 2) (at 206.375 97.79 0)
+    (property "Footprint" "Resistor_SMD:R_0805_2012Metric" (id 2) (at 206.375 97.79 0)
       (effects (font (size 1.27 1.27)) hide)
     )
@@
     (property "Reference" "R11" (id 0) (at 236.22 67.945 90))
     (property "Value" "10M" (id 1) (at 236.855 69.85 90))
-    (property "Footprint" "" (id 2) (at 234.95 71.755 0)
+    (property "Footprint" "Resistor_SMD:R_0805_2012Metric" (id 2) (at 234.95 71.755 0)
       (effects (font (size 1.27 1.27)) hide)
     )
@@
     (property "Reference" "R13" (id 0) (at 123.825 93.98 90))
     (property "Value" "10M" (id 1) (at 124.46 95.885 90))
-    (property "Footprint" "" (id 2) (at 122.555 97.79 0)
+    (property "Footprint" "Resistor_SMD:R_0805_2012Metric" (id 2) (at 122.555 97.79 0)
       (effects (font (size 1.27 1.27)) hide)
     )
@@
     (property "Reference" "R14" (id 0) (at 148.59 93.98 90))
     (property "Value" "10M" (id 1) (at 149.225 95.885 90))
-    (property "Footprint" "" (id 2) (at 147.32 97.79 0)
+    (property "Footprint" "Resistor_SMD:R_0805_2012Metric" (id 2) (at 147.32 97.79 0)
       (effects (font (size 1.27 1.27)) hide)
     )
@@
       (effects (font (size 1.27 1.27)) (justify right))
     )
-    (property "Footprint" "" (id 2) (at 149.86 100.33 90)
+    (property "Footprint" "LED_SMD:LED_0805_2012Metric" (id 2) (at 149.86 100.33 90)
       (effects (font (size 1.27 1.27)) hide)
     )
@@
       (effects (font (size 1.27 1.27)) (justify right))
     )
-    (property "Footprint" "" (id 2) (at 237.49 100.33 90)
+    (property "Footprint" "LED_SMD:LED_0805_2012Metric" (id 2) (at 237.49 100.33 90)
       (effects (font (size 1.27 1.27)) hide)
     )
@@
       (effects (font (size 1.27 1.27)) (justify right))
     )
-    (property "Footprint" "" (id 2) (at 180.975 74.93 90)
+    (property "Footprint" "LED_SMD:LED_0805_2012Metric" (id 2) (at 180.975 74.93 90)
       (effects (font (size 1.27 1.27)) hide)
     )
@@
     (property "Reference" "R2" (id 0) (at 123.825 67.945 90))
     (property "Value" "10M" (id 1) (at 124.46 69.85 90))
-    (property "Footprint" "" (id 2) (at 122.555 71.755 0)
+    (property "Footprint" "Resistor_SMD:R_0805_2012Metric" (id 2) (at 122.555 71.755 0)
       (effects (font (size 1.27 1.27)) hide)
     )
@@
       (effects (font (size 1.27 1.27)) (justify right))
     )
-    (property "Footprint" "" (id 2) (at 208.915 74.295 90)
+    (property "Footprint" "LED_SMD:LED_0805_2012Metric" (id 2) (at 208.915 74.295 90)
       (effects (font (size 1.27 1.27)) hide)
     )
@@
       (effects (font (size 1.27 1.27)) (justify right))
     )
-    (property "Footprint" "" (id 2) (at 265.43 74.295 90)
+    (property "Footprint" "LED_SMD:LED_0805_2012Metric" (id 2) (at 265.43 74.295 90)
       (effects (font (size 1.27 1.27)) hide)
     )
@@
     (property "Reference" "R18" (id 0) (at 264.16 93.98 90))
     (property "Value" "10M" (id 1) (at 264.795 95.885 90))
-    (property "Footprint" "" (id 2) (at 262.89 97.79 0)
+    (property "Footprint" "Resistor_SMD:R_0805_2012Metric" (id 2) (at 262.89 97.79 0)
       (effects (font (size 1.27 1.27)) hide)
     )
@@
     )
     (path "/65dc78f6-b655-4175-8e85-57065401ab91"
-      (reference "J2") (unit 1) (value "XT60_Male") (footprint "PolyuRobotics:XT60PW-M20")
+      (reference "J2") (unit 1) (value "XT60_Male") (footprint "Connector_AMASS:AMASS_XT60-M_1x02_P7.20mm_Vertical")
     )
     (path "/e8517f32-f137-444f-999c-11cefcaac76f"
