File: ESP32_CAN_TEST/ESP32_CAN_TEST.kicad_pcb (KiCad board)
At the start: 2 copper layers, 45.7 x 45.7 mm, 25 parts, among them J1 5V in, J2 Conn_01x05, J3 Molex_2x2, J4 Conn_01x05, J5 i2C, J6 UART, SW1 EN, SW2 EN, U1 AMS1117, U2 ESP32-WROOM-32, U3 SN65HVD230

Commit message: update
Parts:
- moved SW2 31.1 mm to (134.1, 79.2), turned to -90 degrees
- moved C3 28.0 mm to (114.3, 83.3), turned to 180 degrees
- moved U1 20.7 mm to (113.8, 78.2), turned to 180 degrees
- moved C5 19.8 mm to (114.9, 73.2), turned to 0 degrees
- moved R3 11.8 mm to (133.6, 69.6), turned to 0 degrees
- moved C6 11.6 mm to (139.3, 47.8)
- moved C7 11.2 mm to (133.6, 71.6), turned to 180 degrees
- moved JP1 7.33 mm to (138.7, 74.7), turned to 180 degrees
- moved J5 6.89 mm to (118.6, 47.7)
- moved J3 4.52 mm to (140.3, 68.6), turned to 90 degrees
- moved R4 3.61 mm to (138.7, 77.2), turned to 0 degrees
- moved D2 2.09 mm to (139.2, 79.2), turned to 90 degrees
- moved J2 1.53 mm to (144.8, 59.4)
- moved J4 0.51 mm to (127.5, 43.2)
- moved U3 0.51 mm to (134.1, 53.3), turned to -90 degrees
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Routing:
- net +3V3: track 0.00 -> 82.2 mm, vias 0 -> 1
- net +5V: track 0.00 -> 59.2 mm
- net Net-(C4-Pad1): track 0.00 -> 35.9 mm
- net Net-(C7-Pad2): track 0.00 -> 30.2 mm, vias 0 -> 2
- net /IO14: track 0.00 -> 29.5 mm, vias 0 -> 3
- net /IO13: track 0.00 -> 23.8 mm, vias 0 -> 1
- net /CAN_TX: track 0.00 -> 21.9 mm, vias 0 -> 2
- net /IO16: track 0.00 -> 21.7 mm, vias 0 -> 1
- net /IO17: track 0.00 -> 18.5 mm, vias 0 -> 1
- net /IO18: track 0.00 -> 18.2 mm
- net /CAN_RX: track 0.00 -> 16.5 mm
- net /SDA: track 0.00 -> 14.6 mm, vias 0 -> 1
- net /SCL: track 0.00 -> 12.7 mm, vias 0 -> 1
- net /RXD: track 0.00 -> 9.68 mm
- net /TXD: track 0.00 -> 9.46 mm
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
Commit message: update
Parts:
- added G***: LOGO, PolyuRobotics:Club_logo, F.Cu at (133.1, 58.4)
- added J7: GH1.25, Connector_JST:JST_GH_BM02B-GHS-TBT_1x02-1MP_P1.25mm_Vertical, F.Cu at (143.8, 77.2)
- added J8: JST_2.54, Connector_JST:JST_XH_B2B-XH-AM_1x02_P2.50mm_Vertical, F.Cu at (136.1, 83.0)
- added Q1: 2N7002, Package_TO_SOT_SMD:SOT-23, B.Cu at (122.4, 63.5)
- added Q2: 2N7002, Package_TO_SOT_SMD:SOT-23, B.Cu at (122.4, 59.4)
- added R5: 10K, Resistor_SMD:R_0805_2012Metric, B.Cu at (118.4, 63.6)
- added R6: 10K, Resistor_SMD:R_0805_2012Metric, B.Cu at (118.4, 59.5)
- added R7: 10K, Resistor_SMD:R_0805_2012Metric, B.Cu at (127.0, 65.0)
- added R8: 10K, Resistor_SMD:R_0805_2012Metric, B.Cu at (127.0, 57.9)
- C6: value 0.1uf -> 100nF; footprint Capacitor_SMD:C_0805_2012Metric -> Capacitor_SMD:C_0805_2012Metric_Pad1.18x1.45mm_HandSolder; moved to B.Cu
- D2: footprint Button_Switch_SMD:SW_SPST_FSMSM -> LED_SMD:LED_0805_2012Metric
- J2: value Conn_01x05 -> Encoder_1
- J4: value Conn_01x05 -> Encoder2
- SW1, SW2: footprint Button_Switch_SMD:SW_SPST_FSMSM -> Button_Switch_SMD:SW_SPST_TL3342
- U3: value SN65HVD230 -> TJA1050; moved to B.Cu
- moved D1 24.1 mm to (134.1, 70.1), turned to -90 degrees
- moved R1 19.8 mm to (134.1, 74.2)
- moved C4 16.1 mm to (123.4, 76.2), turned to 0 degrees
- moved U1 14.8 mm to (128.5, 79.2), turned to 90 degrees
- moved SW1 12.6 mm to (124.0, 81.8), turned to -90 degrees
- moved D2 11.0 mm to (130.0, 73.2), turned to -90 degrees
- moved J1 10.1 mm to (111.8, 81.1)
- moved J2 9.98 mm to (142.2, 49.8), turned to 0 degrees
- moved J5 9.77 mm to (110.0, 43.2)
- moved C6 9.51 mm to (136.7, 56.9)
- moved C5 9.27 mm to (122.9, 77.7), turned to -90 degrees
- moved U3 8.19 mm to (133.1, 61.5), turned to 0 degrees
- moved C3 7.64 mm to (121.9, 83.8), turned to 90 degrees
- moved R3 7.07 mm to (127.5, 73.2), turned to -90 degrees
- moved C7 6.88 mm to (128.5, 76.2), turned to 0 degrees
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Connections:
- C6 pad 1: +3V3 -> +5V
- J2 pad 3: /IO14 -> /IO13
- J2 pad 4: /IO13 -> /IO14
- U3 pad 1: /CAN_TX -> Net-(Q1-Pad3)
- U3 pad 3: +3V3 -> +5V
- U3 pad 4: /CAN_RX -> Net-(Q2-Pad3)
Routing:
- net +5V: track 59.2 -> 118.2 mm
- net Net-(C7-Pad2): track 30.2 -> 72.4 mm, vias 2 -> 0
- net /CANL-: track 0.00 -> 32.5 mm
- net /CANH+: track 0.00 -> 29.4 mm
- net /IO15: track 0.00 -> 17.4 mm
- net Net-(C4-Pad1): track 35.9 -> 24.8 mm
- net Net-(Q1-Pad3): track 0.00 -> 7.81 mm
- net Net-(Q2-Pad3): track 0.00 -> 7.81 mm
- net /CAN_RX: track 16.5 -> 9.61 mm, vias 0 -> 1
- net /CAN_TX: track 21.9 -> 15.4 mm, vias 2 -> 1
- net /IO16: track 21.7 -> 15.6 mm, vias 1 -> 0
- net Net-(D2-Pad2): track 8.15 -> 2.57 mm
- net +3V3: track 82.2 -> 77.1 mm
- net /TXD: track 9.46 -> 4.89 mm
- net /RXD: track 9.68 -> 5.11 mm
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- added copper zone on B.Cu, net GND
- added copper zone on F.Cu, net GND
Other:
- board text added: "3.3"
- board text added: "5V"
- board text added: "5V A B z GND"
- board text added: "5V_IN"
- board text added: "ESP32_MiniBrain By SamsonChau"
- board text added: "Encoder_1"
- board text added: "GND"
- board text added: "I2C"
- board text added: "Rx"
- board text added: "SCL"
- board text added: "SDA"
- board text added: "Tx"
- board text added: "UART"

Commit message: change footprint
Parts:
- moved R7 0.61 mm to (127.0, 64.4)
- moved R8 0.51 mm to (127.0, 58.4)
Connections:
- U2 pad 26: /CAN_TX -> /CAN_RX
- U2 pad 29: /CAN_RX -> /CAN_TX
Routing:
- net Net-(Q1-Pad3): track 7.81 -> 5.91 mm
- net /CAN_TX: track 15.4 -> 14.2 mm
- net +5V: track 118.2 -> 119.3 mm
- net /CAN_RX: track 9.61 -> 10.6 mm
Changed lines of the file:
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@@
       (net 5 "Net-(C7-Pad2)") (pinfunction "IO0") (pintype "bidirectional"))
     (pad "26" smd rect (at 8.5 6.985 90) (size 2 0.9) (layers "F.Cu" "F.Paste" "F.Mask")
-      (net 40 "/CAN_TX") (pinfunction "IO4") (pintype "bidirectional"))
+      (net 41 "/CAN_RX") (pinfunction "IO4") (pintype "bidirectional"))
     (pad "27" smd rect (at 8.5 5.715 90) (size 2 0.9) (layers "F.Cu" "F.Paste" "F.Mask")
       (net 17 "/IO16") (pinfunction "IO16") (pintype "bidirectional"))
@@
       (net 16 "/IO17") (pinfunction "IO17") (pintype "bidirectional"))
     (pad "29" smd rect (at 8.5 3.175 90) (size 2 0.9) (layers "F.Cu" "F.Paste" "F.Mask")
-      (net 41 "/CAN_RX") (pinfunction "IO5") (pintype "bidirectional"))
+      (net 40 "/CAN_TX") (pinfunction "IO5") (pintype "bidirectional"))
     (pad "30" smd rect (at 8.5 1.905 90) (size 2 0.9) (layers "F.Cu" "F.Paste" "F.Mask")
       (net 15 "/IO18") (pinfunction "IO18") (pintype "bidirectional"))
@@
   )
   (footprint "Resistor_SMD:R_0805_2012Metric" (layer "B.Cu")
-    (at 127 65.024 90)
+    (at 127 64.4125 90)
     (descr "Resistor SMD 0805 (2012 Metric), square (rectangular) end terminal, IPC_7351 nominal, (Body size source: IPC-SM-782 page 72, https://www.pcb-3d.com/wordpress/wp-content/uploads/ipc-sm-782a_amendment_1_and_2.pdf), generated with kicad-footprint-generator")
     (tags "resistor")
@@
   )
   (footprint "Resistor_SMD:R_0805_2012Metric" (layer "B.Cu")
-    (at 127 57.912 -90)
+    (at 127 58.42 -90)
     (descr "Resistor SMD 0805 (2012 Metric), square (rectangular) end terminal, IPC_7351 nominal, (Body size source: IPC-SM-782 page 72, https://www.pcb-3d.com/wordpress/wp-content/uploads/ipc-sm-782a_amendment_1_and_2.pdf), generated with kicad-footprint-generator")
     (tags "resistor")
@@
   (segment (start 134.112 75.152) (end 134.112 81.28) (width 1) (layer "F.Cu") (net 3))
   (segment (start 127.508 47.244) (end 130.048 49.784) (width 1) (layer "B.Cu") (net 3))
+  (segment (start 127 65.9365) (end 127 65.325) (width 0.5) (layer "B.Cu") (net 3))
   (segment (start 133.096 55.372) (end 138.684 49.784) (width 1.5) (layer "B.Cu") (net 3))
   (segment (start 132.9925 56.9995) (end 133.096 56.896) (width 0.5) (layer "B.Cu") (net 3))
@@
   (segment (start 133.096 66.548) (end 133.096 60.96) (width 1.5) (layer "B.Cu") (net 3))
   (segment (start 126.224 81.04) (end 126.224 82.398) (width 1.5) (layer "B.Cu") (net 3))
+  (segment (start 127 57.5075) (end 127 56.9995) (width 0.35) (layer "B.Cu") (net 3))
   (segment (start 132.969 60.833) (end 133.096 60.96) (width 0.5) (layer "B.Cu") (net 3))
   (segment (start 135.128 75.692) (end 131.572 79.248) (width 1.5) (layer "B.Cu") (net 3))
@@
   (segment (start 125.603 69.46) (end 125.603 70.247) (width 0.35) (layer "F.Cu") (net 23))
   (segment (start 125.603 70.247) (end 127.508 72.152) (width 0.35) (layer "F.Cu") (net 23))
-  (segment (start 124.333 57.023) (end 119.888 61.468) (width 0.5) (layer "F.Cu") (net 40))
-  (segment (start 124.333 52.46) (end 124.333 57.023) (width 0.5) (layer "F.Cu") (net 40))
-  (via (at 119.888 61.468) (size 0.8) (drill 0.4) (layers "F.Cu" "B.Cu") (net 40))
-  (segment (start 119.888 61.468) (end 119.888 61.976) (width 0.5) (layer "B.Cu") (net 40))
-  (segment (start 119.888 61.976) (end 120.462 62.55) (width 0.5) (layer "B.Cu") (net 40))
+  (segment (start 120.523 55.245) (end 119.888 55.88) (width 0.35) (layer "F.Cu") (net 40))
+  (segment (start 119.888 60.96) (end 120.396 61.468) (width 0.35) (layer "F.Cu") (net 40))
+  (segment (start 119.888 55.88) (end 119.888 60.96) (width 0.35) (layer "F.Cu") (net 40))
+  (segment (start 120.523 52.46) (end 120.523 55.245) (width 0.35) (layer "F.Cu") (net 40))
+  (via (at 120.396 61.468) (size 0.8) (drill 0.4) (layers "F.Cu" "B.Cu") (net 40))
+  (segment (start 120.4085 61.468) (end 121.4905 62.55) (width 0.35) (layer "B.Cu") (net 40))
+  (segment (start 120.396 61.468) (end 120.4085 61.468) (width 0.35) (layer "B.Cu") (net 40))
   (segment (start 118.505 62.55) (end 118.364 62.691) (width 0.5) (layer "B.Cu") (net 40))
   (segment (start 120.462 62.55) (end 118.505 62.55) (width 0.5) (layer "B.Cu") (net 40))
   (segment (start 120.462 62.55) (end 121.4905 62.55) (width 0.5) (layer "B.Cu") (net 40))
-  (segment (start 120.523 52.46) (end 120.523 54.483) (width 0.35) (layer "F.Cu") (net 41))
-  (segment (start 120.523 54.483) (end 120.904 54.864) (width 0.35) (layer "F.Cu") (net 41))
-  (via (at 120.904 54.864) (size 0.8) (drill 0.4) (layers "F.Cu" "B.Cu") (net 41))
-  (segment (start 120.904 57.8995) (end 121.4905 58.486) (width 0.35) (layer "B.Cu") (net 41))
+  (segment (start 124.473489 52.600489) (end 124.473489 53.326511) (width 0.35) (layer "F.Cu") (net 41))
+  (segment (start 124.333 52.46) (end 124.473489 52.600489) (width 0.35) (layer "F.Cu") (net 41))
+  (segment (start 124.473489 53.326511) (end 121.412 56.388) (width 0.35) (layer "F.Cu") (net 41))
+  (via (at 121.412 56.388) (size 0.8) (drill 0.4) (layers "F.Cu" "B.Cu") (net 41))
+  (segment (start 121.412 58.4075) (end 121.4905 58.486) (width 0.35) (layer "B.Cu") (net 41))
   (segment (start 118.505 58.486) (end 118.364 58.627) (width 0.35) (layer "B.Cu") (net 41))
-  (segment (start 120.904 54.864) (end 120.904 57.8995) (width 0.35) (layer "B.Cu") (net 41))
+  (segment (start 121.412 56.388) (end 121.412 58.4075) (width 0.35) (layer "B.Cu") (net 41))
   (segment (start 121.4905 58.486) (end 118.505 58.486) (width 0.35) (layer "B.Cu") (net 41))
   (segment (start 123.3655 63.5) (end 126.3885 63.5) (width 0.35) (layer "B.Cu") (net 46))
   (segment (start 130.621 63.373) (end 127.7385 63.373) (width 0.35) (layer "B.Cu") (net 46))
-  (segment (start 127.7385 63.373) (end 127 64.1115) (width 0.35) (layer "B.Cu") (net 46))
-  (segment (start 126.3885 63.5) (end 127 64.1115) (width 0.35) (layer "B.Cu") (net 46))
-  (segment (start 126.3885 59.436) (end 127 58.8245) (width 0.35) (layer "B.Cu") (net 47))
-  (segment (start 123.3655 59.436) (end 126.3885 59.436) (width 0.35) (layer "B.Cu") (net 47))
-  (segment (start 127.7385 59.563) (end 127 58.8245) (width 0.35) (layer "B.Cu") (net 47))
-  (segment (start 130.621 59.563) (end 127.7385 59.563) (width 0.35) (layer "B.Cu") (net 47))
+  (segment (start 130.621 59.563) (end 127.2305 59.563) (width 0.35) (layer "B.Cu") (net 47))
+  (segment (start 126.0875 59.3325) (end 125.984 59.436) (width 0.35) (layer "B.Cu") (net 47))
+  (segment (start 123.3655 59.436) (end 125.984 59.436) (width 0.35) (layer "B.Cu") (net 47))
+  (segment (start 127.2305 59.563) (end 127 59.3325) (width 0.35) (layer "B.Cu") (net 47))
+  (segment (start 127 59.3325) (end 126.0875 59.3325) (width 0.35) (layer "B.Cu") (net 47))
+  (segment (start 125.984 59.436) (end 126.3885 59.436) (width 0.35) (layer "B.Cu") (net 47))
   (zone (net 2) (net_name "GND") (layers F&B.Cu) (hatch edge 0.508)
     (connect_pads yes (clearance 0.508))

Commit message: ESP,Power board update
Parts:
- removed G***: LOGO, PolyuRobotics:Club_logo
- added C10: 0.1u, Capacitor_SMD:C_0805_2012Metric, F.Cu at (133.1, 59.7)
- added C8: 100nF, Capacitor_SMD:C_0805_2012Metric, B.Cu at (125.2, 68.3)
- added C9: 16V 22UF, Capacitor_SMD:CP_Elec_6.3x7.7, B.Cu at (115.3, 65.3)
- added D3: SMBJ24CA, Diode_SMD:D_SMB, B.Cu at (135.9, 77.2)
- added D4: SS34, Diode_SMD:D_SMB, B.Cu at (131.1, 77.2)
- added D5: SS34, Diode_SMD:D_SMB, B.Cu at (125.2, 51.8)
- added L1: 22uH, Inductor_SMD:L_Vishay_IHLP-1616, B.Cu at (125.0, 56.6)
- added Q3: 2N7002, Package_TO_SOT_SMD:SOT-23, F.Cu at (132.6, 52.6)
- added Q4: 2N7002, Package_TO_SOT_SMD:SOT-23, B.Cu at (127.3, 46.7)
- added Q5: 2N7002, Package_TO_SOT_SMD:SOT-23, F.Cu at (125.7, 50.5)
- added Q6: 2N7002, Package_TO_SOT_SMD:SOT-23, B.Cu at (137.9, 50.2)
- added R10: 10K, Resistor_SMD:R_0805_2012Metric, F.Cu at (129.3, 52.4)
- added R11: 10K, Resistor_SMD:R_0805_2012Metric, F.Cu at (128.5, 56.9)
- added R12: 10K, Resistor_SMD:R_0805_2012Metric, F.Cu at (140.3, 46.7)
- added R13: 10K, Resistor_SMD:R_0805_2012Metric, F.Cu at (135.6, 51.8)
- added R14: 10K, Resistor_SMD:R_0805_2012Metric, B.Cu at (123.7, 46.9)
- added R15: 10K, Resistor_SMD:R_0805_2012Metric, F.Cu at (125.8, 53.7)
- added R16: 10K, Resistor_SMD:R_0805_2012Metric, B.Cu at (137.8, 46.9)
- added R17: 10K, Resistor_SMD:R_0805_2012Metric, B.Cu at (130.3, 47.5)
- added R18: 10K, Resistor_SMD:R_0805_2012Metric, F.Cu at (124.7, 46.5)
- added R19: 10K, Resistor_SMD:R_0805_2012Metric, B.Cu at (136.8, 53.3)
- added R9: 10K, Resistor_SMD:R_0805_2012Metric, F.Cu at (133.7, 47.5)
- added U4: SN65HVD230, Package_SO:SOIC-8_3.9x4.9mm_P1.27mm, F.Cu at (133.0, 65.3)
- C6: value 100nF -> 50V 10uF; footprint Capacitor_SMD:C_0805_2012Metric_Pad1.18x1.45mm_HandSolder -> Capacitor_SMD:CP_Elec_6.3x7.7
- J1: value 5V in -> XT60; footprint TerminalBlock_Phoenix:TerminalBlock_Phoenix_MKDS-1,5-2_1x02_P5.00mm_Horizontal -> Connector_AMASS:AMASS_XT60-M_1x02_P7.20mm_Vertical
- J8: value JST_2.54 -> Jack-DC; footprint Connector_JST:JST_XH_B2B-XH-AM_1x02_P2.50mm_Vertical -> Connector_BarrelJack:BarrelJack_Horizontal
- Q1, Q2, R8: moved to F.Cu
- R5: value 10K -> 300K
- R6: value 10K -> 5.1k
- R7: value 10K -> 27K
- U3: value TJA1050 -> AOZ1282CI; footprint Package_SO:SOIC-8_3.9x4.9mm_P1.27mm -> Package_TO_SOT_SMD:SOT-23-6
- moved J5 34.8 mm to (140.5, 59.9), turned to 180 degrees
- moved D1 29.9 mm to (104.4, 73.7), turned to 180 degrees
- moved R1 29.8 mm to (104.4, 71.4), turned to 180 degrees
- moved J8 26.1 mm to (112.3, 72.5)
- moved U1 25.4 mm to (106.9, 65.8), turned to 180 degrees
- moved C5 24.4 mm to (105.4, 60.7), turned to 0 degrees
- moved Q2 19.0 mm to (137.2, 47.5)
- moved C3 18.5 mm to (108.0, 71.6), turned to -90 degrees
- moved R2 15.1 mm to (135.4, 72.4)
- moved D2 13.8 mm to (116.8, 69.6), turned to 0 degrees
- moved SW1 13.0 mm to (135.9, 76.7), turned to 0 degrees
- moved J1 12.2 mm to (124.0, 81.6), turned to 90 degrees
- moved C6 12.1 mm to (133.3, 68.6), turned to 90 degrees
- moved R5 10.2 mm to (128.5, 64.3)
- moved U3 8.94 mm to (125.1, 65.5)
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Connections:
- C6 pad 1: +5V -> Net-(C6-Pad1)
- J1 pad 1: +5V -> GND
- J1 pad 2: GND -> +24V
- J2 pad 2: /IO15 -> Net-(J2-Pad2)
- J2 pad 3: /IO13 -> Net-(J2-Pad3)
- J2 pad 4: /IO14 -> Net-(J2-Pad4)
- J4 pad 2: /IO18 -> Net-(J4-Pad2)
- J4 pad 3: /IO17 -> Net-(J4-Pad3)
- J4 pad 4: /IO16 -> Net-(J4-Pad4)
- J7 pad 1: /CANH+ -> /CANL-
- J7 pad 2: /CANL- -> /CANH+
- Q1 pad 2: /CAN_TX -> /IO15
- Q1 pad 3: Net-(Q1-Pad3) -> Net-(J2-Pad2)
- Q2 pad 2: /CAN_RX -> /IO13
- Q2 pad 3: Net-(Q2-Pad3) -> Net-(J2-Pad3)
- R5 pad 1: +3V3 -> Net-(C6-Pad1)
- R5 pad 2: /CAN_TX -> Net-(R5-Pad2)
- R6 pad 1: +3V3 -> Net-(R6-Pad1)
- R6 pad 2: /CAN_RX -> GND
- R7 pad 1: +5V -> Net-(R6-Pad1)
- R7 pad 2: Net-(Q1-Pad3) -> +5V
- R8 pad 1: +5V -> +3V3
- R8 pad 2: Net-(Q2-Pad3) -> /IO15
- U3 pad 1: Net-(Q1-Pad3) -> Net-(C8-Pad1)
- U3 pad 3: +5V -> Net-(R6-Pad1)
- U3 pad 4: Net-(Q2-Pad3) -> Net-(R5-Pad2)
- U3 pad 5: unconnected-(U3-Pad5) -> Net-(C6-Pad1)
- U3 pad 6: /CANH+ -> Net-(C8-Pad2)
Routing:
- net +3V3: track 77.1 -> 141.5 mm, vias 1 -> 6
- net Net-(C4-Pad1): track 24.8 -> 66.7 mm
- net /SCL: track 14.9 -> 53.5 mm
- net Net-(C7-Pad2): track 72.4 -> 102.8 mm, vias 0 -> 2
- net +5V: track 119.3 -> 89.0 mm, vias 0 -> 2
- net /SDA: track 17.2 -> 47.4 mm
- net /IO13: track 22.1 -> 50.2 mm, vias 0 -> 2
- net Net-(J2-Pad2): track 0.00 -> 27.4 mm, vias 0 -> 1
- net /CAN_TX: track 14.2 -> 35.7 mm, vias 1 -> 0
- net Net-(C8-Pad2): track 0.00 -> 18.2 mm
- net Net-(J2-Pad4): track 0.00 -> 17.2 mm
- net /IO16: track 15.6 -> 31.2 mm, vias 0 -> 1
- net Net-(C6-Pad1): track 0.00 -> 15.2 mm
- net /IO15: track 17.4 -> 2.21 mm
- net /CANL-: track 32.5 -> 17.5 mm
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Other:
- board text removed: "3.3"
- board text removed: "5V"
- board text removed: "5V A B z GND"
- board text removed: "5V_IN"
- board text removed: "ESP32_MiniBrain By SamsonChau"
- board text removed: "Encoder_1"
- board text removed: "GND"
- board text removed: "I2C"
- board text removed: "Rx"
- board text removed: "SCL"
- board text removed: "SDA"
- board text removed: "Tx"
- board text removed: "UART"
