File: ESP32_CAN_TEST/ESP32_CAN_TEST.kicad_sch (KiCad schematic)
At the start: 35 parts, among them J1 XT60, J2 Encoder_1, J3 Molex_2x2, J4 Encoder2, J5 Molex_2x2, J6 UART, J7 GH1.25, SW1 EN, SW2 EN, U1 AMS1117, U2 ESP32-WROOM-32, U3 MP1584, U4 TJA1051T, U5 TJA1051T

Commit message: update
Parts:
- added D5: user, LED_SMD:LED_0805_2012Metric, symbol Device:LED_Small
- added JP3: 3.3v, Jumper:SolderJumper-2_P1.3mm_Open_Pad1.0x1.5mm, symbol Jumper:SolderJumper_2_Open
- added JP4: 5v, Jumper:SolderJumper-2_P1.3mm_Open_Pad1.0x1.5mm, symbol Jumper:SolderJumper_2_Open
- added R5: 1K, Resistor_SMD:R_0805_2012Metric_Pad1.20x1.40mm_HandSolder, symbol Device:R_Small
- J1: footprint (none) -> Connector_AMASS:AMASS_XT30U-M_1x02_P5.0mm_Vertical
Connections:
- net +5V: now also JP4.2 (B); no longer J2.1 (Pin_1), J4.1 (Pin_1)
- net GND: now also D5.1 (K)
- net IO23: no longer names the net of U2.37 (IO23)
- net IO23: now also R5.1
- new net: J2.1 (Pin_1), J4.1 (Pin_1), JP3.1 (A), JP4.1 (A)
- new net: D5.2 (A), R5.2
- new net +3.3V: JP3.2 (B)
Other:
- note removed: "Encoder"
