File: arduino_can_bus_shield/arduino_can_bus_shield.kicad_sch (KiCad schematic)
At the start: 8 parts, among them P1 Power, P2 Analog, P3 Digital, P4 Digital, P5 CONN_01X01, P6 CONN_01X01, P7 CONN_01X01, P8 CONN_01X01

Commit message: ohh
Parts:
- added C? (x4): C_Small, symbol Device:C_Small
- added J? (x4): Conn_02x02_Counter_Clockwise, symbol Connector_Generic:Conn_02x02_Counter_Clockwise
- added J?: Conn_01x04_Female, symbol Connector:Conn_01x04_Female
- added R? (x2): R_Small, symbol Device:R_Small
- added U?: MCP2515-xST, Package_SO:TSSOP-20_4.4x6.5mm_P0.65mm, symbol Interface_CAN_LIN:MCP2515-xST
- added U?: MCP2551-I-SN, Package_SO:SOIC-8_3.9x4.9mm_P1.27mm, symbol Interface_CAN_LIN:MCP2551-I-SN
- added Y?: Crystal_Small, symbol Device:Crystal_Small
Connections:
- net GND: now also U?.10 (VSS), U?.2 (VSS)

Commit message: ohh
Parts:
- removed C?: C_Small, symbol Device:C_Small
- removed J? (x3): Conn_02x02_Counter_Clockwise, symbol Connector_Generic:Conn_02x02_Counter_Clockwise
- removed P5, P6, P7, P8: CONN_01X01, Socket_Arduino_Uno:Arduino_1pin, symbol Connector_Generic:Conn_01x01
- added C4: 100nF, Capacitor_SMD:C_0805_2012Metric_Pad1.18x1.45mm_HandSolder, symbol Device:C_Small
- added D1: power, LED_SMD:LED_0805_2012Metric_Pad1.15x1.40mm_HandSolder, symbol Device:LED_Small
- added J2: molex_3.0, Connector_Molex:Molex_Micro-Fit_3.0_43045-0421_2x02-1MP_P3.00mm_Horizontal, symbol Connector_Generic:Conn_02x02_Counter_Clockwise
- added J5: jumper, Connector_PinHeader_2.54mm:PinHeader_1x02_P2.54mm_Vertical, symbol Connector:Conn_01x02_Male
- added R3: 120, Resistor_SMD:R_0805_2012Metric_Pad1.20x1.40mm_HandSolder, symbol Device:R_Small
- added R4, R5: 10K, Resistor_SMD:R_0805_2012Metric_Pad1.20x1.40mm_HandSolder, symbol Device:R_Small
- added SW1: User, Button_Switch_SMD:SW_Push_1P1T_NO_6x6mm_H9.5mm, symbol Switch:SW_Push
- C1, C2: renamed from C?; value C_Small -> 22pF; footprint (none) -> Capacitor_SMD:C_0805_2012Metric_Pad1.18x1.45mm_HandSolder
- C3: renamed from C?; value C_Small -> 100nF; footprint (none) -> Capacitor_SMD:C_0805_2012Metric_Pad1.18x1.45mm_HandSolder
- J1: renamed from J?; value Conn_02x02_Counter_Clockwise -> molex_3.0; footprint (none) -> Connector_Molex:Molex_Micro-Fit_3.0_43045-0421_2x02-1MP_P3.00mm_Horizontal
- J6: renamed from J?; value Conn_01x04_Female -> UART2; footprint (none) -> Connector_PinSocket_2.54mm:PinSocket_1x04_P2.54mm_Vertical
- R1: renamed from R?; value R_Small -> 17K; footprint (none) -> Resistor_SMD:R_0805_2012Metric_Pad1.20x1.40mm_HandSolder
- R2: renamed from R?; value R_Small -> 10K; footprint (none) -> Resistor_SMD:R_0805_2012Metric_Pad1.20x1.40mm_HandSolder
- Y1: renamed from Y?; value Crystal_Small -> 16MHz; footprint (none) -> Crystal:Crystal_HC49-U_Vertical
- gave numbers to parts that had none: 2
Connections:
- net +5V: now also C3.1, J6.1 (Pin_1), R2.1, U1.20 (VDD), U2.3 (VDD), C4.1, R4.1, SW1.2
- net 0(Rx): now also J6.2 (Pin_2)
- net 1(Tx): now also J6.3 (Pin_3)
- net 11(**/MOSI): now also U1.16 (SI)
- net 12(MISO): now also U1.17 (SO)
- net 13(SCK): now also U1.14 (SCK)
- net 5(**): now also R5.1, SW1.1
- net 7: now also U1.18 (~{CS})
- net A4(SDA): no longer P3.2 (Pin_2)
- net A5(SCL): no longer P3.1 (Pin_1)
- net GND: now also C1.2, C2.2, C3.2, J1.3 (Pin_3), J6.4 (Pin_4), R1.2, C4.2, D1.1 (K), J2.3 (Pin_3), R5.2
- net at C1.1: now also U1.8 (OSC2), Y1.1
- net at C2.1: now also U1.9 (OSC1), Y1.2
- net at R2.2: now also U1.19 (~{RESET})
- net at R1.1: now also U2.8 (Rs)
- net CAN_Tx: now reaches U1.1 (TXCAN)
- net CAN_Tx: now also U2.1 (TXD)
- net CAN_Rx: now reaches U1.2 (RXCAN)
- net CAN_Rx: now also U2.4 (RXD)
- net CAN+: now reaches J1.1 (Pin_1)
- net CAN+: now also U2.7 (CANH), J2.1 (Pin_1), J5.1 (Pin_1)
- net CAN-: now reaches J1.2 (Pin_2)
- net CAN-: now also U2.6 (CANL), J2.2 (Pin_2), R3.2
- new net: J5.2 (Pin_2), R3.1
- new net: D1.2 (A), R4.2
- no-connect marks 5 -> 13
Other:
- note added: "CAN BUS"
- note added: "Power LED and button"
- note added: "UART & I2c"
- note removed: "Holes"
- moved on the sheet: C1, C2, C3, J1, J6, R1, R2, U1, U2, Y1

Commit message: mod plug
Parts:
- J1, J2: footprint Connector_Molex:Molex_Micro-Fit_3.0_43045-0421_2x02-1MP_P3.00mm_Horizontal -> Connector_Molex:Molex_Micro-Fit_3.0_43045-0400_2x02_P3.00mm_Horizontal
Changed lines of the file:
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@@
     (property "Reference" "J2" (id 0) (at 55.245 151.13 0))
     (property "Value" "molex_3.0" (id 1) (at 55.245 153.67 0))
-    (property "Footprint" "Connector_Molex:Molex_Micro-Fit_3.0_43045-0421_2x02-1MP_P3.00mm_Horizontal" (id 2) (at 53.975 157.48 0)
+    (property "Footprint" "Connector_Molex:Molex_Micro-Fit_3.0_43045-0400_2x02_P3.00mm_Horizontal" (id 2) (at 53.975 157.48 0)
       (effects (font (size 1.27 1.27)) hide)
     )
@@
     (property "Reference" "J1" (id 0) (at 54.61 165.1 0))
     (property "Value" "molex_3.0" (id 1) (at 54.61 167.64 0))
-    (property "Footprint" "Connector_Molex:Molex_Micro-Fit_3.0_43045-0421_2x02-1MP_P3.00mm_Horizontal" (id 2) (at 53.34 171.45 0)
+    (property "Footprint" "Connector_Molex:Molex_Micro-Fit_3.0_43045-0400_2x02_P3.00mm_Horizontal" (id 2) (at 53.34 171.45 0)
       (effects (font (size 1.27 1.27)) hide)
     )
@@
     )
     (path "/96cfb7bc-c878-46b6-a8e6-c7106d2d2c92"
-      (reference "J1") (unit 1) (value "molex_3.0") (footprint "Connector_Molex:Molex_Micro-Fit_3.0_43045-0421_2x02-1MP_P3.00mm_Horizontal")
+      (reference "J1") (unit 1) (value "molex_3.0") (footprint "Connector_Molex:Molex_Micro-Fit_3.0_43045-0400_2x02_P3.00mm_Horizontal")
     )
     (path "/3afa7e82-7e83-4f38-97e3-319360eebda5"
-      (reference "J2") (unit 1) (value "molex_3.0") (footprint "Connector_Molex:Molex_Micro-Fit_3.0_43045-0421_2x02-1MP_P3.00mm_Horizontal")
+      (reference "J2") (unit 1) (value "molex_3.0") (footprint "Connector_Molex:Molex_Micro-Fit_3.0_43045-0400_2x02_P3.00mm_Horizontal")
     )
     (path "/ee5bdd7e-81f3-4469-a2fa-4ddabc48417d"

Commit message: change footprint
Other:
- note added: "CAN Tranceiver TJA1050 or MCP2551"
- note added: "Connector"
- note added: "Note: For TJA1050 and MCP2551 both scheme are the same, just replace R1 to 0 Ohm if u use TJA1050."
- note added: "SPI to CAN controller"
- note added: "Termination Resistor"
- note removed: "CAN BUS"
- moved on the sheet: C3, C4, J1, J2, J5, R1, R3, U2
