File: arduino_can_bus_shield_canbus_custom/arduino_can_bus_shield_canbus_custom.kicad_pcb (KiCad board)
At the start: 2 copper layers, 56.4 x 53.3 mm, 40 parts, among them J1 USB_A, J2 jumper, J3 molex_3.0, J4 molex_3.0, J5 UART2, P1 Power, P2 Analog, P3 Digital, P4 Digital, SW1 User, U1 MCP2515-xST, U2 MAX3421E, U3 74LVC1G125, U4 74LVC1G125, U5 74LVC1G125, U6 74LVC1G125, U7 74LVC1G125, U8 74LVC1G125, U9 MCP2551-I-SN, Y1 Crystal_Small, Y2 16MHz

Commit message: arduino_shield update
Parts:
- added D2: power, LED_SMD:LED_0805_2012Metric_Pad1.15x1.40mm_HandSolder, F.Cu at (128.0, 122.9)
- added D3: power, LED_SMD:LED_0805_2012Metric_Pad1.15x1.40mm_HandSolder, F.Cu at (130.6, 122.9)
- added J6: i2C, Connector_PinHeader_2.54mm:PinHeader_1x04_P2.54mm_Vertical, F.Cu at (126.0, 142.2)
- added R11: 6K, Resistor_SMD:R_0805_2012Metric_Pad1.20x1.40mm_HandSolder, F.Cu at (123.4, 117.6)
- added R12: 4.7k, Resistor_SMD:R_0805_2012Metric, F.Cu at (126.1, 157.2)
- added R13: 4.7K, Resistor_SMD:R_0805_2012Metric, F.Cu at (126.0, 152.9)
- added R14: 6K, Resistor_SMD:R_0805_2012Metric_Pad1.20x1.40mm_HandSolder, F.Cu at (125.5, 117.6)
- R7: value 10K -> 6K
- moved C3 1.48 mm to (120.9, 143.4), turned to 90 degrees
- moved C4 1.44 mm to (121.2, 156.7), turned to -90 degrees
Routing:
- net /A4(SDA): track 0.00 -> 23.6 mm
- net /A5(SCL): track 0.00 -> 18.6 mm
- net +3V3: track 38.0 -> 56.0 mm, vias 1 -> 2
- net /2: track 0.00 -> 9.11 mm
- net Net-(D3-Pad2): track 0.00 -> 6.44 mm
- net Net-(D2-Pad2): track 0.00 -> 5.94 mm
- net /4: track 0.00 -> 5.30 mm
- added copper zone on B.Cu, net GND
- added copper zone on F.Cu, net GND

Commit message: arduino_shield update
Parts:
- moved R4 0.25 mm to (105.4, 129.0)
Connections:
- J1 pad 5: unconnected-(J1-Pad5) -> GND
Routing:
- net +3V3: track 56.0 -> 74.0 mm
- net GND: track 0.00 -> 12.0 mm, vias 0 -> 42
- net +5V: track 262.5 -> 266.3 mm

Commit message: regular update
Parts:
- Y1: value Crystal_Small -> 12MHz
- moved J5 47.2 mm to (128.8, 164.3), turned to 180 degrees
- moved R6 43.9 mm to (93.0, 163.1), turned to 0 degrees
- moved P3 42.0 mm to (133.9, 119.6), turned to -90 degrees
- moved R8 40.9 mm to (130.3, 116.6), turned to -90 degrees
- moved P2 40.0 mm to (85.6, 151.6), turned to -90 degrees
- moved D1 39.7 mm to (88.4, 118.6), turned to 0 degrees
- moved C5 38.4 mm to (127.8, 116.6), turned to 90 degrees
- moved J2 38.0 mm to (94.5, 159.0), turned to -90 degrees
- moved R7 37.7 mm to (88.4, 120.9), turned to 0 degrees
- moved R12 36.9 mm to (89.4, 153.3), turned to 90 degrees
- moved P4 36.8 mm to (133.9, 146.6), turned to -90 degrees
- moved P1 36.0 mm to (85.6, 128.8), turned to -90 degrees
- moved R14 35.2 mm to (129.0, 152.7), turned to 180 degrees
- moved J3 34.0 mm to (117.1, 159.8), turned to 180 degrees
- moved SW1 33.9 mm to (123.2, 117.1), turned to 0 degrees
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Routing:
- net Net-(D3-Pad2): track 6.44 -> 2.02 mm
- net Net-(D2-Pad2): track 5.94 -> 2.04 mm
Other:
- board size 56.4 x 53.3 mm -> 53.3 x 56.4 mm
- board text added: "(2)"
- board text added: "(4)"
- board text added: "12MHz"
- board text added: "3v3"
- board text added: "5V"
- board text added: "8/16 MHz"
- board text added: "GND"
- board text added: "Rx"
- board text added: "SCL"
- board text added: "SDA"
- board text added: "Tx"
- board text added: "USB canbus Shield Rev 1.1 By SamsonChau 2022-5-20"
- board text added: "power"
- board text added: "user"
