File: arduino_can_bus_shield_canbus_custom/arduino_can_bus_shield_canbus_custom.kicad_sch (KiCad schematic)
At the start: 40 parts, among them J1 USB_A, J2 jumper, J3 molex_3.0, J4 molex_3.0, J5 UART2, P1 Power, P2 Analog, P3 Digital, P4 Digital, SW1 User, U1 MCP2515-xST, U2 MAX3421E, U3 74LVC1G125, U4 74LVC1G125, U5 74LVC1G125, U6 74LVC1G125, U7 74LVC1G125, U8 74LVC1G125, U9 MCP2551-I-SN, Y1 Crystal_Small, Y2 16MHz

Commit message: arduino_shield update
Parts:
- added D2, D3: power, LED_SMD:LED_0805_2012Metric_Pad1.15x1.40mm_HandSolder, symbol Device:LED_Small
- added J6: (no value), symbol Connector_Generic:Conn_01x04
- added R11, R14: 6K, Resistor_SMD:R_0805_2012Metric_Pad1.20x1.40mm_HandSolder, symbol Device:R_Small
- added R12, R13: (no value), symbol Device:R_Small
- R7: value 10K -> 6K
Connections:
- net +3V3: now also J6.1 (Pin_1), R12.1, R13.1
- net 2: now also R14.1
- net 4: now also R11.1
- net A4(SDA): now also J6.3 (Pin_3), R12.2
- net A5(SCL): now also J6.4 (Pin_4), R13.2
- net GND: now also D2.1 (K), D3.1 (K), J6.2 (Pin_2)
- new net: D3.2 (A), R14.2
- new net: D2.2 (A), R11.2
Other:
- moved on the sheet: R8, SW1

Commit message: arduino_shield update
Parts:
- J6: value (none) -> i2C; footprint (none) -> Connector_PinHeader_2.54mm:PinHeader_1x04_P2.54mm_Vertical
- R12: value (none) -> 4.7k; footprint (none) -> Resistor_SMD:R_0805_2012Metric
- R13: value (none) -> 4.7K; footprint (none) -> Resistor_SMD:R_0805_2012Metric
Connections:
- net GND: now also J1.5 (Shield)
Changed lines of the file:
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@@
   (junction (at 236.22 55.245) (diameter 1.016) (color 0 0 0 0)
+  )
+  (junction (at 30.48 112.395) (diameter 0) (color 0 0 0 0)
   )
   (junction (at 127.635 157.48) (diameter 0) (color 0 0 0 0)
@@
     (stroke (width 0) (type solid) (color 0 0 0 0))
   )
+  (wire (pts (xy 27.94 112.395) (xy 30.48 112.395))
+    (stroke (width 0) (type default) (color 0 0 0 0))
+  )
   (wire (pts (xy 51.435 116.84) (xy 51.435 116.205))
     (stroke (width 0) (type default) (color 0 0 0 0))
@@
       (effects (font (size 1.27 1.27)) hide)
     )
-    (property "Value" "" (id 1) (at 258.445 90.17 0))
+    (property "Value" "+3.3V" (id 1) (at 258.445 90.17 0))
     (property "Footprint" "" (id 2) (at 258.445 95.885 0)
       (effects (font (size 1.27 1.27)) hide)
@@
       (effects (font (size 1.27 1.27)) (justify left))
     )
-    (property "Value" "" (id 1) (at 275.59 114.2999 0)
-      (effects (font (size 1.27 1.27)) (justify left))
-    )
-    (property "Footprint" "" (id 2) (at 273.685 113.03 0)
+    (property "Value" "4.7K" (id 1) (at 275.59 114.2999 0)
+      (effects (font (size 1.27 1.27)) (justify left))
+    )
+    (property "Footprint" "Resistor_SMD:R_0805_2012Metric" (id 2) (at 273.685 113.03 0)
       (effects (font (size 1.27 1.27)) hide)
     )
@@
       (effects (font (size 1.27 1.27)) (justify left))
     )
-    (property "Value" "" (id 1) (at 260.985 114.3 0)
-      (effects (font (size 1.27 1.27)) (justify left))
-    )
-    (property "Footprint" "" (id 2) (at 266.065 113.03 0)
+    (property "Value" "4.7k" (id 1) (at 260.985 114.3 0)
+      (effects (font (size 1.27 1.27)) (justify left))
+    )
+    (property "Footprint" "Resistor_SMD:R_0805_2012Metric" (id 2) (at 266.065 113.03 0)
       (effects (font (size 1.27 1.27)) hide)
     )
@@
       (effects (font (size 1.27 1.27)) (justify left))
     )
-    (property "Value" "" (id 1) (at 266.7 100.9649 0)
-      (effects (font (size 1.27 1.27)) (justify left))
-    )
-    (property "Footprint" "" (id 2) (at 263.525 98.425 0)
-      (effects (font (size 1.27 1.27)) hide)
-    )
+    (property "Value" "i2C" (id 1) (at 266.7 100.9649 0)
+      (effects (font (size 1.27 1.27)) (justify left))
+    )
+    (property "Footprint" "Connector_PinHeader_2.54mm:PinHeader_1x04_P2.54mm_Vertical" (id 2) (at 263.525 98.425 0)
+      (effects (font (size 1.27 1.27)) hide)
+    )

Commit message: regular update
Parts:
- Y1: value Crystal_Small -> (none)
Changed lines of the file:
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@@
     (in_bom yes) (on_board yes) (fields_autoplaced)
     (property "Reference" "Y1" (id 0) (at 34.925 147.32 0))
-    (property "Value" "Crystal_Small" (id 1) (at 34.925 149.86 0))
+    (property "Value" "" (id 1) (at 34.925 149.86 0))
     (property "Footprint" "Crystal:Crystal_SMD_HC49-SD" (id 2) (at 34.925 154.305 0)
       (effects (font (size 1.27 1.27)) hide)
@@
     )
     (path "/c73b1ee9-112b-4c0e-98a3-be08fbdc8955"
-      (reference "Y1") (unit 1) (value "Crystal_Small") (footprint "Crystal:Crystal_SMD_HC49-SD")
+      (reference "Y1") (unit 1) (value "12MHz") (footprint "Crystal:Crystal_SMD_HC49-SD")
     )
     (path "/dd01ca49-c8a2-4580-af9a-2e9bce9769bc"
