File: VESC_MINI_Shield_IGGG/VESC_MINI_Shield_IGGG.kicad_sch (KiCad schematic)
At the start: 8 parts

Commit message: v2.1 added BOM
Parts:
- gave numbers to parts that had none: 8
Changed lines of the file:
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@@
   (symbol (lib_id "Connector_Generic:Conn_01x06") (at 66.04 68.58 0) (unit 1)
     (in_bom yes) (on_board yes) (fields_autoplaced)
-    (property "Reference" "J?" (id 0) (at 68.58 68.5799 0)
+    (property "Reference" "J1" (id 0) (at 68.58 68.5799 0)
       (effects (font (size 1.27 1.27)) (justify left))
     )
@@
   (symbol (lib_id "Device:R_Small") (at 86.36 73.66 0) (unit 1)
     (in_bom yes) (on_board yes)
-    (property "Reference" "R?" (id 0) (at 82.55 72.39 0)
+    (property "Reference" "R1" (id 0) (at 82.55 72.39 0)
       (effects (font (size 1.27 1.27)) (justify left))
     )
@@
   (symbol (lib_id "Connector_Generic:Conn_01x06") (at 100.33 88.9 0) (unit 1)
     (in_bom yes) (on_board yes) (fields_autoplaced)
-    (property "Reference" "J?" (id 0) (at 102.87 88.8999 0)
+    (property "Reference" "J6" (id 0) (at 102.87 88.8999 0)
       (effects (font (size 1.27 1.27)) (justify left))
     )
@@
   (symbol (lib_id "power:GND") (at 49.53 87.63 0) (unit 1)
     (in_bom yes) (on_board yes) (fields_autoplaced)
-    (property "Reference" "#PWR?" (id 0) (at 49.53 93.98 0)
+    (property "Reference" "#PWR0106" (id 0) (at 49.53 93.98 0)
       (effects (font (size 1.27 1.27)) hide)
     )
@@
   (symbol (lib_id "power:GND") (at 54.61 63.5 0) (unit 1)
     (in_bom yes) (on_board yes) (fields_autoplaced)
-    (property "Reference" "#PWR?" (id 0) (at 54.61 69.85 0)
+    (property "Reference" "#PWR0104" (id 0) (at 54.61 69.85 0)
       (effects (font (size 1.27 1.27)) hide)
     )
@@
   (symbol (lib_id "power:+3.3V") (at 86.36 66.04 0) (unit 1)
     (in_bom yes) (on_board yes) (fields_autoplaced)
-    (property "Reference" "#PWR?" (id 0) (at 86.36 69.85 0)
+    (property "Reference" "#PWR0101" (id 0) (at 86.36 69.85 0)
       (effects (font (size 1.27 1.27)) hide)
     )
@@
   (symbol (lib_id "power:GND") (at 90.17 76.2 0) (unit 1)
     (in_bom yes) (on_board yes) (fields_autoplaced)
-    (property "Reference" "#PWR?" (id 0) (at 90.17 82.55 0)
+    (property "Reference" "#PWR0102" (id 0) (at 90.17 82.55 0)
       (effects (font (size 1.27 1.27)) hide)
     )
@@
   (symbol (lib_id "power:+5V") (at 54.61 76.2 0) (unit 1)
     (in_bom yes) (on_board yes) (fields_autoplaced)
-    (property "Reference" "#PWR?" (id 0) (at 54.61 80.01 0)
+    (property "Reference" "#PWR0105" (id 0) (at 54.61 80.01 0)
       (effects (font (size 1.27 1.27)) hide)
     )
@@
   (symbol (lib_id "Connector_Generic:Conn_02x02_Counter_Clockwise") (at 78.74 124.46 0) (unit 1)
     (in_bom yes) (on_board yes) (fields_autoplaced)
-    (property "Reference" "J?" (id 0) (at 80.01 118.11 0))
+    (property "Reference" "J3" (id 0) (at 80.01 118.11 0))
     (property "Value" "CAN_MOLEX" (id 1) (at 80.01 120.65 0))
     (property "Footprint" "Connector_Molex:Molex_Micro-Fit_3.0_43045-0400_2x02_P3.00mm_Horizontal" (id 2) (at 78.74 124.46 0)
@@
   (symbol (lib_id "Connector_Generic:Conn_01x04") (at 66.04 90.17 0) (unit 1)
     (in_bom yes) (on_board yes) (fields_autoplaced)
-    (property "Reference" "J?" (id 0) (at 68.58 90.1699 0)
+    (property "Reference" "J2" (id 0) (at 68.58 90.1699 0)
       (effects (font (size 1.27 1.27)) (justify left))
     )
@@
   (symbol (lib_id "Device:LED_Small") (at 86.36 68.58 90) (unit 1)
     (in_bom yes) (on_board yes)
-    (property "Reference" "D?" (id 0) (at 81.28 67.31 90)
+    (property "Reference" "D1" (id 0) (at 81.28 67.31 90)
       (effects (font (size 1.27 1.27)) (justify right))
     )
@@
   (symbol (lib_id "power:GND") (at 86.36 76.2 0) (unit 1)
     (in_bom yes) (on_board yes) (fields_autoplaced)
-    (property "Reference" "#PWR?" (id 0) (at 86.36 82.55 0)
+    (property "Reference" "#PWR0103" (id 0) (at 86.36 82.55 0)
       (effects (font (size 1.27 1.27)) hide)
     )
@@
   (symbol (lib_id "power:+5V") (at 53.34 95.25 0) (unit 1)
     (in_bom yes) (on_board yes) (fields_autoplaced)
-    (property "Reference" "#PWR?" (id 0) (at 53.34 99.06 0)
+    (property "Reference" "#PWR0107" (id 0) (at 53.34 99.06 0)
       (effects (font (size 1.27 1.27)) hide)
     )
@@
   (symbol (lib_id "Connector_Generic:Conn_01x06") (at 81.28 106.68 270) (unit 1)
     (in_bom yes) (on_board yes) (fields_autoplaced)
-    (property "Reference" "J?" (id 0) (at 80.01 110.49 90))
+    (property "Reference" "J4" (id 0) (at 80.01 110.49 90))
     (property "Value" "Encoder" (id 1) (at 80.01 113.03 90))
     (property "Footprint" "" (id 2) (at 81.28 106.68 0)
@@
   (symbol (lib_id "Connector_Generic:Conn_01x07") (at 100.33 71.12 0) (unit 1)
     (in_bom yes) (on_board yes) (fields_autoplaced)
-    (property "Reference" "J?" (id 0) (at 102.87 69.8499 0)
+    (property "Reference" "J5" (id 0) (at 102.87 69.8499 0)
       (effects (font (size 1.27 1.27)) (justify left))
     )
@@
   )
   (symbol_instances
+    (path "/345fcd19-152d-45f9-9f51-044de98d9f74"
+      (reference "#PWR0101") (unit 1) (value "+3.3V") (footprint "")
+    )
+    (path "/57c5edf6-bae1-41cd-b759-6b298b7760e7"
+      (reference "#PWR0102") (unit 1) (value "GND") (footprint "")
+    )
+    (path "/bef9905f-5d77-49a6-a305-5da85f9676e0"
+      (reference "#PWR0103") (unit 1) (value "GND") (footprint "")
+    )
+    (path "/323713c0-4e84-4403-b6ce-e2f8e4993c97"
+      (reference "#PWR0104") (unit 1) (value "GND") (footprint "")
+    )
+    (path "/600d23f0-1422-4a49-beff-750dc11dd6b8"
+      (reference "#PWR0105") (unit 1) (value "+5V") (footprint "")
+    )
     (path "/2130a471-0818-47d9-934b-0c1900e5f958"
-      (reference "#PWR?") (unit 1) (value "GND") (footprint "")
-    )
-    (path "/323713c0-4e84-4403-b6ce-e2f8e4993c97"
-      (reference "#PWR?") (unit 1) (value "GND") (footprint "")
-    )
-    (path "/345fcd19-152d-45f9-9f51-044de98d9f74"
-      (reference "#PWR?") (unit 1) (value "+3.3V") (footprint "")
-    )
-    (path "/57c5edf6-bae1-41cd-b759-6b298b7760e7"
-      (reference "#PWR?") (unit 1) (value "GND") (footprint "")
-    )
-    (path "/600d23f0-1422-4a49-beff-750dc11dd6b8"
-      (reference "#PWR?") (unit 1) (value "+5V") (footprint "")
-    )
-    (path "/bef9905f-5d77-49a6-a305-5da85f9676e0"
-      (reference "#PWR?") (unit 1) (value "GND") (footprint "")
+      (reference "#PWR0106") (unit 1) (value "GND") (footprint "")
     )
     (path "/e30a5edd-672f-4fa8-b6f2-35cadc523f91"
-      (reference "#PWR?") (unit 1) (value "+5V") (footprint "")
+      (reference "#PWR0107") (unit 1) (value "+5V") (footprint "")
     )
     (path "/bdb20739-f361-4f6b-b100-244bf2b0cb72"
-      (reference "D?") (unit 1) (value "PWR") (footprint "LED_SMD:LED_0805_2012Metric_Pad1.15x1.40mm_HandSolder")
+      (reference "D1") (unit 1) (value "PWR") (footprint "LED_SMD:LED_0805_2012Metric_Pad1.15x1.40mm_HandSolder")
     )
     (path "/0556d257-88b4-4108-8d5d-2c5f4a9b82de"
-      (reference "J?") (unit 1) (value "Sensor") (footprint "Connector_PinHeader_2.00mm:PinHeader_1x06_P2.00mm_Vertical")
+      (reference "J1") (unit 1) (value "Sensor") (footprint "Connector_PinHeader_2.00mm:PinHeader_1x06_P2.00mm_Vertical")
+    )
+    (path "/8c795137-91f5-4740-ad66-b1e3e1450c80"
+      (reference "J2") (unit 1) (value "CAN") (footprint "Connector_PinHeader_2.00mm:PinHeader_1x04_P2.00mm_Vertical")
+    )
+    (path "/6f7c8405-4ea4-41d4-a219-a4db7dafd620"
+      (reference "J3") (unit 1) (value "CAN_MOLEX") (footprint "Connector_Molex:Molex_Micro-Fit_3.0_43045-0400_2x02_P3.00mm_Horizontal")
+    )
+    (path "/ebc751ce-b376-4168-8034-5a2e159e2924"
+      (reference "J4") (unit 1) (value "Encoder") (footprint "")
+    )
+    (path "/f25ce7ca-921e-43e9-a994-cbc8850eb654"
+      (reference "J5") (unit 1) (value "General") (footprint "Connector_PinHeader_2.00mm:PinHeader_1x07_P2.00mm_Vertical")
     )
     (path "/15c94cca-2203-45a5-94f6-178bcdb32a6f"
-      (reference "J?") (unit 1) (value "NC") (footprint "Connector_PinHeader_2.00mm:PinHeader_1x06_P2.00mm_Vertical")
-    )
-    (path "/6f7c8405-4ea4-41d4-a219-a4db7dafd620"
-      (reference "J?") (unit 1) (value "CAN_MOLEX") (footprint "Connector_Molex:Molex_Micro-Fit_3.0_43045-0400_2x02_P3.00mm_Horizontal")
-    )
-    (path "/8c795137-91f5-4740-ad66-b1e3e1450c80"
-      (reference "J?") (unit 1) (value "CAN") (footprint "Connector_PinHeader_2.00mm:PinHeader_1x04_P2.00mm_Vertical")
-    )
-    (path "/ebc751ce-b376-4168-8034-5a2e159e2924"
-      (reference "J?") (unit 1) (value "Encoder") (footprint "")
-    )
-    (path "/f25ce7ca-921e-43e9-a994-cbc8850eb654"
-      (reference "J?") (unit 1) (value "General") (footprint "Connector_PinHeader_2.00mm:PinHeader_1x07_P2.00mm_Vertical")
+      (reference "J6") (unit 1) (value "NC") (footprint "Connector_PinHeader_2.00mm:PinHeader_1x06_P2.00mm_Vertical")
     )
     (path "/0b74ab11-ad40-46d6-950a-4eff00b2edb1"
-      (reference "R?") (unit 1) (value "3.3K") (footprint "")
-    )
-  )
+      (reference "R1") (unit 1) (value "3.3K") (footprint "")
+    )
+  )
