File: arduino_can_bus_shield_v2.1/arduino_can_bus_shield_v2.1.kicad_sch (KiCad schematic)
At the start: 32 parts, among them J1 Power, J2 Digital/PWM, J3 Analog, J4 Digital/PWM, J6 xt60 male, J7 molex_3.0, M1 MPU9250_module, SW1 User, SW2 User, SW3 SW_DIP_x04, U1 MP1584, U2 MCP2551-I-SN, U3 MCP2515-xST, Y1 16MHz

Commit message: Add files via upload
Connections:
- net *11 is gone; now on net 11(**/MOSI): J2.7 (Pin_7)
- net *9 is gone; now on net 9(**): J2.9 (Pin_9)
- net +3.3V is gone; now on net +3V3: Brd1.2 (VCC)
- net 12 is gone; now on net 12(MISO): J2.6 (Pin_6)
- net 13 is gone; now on net 13(SCK): J2.5 (Pin_5)
- net A4(SDA) is gone; now on net SDA/A4: Brd1.4 (SDA), M1.3 (SDA)
- net A5(SCL) is gone; now on net SCL/A5: Brd1.3 (SCL), M1.2 (SCL)
Changed lines of the file:
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@@
     (effects (font (size 1.27 1.27)) (justify right bottom))
+  )
+  (label "11(**/MOSI)" (at 119.38 26.416 180)
+    (effects (font (size 1.524 1.524)) (justify right bottom))
   )
   (label "A2" (at 21.59 64.77 0)
@@
     (effects (font (size 1.27 1.27)) (justify left bottom))
   )
+  (label "13(SCK)" (at 74.93 36.83 0)
+    (effects (font (size 1.524 1.524)) (justify left bottom))
+  )
   (label "2" (at 74.93 72.39 180)
     (effects (font (size 1.27 1.27)) (justify right bottom))
@@
     (effects (font (size 1.27 1.27)) (justify left bottom))
   )
-  (label "13" (at 74.93 36.83 180)
-    (effects (font (size 1.27 1.27)) (justify right bottom))
+  (label "SCL{slash}A5" (at 117.094 166.624 180)
+    (effects (font (size 1.27 1.27)) (justify right bottom))
+  )
+  (label "11(**/MOSI)" (at 74.93 41.91 0)
+    (effects (font (size 1.524 1.524)) (justify left bottom))
   )
   (label "can_enable" (at 144.526 135.382 0)
     (effects (font (size 1.27 1.27)) (justify left bottom))
   )
-  (label "12" (at 74.93 39.37 180)
-    (effects (font (size 1.27 1.27)) (justify right bottom))
+  (label "12(MISO)" (at 74.93 39.37 0)
+    (effects (font (size 1.524 1.524)) (justify left bottom))
+  )
+  (label "~{RESET}" (at 19.05 36.83 0)
+    (effects (font (size 1.27 1.27)) (justify left bottom))
   )
   (label "13(SCK)" (at 119.38 34.036 180)
     (effects (font (size 1.524 1.524)) (justify right bottom))
   )
-  (label "~{RESET}" (at 19.05 36.83 0)
-    (effects (font (size 1.27 1.27)) (justify left bottom))
-  )
   (label "*10" (at 74.93 44.45 180)
     (effects (font (size 1.27 1.27)) (justify right bottom))
@@
   (label "CAN-" (at 144.78 143.002 0)
     (effects (font (size 1.27 1.27)) (justify left bottom))
-  )
-  (label "A5(SCL)" (at 117.094 166.624 180)
-    (effects (font (size 1.27 1.27)) (justify right bottom))
   )
   (label "A0" (at 57.15 96.012 0)
@@
     (effects (font (size 1.524 1.524)) (justify left bottom))
   )
-  (label "A4(SDA)" (at 37.338 144.018 0)
-    (effects (font (size 1.524 1.524)) (justify left bottom))
-  )
   (label "CAN_Tx" (at 105.156 86.868 180)
     (effects (font (size 1.27 1.27)) (justify right bottom))
@@
     (effects (font (size 1.524 1.524)) (justify right bottom))
   )
-  (label "*11" (at 74.93 41.91 180)
-    (effects (font (size 1.27 1.27)) (justify right bottom))
-  )
   (label "*3" (at 74.93 69.85 180)
     (effects (font (size 1.27 1.27)) (justify right bottom))
   )
+  (label "SCL{slash}A5" (at 37.338 141.478 0)
+    (effects (font (size 1.27 1.27)) (justify left bottom))
+  )
   (label "A1" (at 21.59 62.23 0)
     (effects (font (size 1.27 1.27)) (justify left bottom))
   )
+  (label "9(**)" (at 74.93 46.99 0)
+    (effects (font (size 1.524 1.524)) (justify left bottom))
+  )
   (label "TX{slash}1" (at 74.93 74.93 180)
     (effects (font (size 1.27 1.27)) (justify right bottom))
@@
     (effects (font (size 1.27 1.27)) (justify right bottom))
   )
+  (label "SDA{slash}A4" (at 37.338 144.018 0)
+    (effects (font (size 1.27 1.27)) (justify left bottom))
+  )
   (label "A0" (at 21.59 59.69 0)
     (effects (font (size 1.27 1.27)) (justify left bottom))
@@
     (effects (font (size 1.27 1.27)) (justify right bottom))
   )
-  (label "A5(SCL)" (at 37.338 141.478 0)
-    (effects (font (size 1.524 1.524)) (justify left bottom))
-  )
-  (label "A4(SDA)" (at 117.094 169.164 180)
-    (effects (font (size 1.27 1.27)) (justify right bottom))
-  )
   (label "Vin" (at 26.67 26.67 270)
     (effects (font (size 1.27 1.27)) (justify right bottom))
@@
     (effects (font (size 1.27 1.27)) (justify right bottom))
   )
-  (label "*9" (at 74.93 46.99 180)
-    (effects (font (size 1.27 1.27)) (justify right bottom))
-  )
   (label "CAN-" (at 105.664 140.462 180)
     (effects (font (size 1.27 1.27)) (justify right bottom))
@@
     (effects (font (size 1.27 1.27)) (justify right bottom))
   )
-  (label "11(**/MOSI)" (at 119.38 26.416 180)
-    (effects (font (size 1.524 1.524)) (justify right bottom))
-  )
   (label "can_enable" (at 117.856 78.994 0)
     (effects (font (size 1.27 1.27)) (justify left bottom))
+  )
+  (label "SDA{slash}A4" (at 117.094 169.164 180)
+    (effects (font (size 1.27 1.27)) (justify right bottom))
   )
   (label "9(**)" (at 27.686 106.172 0)
@@
     (pin "1")
   )
-  (symbol (lib_name "+3.3V_1") (lib_id "power:+3.3V") (at 41.148 133.858 0) (unit 1)
-    (in_bom yes) (on_board yes) (fields_autoplaced)
-    (property "Reference" "#PWR0122" (id 0) (at 41.148 137.668 0)
-      (effects (font (size 1.27 1.27)) hide)
-    )
-    (property "Value" "+3.3V" (id 1) (at 41.148 128.143 0))
-    (property "Footprint" "" (id 2) (at 41.148 133.858 0)
-      (effects (font (size 1.27 1.27)) hide)
-    )
-    (property "Datasheet" "" (id 3) (at 41.148 133.858 0)
-      (effects (font (size 1.27 1.27)) hide)
-    )
-    (pin "1")
-  )
   (symbol (lib_id "power:GND") (at 36.83 168.148 0) (unit 1)
     (in_bom yes) (on_board yes) (fields_autoplaced)
@@
     (pin "1")
     (pin "2")
+  )
+  (symbol (lib_id "power:+3V3") (at 41.148 133.858 0) (unit 1)
+    (in_bom yes) (on_board yes)
+    (property "Reference" "#PWR0111" (id 0) (at 41.148 137.668 0)
+      (effects (font (size 1.27 1.27)) hide)
+    )
+    (property "Value" "+3.3V" (id 1) (at 41.529 130.81 0)
+      (effects (font (size 1.27 1.27)) (justify left))
+    )
+    (property "Footprint" "" (id 2) (at 41.148 133.858 0))
+    (property "Datasheet" "" (id 3) (at 41.148 133.858 0))
+    (pin "1")
   )
   (symbol (lib_id "power:GND") (at 102.616 104.648 0) (unit 1)
@@
       (reference "#PWR0110") (unit 1) (value "GND") (footprint "")
     )
+    (path "/93f9769f-f781-4897-b7df-5e885966d4de"
+      (reference "#PWR0111") (unit 1) (value "+3.3V") (footprint "")
+    )
     (path "/857460db-715f-48cb-b70e-f471e70e1068"
       (reference "#PWR0112") (unit 1) (value "GND") (footprint "")
@@
       (reference "#PWR0121") (unit 1) (value "GND") (footprint "")
     )
-    (path "/5ce183c6-2967-42c5-830a-acf6b121894c"
-      (reference "#PWR0122") (unit 1) (value "+3.3V") (footprint "")
-    )
     (path "/d2206518-63a4-4f61-8014-f99d9cb05acc"

Commit message: v2.1 added BOM
Connections:
- net GND: no longer U1.IN1- (VIN-), U1.OUT1- (VOUT-)
- net VCC: no longer U1.OUT1+ (VOUT+)
- net at C1.1, D2.1 (K), U1.IN2+ (VIN+): no longer U1.IN1+ (VIN+)
Changed lines of the file:
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@@
       (effects (font (size 1.27 1.27)) hide)
     )
-    (property "Datasheet" "" (id 3) (at 39.37 39.37 0))
+    (property "Datasheet" "~" (id 3) (at 39.37 39.37 0))
     (pin "1")
     (pin "2")
@@
       (effects (font (size 1.27 1.27)) hide)
     )
-    (property "Datasheet" "" (id 3) (at 57.15 36.83 0))
+    (property "Datasheet" "~" (id 3) (at 57.15 36.83 0))
     (pin "1")
     (pin "10")
@@
       (effects (font (size 1.27 1.27)) hide)
     )
-    (property "Datasheet" "" (id 3) (at 57.15 67.31 0))
+    (property "Datasheet" "~" (id 3) (at 57.15 67.31 0))
     (pin "1")
     (pin "2")
@@
       (effects (font (size 1.27 1.27)) (justify left bottom) hide)
     )
-    (pin "IN1+")
-    (pin "IN1-")
     (pin "IN2+")
     (pin "IN2-")
-    (pin "OUT1+")
-    (pin "OUT1-")
     (pin "OUT2+")
     (pin "OUT2-")
@@
     (pin "1")
   )
-  (symbol (lib_name "D_Schottky_2") (lib_id "Device:D_Schottky") (at 21.844 166.878 270) (unit 1)
+  (symbol (lib_id "Device:D_Schottky") (at 21.844 166.878 270) (unit 1)
     (in_bom yes) (on_board yes)
     (property "Reference" "D1" (id 0) (at 17.526 166.37 90)
